Commit message: [INIT] add urdf and transmissions (todo)

File: sobit_light_description/urdf/arm/open_manipulator_x.urdf.xacro (robot description, xacro)
@@ -8,5 +8,5 @@
       <origin xyz="0 0 0" rpy="0 0 ${M_PI/2}"/>
       <geometry>
-        <mesh filename="file://$(find open_manipulator_x_description)/meshes/omx1_link_base.stl" scale="0.001 0.001 0.001"/>
+        <mesh filename="file://$(find sobit_light_description)/meshes/omx1_link_base.stl" scale="0.001 0.001 0.001"/>
       </geometry>
       <material name="grey"/>
@@ -16,5 +16,5 @@
       <origin xyz="0 0 0" rpy="0 0 ${M_PI/2}"/>
       <geometry>
-        <mesh filename="file://$(find open_manipulator_x_description)/meshes/omx1_link_base.stl" scale="0.001 0.001 0.001"/>
+        <mesh filename="file://$(find sobit_light_description)/meshes/omx1_link_base.stl" scale="0.001 0.001 0.001"/>
       </geometry>
     </collision>
@@ -39,12 +39,12 @@
       <origin xyz="0 0 0" rpy="0 0 ${M_PI/2}"/>
       <geometry>
-        <mesh filename="file://$(find open_manipulator_x_description)/meshes/omx1_link1.stl" scale="0.001 0.001 0.001"/>
-      </geometry>
-      <material name="grey"/>
-    </visual>
-    <collision>
-      <origin xyz="0 0 0" rpy="0 0 ${M_PI/2}"/>
-      <geometry>
-        <mesh filename="file://$(find open_manipulator_x_description)/meshes/omx1_link1.stl" scale="0.001 0.001 0.001"/>
+        <mesh filename="file://$(find sobit_light_description)/meshes/omx1_link1.stl" scale="0.001 0.001 0.001"/>
+      </geometry>
+      <material name="grey"/>
+    </visual>
+    <collision>
+      <origin xyz="0 0 0" rpy="0 0 ${M_PI/2}"/>
+      <geometry>
+        <mesh filename="file://$(find sobit_light_description)/meshes/omx1_link1.stl" scale="0.001 0.001 0.001"/>
       </geometry>
     </collision>
@@ -70,5 +70,5 @@
       <origin xyz="0 0 0.0" rpy="0 0 ${M_PI/2}"/>
       <geometry>
-        <mesh filename="file://$(find open_manipulator_x_description)/meshes/omx1_link2.stl" scale="0.001 0.001 0.001"/>
+        <mesh filename="file://$(find sobit_light_description)/meshes/omx1_link2.stl" scale="0.001 0.001 0.001"/>
       </geometry>
       <material name="grey"/>
@@ -77,5 +77,5 @@
       <origin xyz="0 0 0.0" rpy="0 0 ${M_PI/2}"/>
       <geometry>
-        <mesh filename="file://$(find open_manipulator_x_description)/meshes/omx1_link2.stl" scale="0.001 0.001 0.001"/>
+        <mesh filename="file://$(find sobit_light_description)/meshes/omx1_link2.stl" scale="0.001 0.001 0.001"/>
       </geometry>
     </collision>
@@ -101,12 +101,12 @@
       <origin xyz="0 0 0" rpy="0 0 ${M_PI/2}"/>
       <geometry>
-        <mesh filename="file://$(find open_manipulator_x_description)/meshes/omx1_link3.stl" scale="0.001 0.001 0.001"/>
-      </geometry>
-      <material name="grey"/>
-    </visual>
-    <collision>
-      <origin xyz="0 0 0" rpy="0 0 ${M_PI/2}"/>
-      <geometry>
-        <mesh filename="file://$(find open_manipulator_x_description)/meshes/omx1_link3.stl" scale="0.001 0.001 0.001"/>
+        <mesh filename="file://$(find sobit_light_description)/meshes/omx1_link3.stl" scale="0.001 0.001 0.001"/>
+      </geometry>
+      <material name="grey"/>
+    </visual>
+    <collision>
+      <origin xyz="0 0 0" rpy="0 0 ${M_PI/2}"/>
+      <geometry>
+        <mesh filename="file://$(find sobit_light_description)/meshes/omx1_link3.stl" scale="0.001 0.001 0.001"/>
       </geometry>
     </collision>
@@ -132,12 +132,12 @@
       <origin xyz="0 0 0" rpy="0 0 ${M_PI/2}"/>
       <geometry>
-        <mesh filename="file://$(find open_manipulator_x_description)/meshes/omx1_link4.stl" scale="0.001 0.001 0.001"/>
-      </geometry>
-      <material name="grey"/>
-    </visual>
-    <collision>
-      <origin xyz="0 0 0" rpy="0 0 ${M_PI/2}"/>
-      <geometry>
-        <mesh filename="file://$(find open_manipulator_x_description)/meshes/omx1_link4.stl" scale="0.001 0.001 0.001"/>
+        <mesh filename="file://$(find sobit_light_description)/meshes/omx1_link4.stl" scale="0.001 0.001 0.001"/>
+      </geometry>
+      <material name="grey"/>
+    </visual>
+    <collision>
+      <origin xyz="0 0 0" rpy="0 0 ${M_PI/2}"/>
+      <geometry>
+        <mesh filename="file://$(find sobit_light_description)/meshes/omx1_link4.stl" scale="0.001 0.001 0.001"/>
       </geometry>
     </collision>
@@ -163,12 +163,12 @@
       <origin xyz="0 0 0" rpy="0 0 ${M_PI/2}"/>
       <geometry>
-        <mesh filename="file://$(find open_manipulator_x_description)/meshes/omx1_link5.stl" scale="0.001 0.001 0.001"/>
-      </geometry>
-      <material name="grey"/>
-    </visual>
-    <collision>
-      <origin xyz="0 0 0" rpy="0 0 ${M_PI/2}"/>
-      <geometry>
-        <mesh filename="file://$(find open_manipulator_x_description)/meshes/omx1_link5.stl" scale="0.001 0.001 0.001"/>
+        <mesh filename="file://$(find sobit_light_description)/meshes/omx1_link5.stl" scale="0.001 0.001 0.001"/>
+      </geometry>
+      <material name="grey"/>
+    </visual>
+    <collision>
+      <origin xyz="0 0 0" rpy="0 0 ${M_PI/2}"/>
+      <geometry>
+        <mesh filename="file://$(find sobit_light_description)/meshes/omx1_link5.stl" scale="0.001 0.001 0.001"/>
       </geometry>
     </collision>
@@ -194,12 +194,12 @@
       <origin xyz="0 0 0" rpy="0 0 ${M_PI/2}"/>
       <geometry>
-        <mesh filename="file://$(find open_manipulator_x_description)/meshes/omx1_link6.stl" scale="0.001 0.001 0.001"/>
-      </geometry>
-      <material name="grey"/>
-    </visual>
-    <collision>
-      <origin xyz="0 0 0" rpy="0 0 ${M_PI/2}"/>
-      <geometry>
-        <mesh filename="file://$(find open_manipulator_x_description)/meshes/omx1_link6.stl" scale="0.001 0.001 0.001"/>
+        <mesh filename="file://$(find sobit_light_description)/meshes/omx1_link6.stl" scale="0.001 0.001 0.001"/>
+      </geometry>
+      <material name="grey"/>
+    </visual>
+    <collision>
+      <origin xyz="0 0 0" rpy="0 0 ${M_PI/2}"/>
+      <geometry>
+        <mesh filename="file://$(find sobit_light_description)/meshes/omx1_link6.stl" scale="0.001 0.001 0.001"/>
       </geometry>
     </collision>
@@ -225,12 +225,12 @@
       <origin xyz="0 0 0" rpy="0 0 ${M_PI/2}"/>
       <geometry>
-        <mesh filename="file://$(find open_manipulator_x_description)/meshes/omx1_link7_gripper_base.stl" scale="0.001 0.001 0.001"/>
-      </geometry>
-      <material name="grey"/>
-    </visual>
-    <collision>
-      <origin xyz="0 0 0" rpy="0 0 ${M_PI/2}"/>
-      <geometry>
-        <mesh filename="file://$(find open_manipulator_x_description)/meshes/omx1_link7_gripper_base.stl" scale="0.001 0.001 0.001"/>
+        <mesh filename="file://$(find sobit_light_description)/meshes/omx1_link7_gripper_base.stl" scale="0.001 0.001 0.001"/>
+      </geometry>
+      <material name="grey"/>
+    </visual>
+    <collision>
+      <origin xyz="0 0 0" rpy="0 0 ${M_PI/2}"/>
+      <geometry>
+        <mesh filename="file://$(find sobit_light_description)/meshes/omx1_link7_gripper_base.stl" scale="0.001 0.001 0.001"/>
       </geometry>
     </collision>
@@ -254,12 +254,12 @@
       <origin xyz="0 0 0" rpy="0 0 ${M_PI/2}"/>
       <geometry>
-        <mesh filename="file://$(find open_manipulator_x_description)/meshes/omx1_link8_gripper.stl" scale="0.001 0.001 0.001"/>
-      </geometry>
-      <material name="grey"/>
-    </visual>
-    <collision>
-      <origin xyz="0 0 0" rpy="0 0 ${M_PI/2}"/>
-      <geometry>
-        <mesh filename="file://$(find open_manipulator_x_description)/meshes/omx1_link8_gripper.stl" scale="0.001 0.001 0.001"/>
+        <mesh filename="file://$(find sobit_light_description)/meshes/omx1_link8_gripper.stl" scale="0.001 0.001 0.001"/>
+      </geometry>
+      <material name="grey"/>
+    </visual>
+    <collision>
+      <origin xyz="0 0 0" rpy="0 0 ${M_PI/2}"/>
+      <geometry>
+        <mesh filename="file://$(find sobit_light_description)/meshes/omx1_link8_gripper.stl" scale="0.001 0.001 0.001"/>
       </geometry>
     </collision>
@@ -283,12 +283,12 @@
       <origin xyz="0 0 0" rpy="0 0 ${M_PI/2}"/>
       <geometry>
-        <mesh filename="file://$(find open_manipulator_x_description)/meshes/omx1_link9-10_gripper.stl" scale="0.001 0.001 0.001"/>
-      </geometry>
-      <material name="grey"/>
-    </visual>
-    <collision>
-      <origin xyz="0 0 0" rpy="0 0 ${M_PI/2}"/>
-      <geometry>
-        <mesh filename="file://$(find open_manipulator_x_description)/meshes/omx1_link9-10_gripper.stl" scale="0.001 0.001 0.001"/>
+        <mesh filename="file://$(find sobit_light_description)/meshes/omx1_link9-10_gripper.stl" scale="0.001 0.001 0.001"/>
+      </geometry>
+      <material name="grey"/>
+    </visual>
+    <collision>
+      <origin xyz="0 0 0" rpy="0 0 ${M_PI/2}"/>
+      <geometry>
+        <mesh filename="file://$(find sobit_light_description)/meshes/omx1_link9-10_gripper.stl" scale="0.001 0.001 0.001"/>
       </geometry>
     </collision>
@@ -312,5 +312,5 @@
       <origin xyz="0 0 0" rpy="0 ${M_PI} ${M_PI/2}"/>
       <geometry>
-        <mesh filename="file://$(find open_manipulator_x_description)/meshes/omx1_link9-10_gripper.stl" scale="0.001 0.001 0.001"/>
+        <mesh filename="file://$(find sobit_light_description)/meshes/omx1_link9-10_gripper.stl" scale="0.001 0.001 0.001"/>
       </geometry>
       <material name="grey"/>
@@ -319,5 +319,5 @@
       <origin xyz="0 0 0" rpy="0 ${M_PI} ${M_PI/2}"/>
       <geometry>
-        <mesh filename="file://$(find open_manipulator_x_description)/meshes/omx1_link9-10_gripper.stl" scale="0.001 0.001 0.001"/>
+        <mesh filename="file://$(find sobit_light_description)/meshes/omx1_link9-10_gripper.stl" scale="0.001 0.001 0.001"/>
       </geometry>
     </collision>
@@ -343,5 +343,5 @@
       <origin xyz="0.0 0.0 0" rpy="0 0 ${M_PI/2}"/>
       <geometry>
-        <mesh filename="file://$(find open_manipulator_x_description)/meshes/omx1_link11-12_finger.stl" scale="0.001 0.001 0.001"/>
+        <mesh filename="file://$(find sobit_light_description)/meshes/omx1_link11-12_finger.stl" scale="0.001 0.001 0.001"/>
       </geometry>
       <material name="grey"/>
@@ -350,5 +350,5 @@
       <origin xyz="0.0 0.0 0" rpy="0 0 ${M_PI/2}"/>
       <geometry>
-        <mesh filename="file://$(find open_manipulator_x_description)/meshes/omx1_link11-12_finger.stl" scale="0.001 0.001 0.001"/>
+        <mesh filename="file://$(find sobit_light_description)/meshes/omx1_link11-12_finger.stl" scale="0.001 0.001 0.001"/>
       </geometry>
     </collision>
@@ -375,12 +375,12 @@
       <origin xyz="0.0 -0.0 0" rpy="0 ${M_PI} ${M_PI/2}"/>
       <geometry>
-        <mesh filename="file://$(find open_manipulator_x_description)/meshes/omx1_link11-12_finger.stl" scale="0.001 0.001 0.001"/>
-      </geometry>
-      <material name="grey"/>
-    </visual>
-    <collision>
-      <origin xyz="0.0 -0.0 0" rpy="0 ${M_PI} ${M_PI/2}"/>
-      <geometry>
-        <mesh filename="file://$(find open_manipulator_x_description)/meshes/omx1_link11-12_finger.stl" scale="0.001 0.001 0.001"/>
+        <mesh filename="file://$(find sobit_light_description)/meshes/omx1_link11-12_finger.stl" scale="0.001 0.001 0.001"/>
+      </geometry>
+      <material name="grey"/>
+    </visual>
+    <collision>
+      <origin xyz="0.0 -0.0 0" rpy="0 ${M_PI} ${M_PI/2}"/>
+      <geometry>
+        <mesh filename="file://$(find sobit_light_description)/meshes/omx1_link11-12_finger.stl" scale="0.001 0.001 0.001"/>
       </geometry>
     </collision>
@@ -404,5 +404,5 @@
       <origin xyz="0.0 -0.0 0" rpy="0 0 ${M_PI/2}"/>
       <geometry>
-        <mesh filename="file://$(find open_manipulator_x_description)/meshes/omx1_link13-14_finger.stl" scale="0.001 0.001 0.001"/>
+        <mesh filename="file://$(find sobit_light_description)/meshes/omx1_link13-14_finger.stl" scale="0.001 0.001 0.001"/>
       </geometry>
       <material name="grey"/>
@@ -411,5 +411,5 @@
       <origin xyz="0.0 -0.0 0" rpy="0 0 ${M_PI/2}"/>
       <geometry>
-        <mesh filename="file://$(find open_manipulator_x_description)/meshes/omx1_link13-14_finger.stl" scale="0.001 0.001 0.001"/>
+        <mesh filename="file://$(find sobit_light_description)/meshes/omx1_link13-14_finger.stl" scale="0.001 0.001 0.001"/>
       </geometry>
     </collision>
@@ -433,12 +433,12 @@
       <origin xyz="0.0 -0.0 0" rpy="0 ${M_PI} ${M_PI/2}"/>
       <geometry>
-        <mesh filename="file://$(find open_manipulator_x_description)/meshes/omx1_link13-14_finger.stl" scale="0.001 0.001 0.001"/>
-      </geometry>
-      <material name="grey"/>
-    </visual>
-    <collision>
-      <origin xyz="0.0 -0.0 0" rpy="0 ${M_PI} ${M_PI/2}"/>
-      <geometry>
-        <mesh filename="file://$(find open_manipulator_x_description)/meshes/omx1_link13-14_finger.stl" scale="0.001 0.001 0.001"/>
+        <mesh filename="file://$(find sobit_light_description)/meshes/omx1_link13-14_finger.stl" scale="0.001 0.001 0.001"/>
+      </geometry>
+      <material name="grey"/>
+    </visual>
+    <collision>
+      <origin xyz="0.0 -0.0 0" rpy="0 ${M_PI} ${M_PI/2}"/>
+      <geometry>
+        <mesh filename="file://$(find sobit_light_description)/meshes/omx1_link13-14_finger.stl" scale="0.001 0.001 0.001"/>
       </geometry>
     </collision>

File: sobit_light_description/urdf/common.xacro (robot description, xacro)
@@ -3,5 +3,5 @@
 <robot name="sobit_light"
        xmlns:xacro="http://ros.org/wiki/xacro">
-  <xacro:property name="M_PI" value="3.14159265359" />
+  <xacro:property name="PI" value="3.14159265359" />
   <!-- Transmission macro: Position -->
   <xacro:macro name="SimpleTransmissionPosition" params="joint reduction">

File: sobit_light_description/urdf/materials.xacro (robot description, xacro)
@@ -21,3 +21,12 @@
     <color rgba="0.5 0.5 0.5 1.0"/>
   </material>
+  <material name="body">
+    <color rgba="0.2175 0.2355 0.246 1.0" />
+  </material>
+  <material name="tire">
+    <color rgba="0.3 0.3 0.3 1.0" />
+  </material>
+  <material name="black">
+    <color rgba="0.0 0.0 0.0 1.0" />
+  </material>
 </robot>
