Commit message: [UPD] make macro file

File: sobit_light_description/urdf/arm/open_manipulator_x.transmission.xacro (robot description, xacro)
@@ -1,45 +1,12 @@
-<?xml version="1.0"?>
+<?xml version="1.0" encoding="UTF-8" ?>
 <!-- OpenManipulator X1000 (ROS Control: Transmission) -->
-<robot name="open_manipulator_x1000"
-       xmlns:xacro="http://ros.org/wiki/xacro">
-  <!-- Transmission macro -->
-  <xacro:macro name="SimpleTransmissionPosition" params="name">
-    <transmission name="${name}_tran">
-      <type>transmission_interface/SimpleTransmission</type>
-      <joint name="${name}_joint">
-        <hardwareInterface>hardware_interface/PositionJointInterface</hardwareInterface>
-      </joint>
-      <actuator name="${name}_act">
-        <mechanicalReduction>1</mechanicalReduction>
-      </actuator>
-    </transmission>
+<robot name="arm_transmission" xmlns:xacro="http://ros.org/wiki/xacro">
+  <xacro:macro name="arm_transmission" params="prefix">
+    <position_joint_transmission joint="${prefix}_arm1" reduction="1" />
+    <position_joint_transmission joint="${prefix}_arm2" reduction="1" />
+    <position_joint_transmission joint="${prefix}_arm3" reduction="1" />
+    <position_joint_transmission joint="${prefix}_arm4" reduction="1" />
+    <position_joint_transmission joint="${prefix}_arm5" reduction="1" />
+    <position_joint_transmission joint="${prefix}_arm6" reduction="1" />
   </xacro:macro>
-  <!-- Transmission macro -->
-  <xacro:macro name="SimpleTransmissionEffort" params="name">
-    <transmission name="${name}_tran">
-      <type>transmission_interface/SimpleTransmission</type>
-      <joint name="${name}_joint">
-        <hardwareInterface>hardware_interface/EffortJointInterface</hardwareInterface>
-      </joint>
-      <actuator name="${name}_act">
-        <mechanicalReduction>1</mechanicalReduction>
-      </actuator>
-    </transmission>
-  </xacro:macro>
-  <!-- Transmission 1: Shoulder -->
-  <xacro:SimpleTransmissionPosition name="omx1_arm1" />
-  <!-- Transmission 2: Upper Arm -->
-  <xacro:SimpleTransmissionPosition name="omx1_arm2" />
-  <!-- Transmission 3: Lower Arm -->
-  <xacro:SimpleTransmissionPosition name="omx1_arm3" />
-  <!-- Transmission 4: Forearm Upper -->
-  <xacro:SimpleTransmissionPosition name="omx1_arm4" />
-  <!-- Transmission 5: Forearm Lower -->
-  <xacro:SimpleTransmissionPosition name="omx1_arm5" />
-  <!-- Transmission 6: Wrist (Gripper Base) -->
-  <xacro:SimpleTransmissionPosition name="omx1_arm6" />
-  <!-- Transmission 7: Gripper Finger Left -->
-  <xacro:SimpleTransmissionEffort name="omx1_gripper_l_finger" />
-  <!-- Transmission 8: Gripper Finger Right -->
-  <xacro:SimpleTransmissionEffort name="omx1_gripper_r_finger" />
 </robot>

File: sobit_light_description/urdf/arm/open_manipulator_x.urdf.xacro (robot description, xacro)
@@ -1,484 +1,282 @@
-<?xml version="1.0"?>
+<?xml version="1.0" encoding="UTF-8" ?>
 <!-- OpenManipulator X1000 (Arm) -->
-<robot name="open_manipulator_x1000"
-       xmlns:xacro="http://ros.org/wiki/xacro">
-  <!-- Link 0: Platform -->
-  <link name="omx1_platform_link">
-    <visual>
-      <origin xyz="0 0 0" rpy="0 0 ${M_PI/2}"/>
-      <geometry>
-        <mesh filename="file://$(find sobit_light_description)/meshes/omx1_link_base.stl" scale="0.001 0.001 0.001"/>
-      </geometry>
-      <material name="grey"/>
-    </visual>
-    <!-- TODO: Collision with simple geometry -->
-    <collision>
-      <origin xyz="0 0 0" rpy="0 0 ${M_PI/2}"/>
-      <geometry>
-        <mesh filename="file://$(find sobit_light_description)/meshes/omx1_link_base.stl" scale="0.001 0.001 0.001"/>
-      </geometry>
-    </collision>
-    <!-- TODO: Inertial with simple geometry -->
-    <inertial>
-      <origin xyz="0 0 0" rpy="0 0 ${M_PI/2}"/>
-      <mass value="0.2" />
-      <inertia ixx="1.0" ixy="0.0" ixz="1.0"
-               iyy="1.0" iyz="0.0"
-               izz="1.0" />
-    </inertial>
-  </link>
-  <!-- Joint 1: Base -->
-  <joint name="omx1_base_joint" type="fixed">
-    <parent link="omx1_platform_link"/>
-    <child link="omx1_base_link"/>
-    <origin xyz="-0.0105 -0.0135 0.006" rpy="0 0 0"/>
-  </joint>
-  <!-- Link 1: Base -->
-  <link name="omx1_base_link">
-    <visual>
-      <origin xyz="0 0 0" rpy="0 0 ${M_PI/2}"/>
-      <geometry>
-        <mesh filename="file://$(find sobit_light_description)/meshes/omx1_link1.stl" scale="0.001 0.001 0.001"/>
-      </geometry>
-      <material name="grey"/>
-    </visual>
-    <collision>
-      <origin xyz="0 0 0" rpy="0 0 ${M_PI/2}"/>
-      <geometry>
-        <mesh filename="file://$(find sobit_light_description)/meshes/omx1_link1.stl" scale="0.001 0.001 0.001"/>
-      </geometry>
-    </collision>
-    <inertial>
-      <origin xyz="0 0 0" rpy="0 0 ${M_PI/2}"/>
-      <mass value="0.2" />
-      <inertia ixx="1.0" ixy="0.0" ixz="1.0"
-               iyy="1.0" iyz="0.0"
-               izz="1.0" />
-    </inertial>
-  </link>
-  <!-- Joint 2: Shoulder -->
-  <joint name="omx1_arm1_joint" type="revolute">
-    <parent link="omx1_base_link"/>
-    <child link="omx1_arm1_link"/>
-    <origin xyz="0.0 0.0 0.0465" rpy="0 0 0"/>
-    <axis xyz="0 0 1"/>
-    <limit velocity="4.8" effort="1" lower="${-M_PI}" upper="${M_PI}" />
-  </joint>
-  <!--  Link 2: Shoulder -->
-  <link name="omx1_arm1_link">
-    <visual>
-      <origin xyz="0 0 0.0" rpy="0 0 ${M_PI/2}"/>
-      <geometry>
-        <mesh filename="file://$(find sobit_light_description)/meshes/omx1_link2.stl" scale="0.001 0.001 0.001"/>
-      </geometry>
-      <material name="grey"/>
-    </visual>
-    <collision>
-      <origin xyz="0 0 0.0" rpy="0 0 ${M_PI/2}"/>
-      <geometry>
-        <mesh filename="file://$(find sobit_light_description)/meshes/omx1_link2.stl" scale="0.001 0.001 0.001"/>
-      </geometry>
-    </collision>
-    <inertial>
-      <origin xyz="0 0 0.0" rpy="0 0 ${M_PI/2}"/>
-      <mass value="0.2" />
-      <inertia ixx="1.0" ixy="0.0" ixz="1.0"
-               iyy="1.0" iyz="0.0"
-               izz="1.0" />
-    </inertial>
-  </link>
-  <!--  Joint 3: Upper Arm -->
-  <joint name="omx1_arm2_joint" type="revolute">
-    <parent link="omx1_arm1_link"/>
-    <child link="omx1_arm2_link"/>
-    <origin xyz="0.0 0.0 0.05095" rpy="0 0 0"/>
-    <axis xyz="0 1 0"/>
-    <limit velocity="4.8" effort="1" lower="${-M_PI/2}" upper="${M_PI/2}" />
-  </joint>
-  <!--  Link 3: Upper Arm -->
-  <link name="omx1_arm2_link">
-    <visual>
-      <origin xyz="0 0 0" rpy="0 0 ${M_PI/2}"/>
-      <geometry>
-        <mesh filename="file://$(find sobit_light_description)/meshes/omx1_link3.stl" scale="0.001 0.001 0.001"/>
-      </geometry>
-      <material name="grey"/>
-    </visual>
-    <collision>
-      <origin xyz="0 0 0" rpy="0 0 ${M_PI/2}"/>
-      <geometry>
-        <mesh filename="file://$(find sobit_light_description)/meshes/omx1_link3.stl" scale="0.001 0.001 0.001"/>
-      </geometry>
-    </collision>
-    <inertial>
-      <origin xyz="0 0 0" rpy="0 0 ${M_PI/2}"/>
-      <mass value="0.2" />
-      <inertia ixx="1.0" ixy="0.0" ixz="1.0"
-               iyy="1.0" iyz="0.0"
-               izz="1.0" />
-    </inertial>
-  </link>
-  <!--  Joint 4: Lower Arm -->
-  <joint name="omx1_arm3_joint" type="revolute">
-    <parent link="omx1_arm2_link"/>
-    <child link="omx1_arm3_link"/>
-    <origin xyz="0.022 -0.0 0.128" rpy="0 0 0"/>
-    <axis xyz="0 1 0"/>
-    <limit velocity="4.8" effort="1" lower="${-M_PI/2}" upper="${M_PI/2}" />
-  </joint>
-  <!--  Link 4: Lower Arm -->
-  <link name="omx1_arm3_link">
-    <visual>
-      <origin xyz="0 0 0" rpy="0 0 ${M_PI/2}"/>
-      <geometry>
-        <mesh filename="file://$(find sobit_light_description)/meshes/omx1_link4.stl" scale="0.001 0.001 0.001"/>
-      </geometry>
-      <material name="grey"/>
-    </visual>
-    <collision>
-      <origin xyz="0 0 0" rpy="0 0 ${M_PI/2}"/>
-      <geometry>
-        <mesh filename="file://$(find sobit_light_description)/meshes/omx1_link4.stl" scale="0.001 0.001 0.001"/>
-      </geometry>
-    </collision>
-    <inertial>
-      <origin xyz="0 0 0" rpy="0 0 ${M_PI/2}"/>
-      <mass value="0.2" />
-      <inertia ixx="1.0" ixy="0.0" ixz="1.0"
-               iyy="1.0" iyz="0.0"
-               izz="1.0" />
-    </inertial>
-  </link>
-  <!--  Joint 5: Forearm Upper -->
-  <joint name="omx1_arm4_joint" type="revolute">
-    <parent link="omx1_arm3_link"/>
-    <child link="omx1_arm4_link"/>
-    <origin xyz="0.0835 0.0 0.0" rpy="0 0 0"/>
-    <axis xyz="1 0 0"/>
-    <limit velocity="4.8" effort="1" lower="${-M_PI}" upper="${M_PI}" />
-  </joint>
-  <!--  Link 5: Forearm Upper -->
-  <link name="omx1_arm4_link">
-    <visual>
-      <origin xyz="0 0 0" rpy="0 0 ${M_PI/2}"/>
-      <geometry>
-        <mesh filename="file://$(find sobit_light_description)/meshes/omx1_link5.stl" scale="0.001 0.001 0.001"/>
-      </geometry>
-      <material name="grey"/>
-    </visual>
-    <collision>
-      <origin xyz="0 0 0" rpy="0 0 ${M_PI/2}"/>
-      <geometry>
-        <mesh filename="file://$(find sobit_light_description)/meshes/omx1_link5.stl" scale="0.001 0.001 0.001"/>
-      </geometry>
-    </collision>
-    <inertial>
-      <origin xyz="0 0 0" rpy="0 0 ${M_PI/2}"/>
-      <mass value="0.2" />
-      <inertia ixx="1.0" ixy="0.0" ixz="1.0"
-               iyy="1.0" iyz="0.0"
-               izz="1.0" />
-    </inertial>
-  </link>
-  <!--  Joint 6: Forearm Lower -->
-  <joint name="omx1_arm5_joint" type="revolute">
-    <parent link="omx1_arm4_link"/>
-    <child link="omx1_arm5_link"/>
-    <origin xyz="0.0405 0.0 0.0" rpy="0 0 0"/>
-    <axis xyz="0 1 0"/>
-    <limit velocity="4.8" effort="1" lower="${-M_PI/2}" upper="${M_PI/2}" />
-  </joint>
-  <!--  Link 6: Forearm Lower -->
-  <link name="omx1_arm5_link">
-    <visual>
-      <origin xyz="0 0 0" rpy="0 0 ${M_PI/2}"/>
-      <geometry>
-        <mesh filename="file://$(find sobit_light_description)/meshes/omx1_link6.stl" scale="0.001 0.001 0.001"/>
-      </geometry>
-      <material name="grey"/>
-    </visual>
-    <collision>
-      <origin xyz="0 0 0" rpy="0 0 ${M_PI/2}"/>
-      <geometry>
-        <mesh filename="file://$(find sobit_light_description)/meshes/omx1_link6.stl" scale="0.001 0.001 0.001"/>
-      </geometry>
-    </collision>
-    <inertial>
-      <origin xyz="0 0 0" rpy="0 0 ${M_PI/2}"/>
-      <mass value="0.2" />
-      <inertia ixx="1.0" ixy="0.0" ixz="1.0"
-               iyy="1.0" iyz="0.0"
-               izz="1.0" />
-    </inertial>
-  </link>
-  <!--  Joint 7: Wrist (Gripper Base) -->
-  <joint name="omx1_arm6_joint" type="revolute">
-    <parent link="omx1_arm5_link"/>
-    <child link="omx1_arm6_link"/>
-    <origin xyz="0.064 0 0.0" rpy="0 0 0"/>
-    <axis xyz="1 0 0"/>
-    <limit velocity="4.8" effort="1" lower="${-M_PI}" upper="${M_PI}" />
-  </joint>
-  <!--  Link 7: Wrist (Gripper Base) -->
-  <link name="omx1_arm6_link">
-    <visual>
-      <origin xyz="0 0 0" rpy="0 0 ${M_PI/2}"/>
-      <geometry>
-        <mesh filename="file://$(find sobit_light_description)/meshes/omx1_link7_gripper_base.stl" scale="0.001 0.001 0.001"/>
-      </geometry>
-      <material name="grey"/>
-    </visual>
-    <collision>
-      <origin xyz="0 0 0" rpy="0 0 ${M_PI/2}"/>
-      <geometry>
-        <mesh filename="file://$(find sobit_light_description)/meshes/omx1_link7_gripper_base.stl" scale="0.001 0.001 0.001"/>
-      </geometry>
-    </collision>
-    <inertial>
-      <origin xyz="0 0 0" rpy="0 0 ${M_PI/2}"/>
-      <mass value="0.2" />
-      <inertia ixx="1.0" ixy="0.0" ixz="1.0"
-               iyy="1.0" iyz="0.0"
-               izz="1.0" />
-    </inertial>
-  </link>
-  <!--  Joint 8: Gripper -->
-  <joint name="omx1_gripper_joint" type="fixed">
-    <parent link="omx1_arm6_link"/>
-    <child link="omx1_gripper_link"/>
-    <origin xyz="0.05 0.0 0.0" rpy="0 0 0"/>
-  </joint>
-  <!--  Link 8: Gripper -->
-  <link name="omx1_gripper_link">
-    <visual>
-      <origin xyz="0 0 0" rpy="0 0 ${M_PI/2}"/>
-      <geometry>
-        <mesh filename="file://$(find sobit_light_description)/meshes/omx1_link8_gripper.stl" scale="0.001 0.001 0.001"/>
-      </geometry>
-      <material name="grey"/>
-    </visual>
-    <collision>
-      <origin xyz="0 0 0" rpy="0 0 ${M_PI/2}"/>
-      <geometry>
-        <mesh filename="file://$(find sobit_light_description)/meshes/omx1_link8_gripper.stl" scale="0.001 0.001 0.001"/>
-      </geometry>
-    </collision>
-    <inertial>
-      <origin xyz="0 0 0" rpy="0 0 ${M_PI/2}"/>
-      <mass value="0.2" />
-      <inertia ixx="1.0" ixy="0.0" ixz="1.0"
-               iyy="1.0" iyz="0.0"
-               izz="1.0" />
-    </inertial>
-  </link>
-  <!--  Joint 9: Gripper left sub -->
-  <joint name="omx1_gripper_l_sub_joint" type="fixed">
-    <parent link="omx1_gripper_link"/>
-    <child link="omx1_gripper_l_sub_link"/>
-    <origin xyz="0.009 0.015 0.0" rpy="0 0 0"/>
-  </joint>
-  <!--  Link 9: Gripper left sub -->
-  <link name="omx1_gripper_l_sub_link">
-    <visual>
-      <origin xyz="0 0 0" rpy="0 0 ${M_PI/2}"/>
-      <geometry>
-        <mesh filename="file://$(find sobit_light_description)/meshes/omx1_link9-10_gripper.stl" scale="0.001 0.001 0.001"/>
-      </geometry>
-      <material name="grey"/>
-    </visual>
-    <collision>
-      <origin xyz="0 0 0" rpy="0 0 ${M_PI/2}"/>
-      <geometry>
-        <mesh filename="file://$(find sobit_light_description)/meshes/omx1_link9-10_gripper.stl" scale="0.001 0.001 0.001"/>
-      </geometry>
-    </collision>
-    <inertial>
-      <origin xyz="0 0 0" rpy="0 0 ${M_PI/2}"/>
-      <mass value="0.2" />
-      <inertia ixx="1.0" ixy="0.0" ixz="1.0"
-               iyy="1.0" iyz="0.0"
-               izz="1.0" />
-    </inertial>
-  </link>
-  <!--  Joint 10: Gripper right sub -->
-  <joint name="omx1_gripper_r_sub_joint" type="fixed">
-    <parent link="omx1_gripper_link"/>
-    <child link="omx1_gripper_r_sub_link"/>
-    <origin xyz="0.009 -0.015 0.0" rpy="0 0 0"/>
-  </joint>
-  <!--  Link 10: Gripper right sub -->
-  <link name="omx1_gripper_r_sub_link">
-    <visual>
-      <origin xyz="0 0 0" rpy="0 ${M_PI} ${M_PI/2}"/>
-      <geometry>
-        <mesh filename="file://$(find sobit_light_description)/meshes/omx1_link9-10_gripper.stl" scale="0.001 0.001 0.001"/>
-      </geometry>
-      <material name="grey"/>
-    </visual>
-    <collision>
-      <origin xyz="0 0 0" rpy="0 ${M_PI} ${M_PI/2}"/>
-      <geometry>
-        <mesh filename="file://$(find sobit_light_description)/meshes/omx1_link9-10_gripper.stl" scale="0.001 0.001 0.001"/>
-      </geometry>
-    </collision>
-    <inertial>
-      <origin xyz="0 0 0" rpy="0 ${M_PI} ${M_PI/2}"/>
-      <mass value="0.2" />
-      <inertia ixx="1.0" ixy="0.0" ixz="1.0"
-               iyy="1.0" iyz="0.0"
-               izz="1.0" />
-    </inertial>
-  </link>
-  <!--  Joint 11: Gripper Finger Left -->
-  <joint name="omx1_gripper_l_finger_joint" type="prismatic">
-    <parent link="omx1_gripper_l_sub_link"/>
-    <child link="omx1_gripper_l_finger_link"/>
-    <origin xyz="0.0 0.04 0.0" rpy="0 0 0"/>
-    <axis xyz="0 1 0"/>
-    <limit velocity="4.8" effort="1" lower="${-0.055+0.02675}" upper="0.0" />
-  </joint>
-  <!--  Link 11: Gripper Finger Left -->
-  <link name="omx1_gripper_l_finger_link">
-    <visual>
-      <origin xyz="0.0 0.0 0" rpy="0 0 ${M_PI/2}"/>
-      <geometry>
-        <mesh filename="file://$(find sobit_light_description)/meshes/omx1_link11-12_finger.stl" scale="0.001 0.001 0.001"/>
-      </geometry>
-      <material name="grey"/>
-    </visual>
-    <collision>
-      <origin xyz="0.0 0.0 0" rpy="0 0 ${M_PI/2}"/>
-      <geometry>
-        <mesh filename="file://$(find sobit_light_description)/meshes/omx1_link11-12_finger.stl" scale="0.001 0.001 0.001"/>
-      </geometry>
-    </collision>
-    <inertial>
-      <origin xyz="0.0 0.0 0" rpy="0 0 ${M_PI/2}"/>
-      <mass value="0.2" />
-      <inertia ixx="1.0" ixy="0.0" ixz="1.0"
-               iyy="1.0" iyz="0.0"
-               izz="1.0" />
-    </inertial>
-  </link>
-  <!--  Joint 12: Gripper Finger Right -->
-  <joint name="omx1_gripper_r_finger_joint" type="prismatic">
-    <parent link="omx1_gripper_r_sub_link"/>
-    <child link="omx1_gripper_r_finger_link"/>
-    <origin xyz="0.0 -0.04 0.0" rpy="0 0 0"/>
-    <axis xyz="0 -1 0"/>
-    <limit velocity="4.8" effort="1" lower="0.0" upper="${-0.055+0.02675}" />
-    <mimic joint="omx1_gripper_l_finger_joint" multiplier="1"/>
-  </joint>
-  <!--  Link 12: Gripper Finger Right -->
-  <link name="omx1_gripper_r_finger_link">
-    <visual>
-      <origin xyz="0.0 -0.0 0" rpy="0 ${M_PI} ${M_PI/2}"/>
-      <geometry>
-        <mesh filename="file://$(find sobit_light_description)/meshes/omx1_link11-12_finger.stl" scale="0.001 0.001 0.001"/>
-      </geometry>
-      <material name="grey"/>
-    </visual>
-    <collision>
-      <origin xyz="0.0 -0.0 0" rpy="0 ${M_PI} ${M_PI/2}"/>
-      <geometry>
-        <mesh filename="file://$(find sobit_light_description)/meshes/omx1_link11-12_finger.stl" scale="0.001 0.001 0.001"/>
-      </geometry>
-    </collision>
-    <inertial>
-      <origin xyz="0.0 -0.0 0" rpy="0 ${M_PI} ${M_PI/2}"/>
-      <mass value="0.2" />
-      <inertia ixx="1.0" ixy="0.0" ixz="1.0"
-               iyy="1.0" iyz="0.0"
-               izz="1.0" />
-    </inertial>
-  </link>
-  <!--  Joint 13: Gripper Tip Left -->
-  <joint name="omx1_gripper_l_tip_joint" type="fixed">
-    <parent link="omx1_gripper_l_finger_link"/>
-    <child link="omx1_gripper_l_tip_link"/>
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