Commit message: [UPD] add parallel actuator as arm_2_sub

File: sobit_light_description/urdf/arm/arm.transmission.xacro (robot description, xacro)
@@ -5,4 +5,5 @@
     <position_joint_transmission joint="${prefix}_1_joint" reduction="1" />
     <position_joint_transmission joint="${prefix}_2_joint" reduction="1" />
+    <position_joint_transmission joint="${prefix}_2_sub_joint" reduction="1" />
     <position_joint_transmission joint="${prefix}_3_joint" reduction="1" />
     <position_joint_transmission joint="${prefix}_4_joint" reduction="1" />

File: sobit_light_description/urdf/arm/arm.urdf.xacro (robot description, xacro)
@@ -124,4 +124,36 @@
       </inertial>
     </link>
+    <!--  Joint 3: Upper Arm (SUB) -->
+    <joint name="${prefix}_2_sub_joint" type="revolute">
+      <parent link="${prefix}_1_link"/>
+      <child link="${prefix}_2_sub_link"/>
+      <origin xyz="0.0 0.0 0.05095" rpy="0 0 0"/>
+      <axis xyz="0 1 0"/>
+      <limit velocity="4.8" effort="1" lower="${-M_PI/2}" upper="${M_PI/2}" />
+      <mimic joint="${prefix}_2_joint" multiplier="-1" offset="0"/>
+    </joint>
+    <!--  Link 3: Upper Arm (SUB) -->
+    <link name="${prefix}_2_sub_link">
+      <!-- <visual>
+        <origin xyz="0 0 0" rpy="0 0 ${M_PI/2}"/>
+        <geometry>
+          <mesh filename="file://$(find sobit_light_description)/meshes/arm/omx1_link3.stl" scale="0.001 0.001 0.001"/>
+        </geometry>
+        <material name="grey"/>
+      </visual>
+      <collision>
+        <origin xyz="${0.03575-0.0585/2} 0.0 ${-0.016+(0.14475+0.016)/2}" rpy="0 0 0"/>
+        <geometry>
+          <box size="0.0585 0.0440 ${0.14475+0.016}"/>
+        </geometry>
+      </collision>
+      <inertial>
+        <origin xyz="${0.03575-0.0585/2} 0.0 ${-0.016+(0.14475+0.016)/2}" rpy="0 0 0"/>
+        <mass value="0.261" />
+        <inertia  ixx="${1/12*0.261*(0.0585**2+(0.14475+0.016)**2)}" ixy="0.0" ixz="0.0"
+                  iyy="${1/12*0.261*(0.0440**2+(0.14475+0.016)**2)}" iyz="0.0"
+                  izz="${1/12*0.261*(0.0585**2+0.0440**2)}" />
+      </inertial> -->
+    </link>
     <!--  Joint 4: Lower Arm -->
     <joint name="${prefix}_3_joint" type="revolute">

Commit message: [UPD] naming based on motion

File: sobit_light_description/urdf/arm/arm.transmission.xacro (robot description, xacro)
@@ -3,11 +3,11 @@
 <robot name="arm_transmission" xmlns:xacro="http://ros.org/wiki/xacro">
   <xacro:macro name="arm_transmission" params="prefix">
-    <position_joint_transmission joint="${prefix}_1_joint" reduction="1" />
-    <position_joint_transmission joint="${prefix}_2_joint" reduction="1" />
-    <position_joint_transmission joint="${prefix}_2_sub_joint" reduction="1" />
-    <position_joint_transmission joint="${prefix}_3_joint" reduction="1" />
-    <position_joint_transmission joint="${prefix}_4_joint" reduction="1" />
-    <position_joint_transmission joint="${prefix}_5_joint" reduction="1" />
-    <position_joint_transmission joint="${prefix}_6_joint" reduction="1" />
+    <position_joint_transmission joint="${prefix}_shoulder_roll_joint" reduction="1" />
+    <position_joint_transmission joint="${prefix}_shoulder_pitch_joint" reduction="1" />
+    <position_joint_transmission joint="${prefix}_shoulder_pitch_sub_joint" reduction="1" />
+    <position_joint_transmission joint="${prefix}_elbow_pitch_joint" reduction="1" />
+    <position_joint_transmission joint="${prefix}_forearm_roll_joint" reduction="1" />
+    <position_joint_transmission joint="${prefix}_wrist_pitch_joint" reduction="1" />
+    <position_joint_transmission joint="${prefix}_wrist_roll_joint" reduction="1" />
   </xacro:macro>
 </robot>

File: sobit_light_description/urdf/arm/arm.urdf.xacro (robot description, xacro)
@@ -4,5 +4,5 @@
   <xacro:include filename="$(find sobit_light_description)/urdf/arm/arm.transmission.xacro" />
   <xacro:macro name="arm" params="prefix parent">
-    <!-- Joint 0: Platform -->
+    <!-- Joint: Platform -->
     <joint name="${prefix}_platform_joint" type="fixed">
       <parent link="${parent}"/>
@@ -10,5 +10,5 @@
       <origin xyz="0.122 0.0 0.0" rpy="0 0 0"/>
     </joint>
-    <!-- Link 0: Platform -->
+    <!-- Link: Platform -->
     <link name="${prefix}_platform_link">
       <visual>
@@ -17,5 +17,5 @@
           <mesh filename="file://$(find sobit_light_description)/meshes/arm/omx1_link_base.stl" scale="0.001 0.001 0.001"/>
         </geometry>
-        <material name="grey"/>
+        <material name="black"/>
       </visual>
       <collision>
@@ -33,5 +33,5 @@
       </inertial>
     </link>
-    <!-- Joint 1: Base -->
+    <!-- Joint: Base -->
     <joint name="${prefix}_base_joint" type="fixed">
       <parent link="${prefix}_platform_link"/>
@@ -39,5 +39,5 @@
       <origin xyz="${-0.0112-0.016/2} 0.0 0.008" rpy="0 0 0"/>
     </joint>
-    <!-- Link 1: Base -->
+    <!-- Link: Base -->
     <link name="${prefix}_base_link">
       <visual>
@@ -46,5 +46,5 @@
           <mesh filename="file://$(find sobit_light_description)/meshes/arm/omx1_link1.stl" scale="0.001 0.001 0.001"/>
         </geometry>
-        <material name="grey"/>
+        <material name="black"/>
       </visual>
       <collision>
@@ -62,14 +62,14 @@
       </inertial>
     </link>
-    <!-- Joint 2: Shoulder -->
-    <joint name="${prefix}_1_joint" type="revolute">
+    <!-- Act 1: Shoulder Roll -->
+    <joint name="${prefix}_shoulder_roll_joint" type="revolute">
       <parent link="${prefix}_base_link"/>
-      <child link="${prefix}_1_link"/>
+      <child link="${prefix}_shoulder_roll_link"/>
       <origin xyz="0.0 0.0 0.0465" rpy="0 ${M_PI/2} 0"/>
       <axis xyz="0 0 1"/>
       <limit velocity="4.8" effort="1" lower="${-M_PI}" upper="${M_PI}" />
     </joint>
-    <!--  Link 2: Shoulder -->
-    <link name="${prefix}_1_link">
+    <!--  Act 1: Shoulder Roll -->
+    <link name="${prefix}_shoulder_roll_link">
       <visual>
         <origin xyz="0 0 0.0" rpy="0 0 ${M_PI/2}"/>
@@ -77,5 +77,5 @@
           <mesh filename="file://$(find sobit_light_description)/meshes/arm/omx1_link2.stl" scale="0.001 0.001 0.001"/>
         </geometry>
-        <material name="grey"/>
+        <material name="black"/>
       </visual>
       <collision>
@@ -93,14 +93,14 @@
       </inertial>
     </link>
-    <!--  Joint 3: Upper Arm -->
-    <joint name="${prefix}_2_joint" type="revolute">
-      <parent link="${prefix}_1_link"/>
-      <child link="${prefix}_2_link"/>
+    <!--  Act 2: Shoulder Pitch (right) -->
+    <joint name="${prefix}_shoulder_pitch_joint" type="revolute">
+      <parent link="${prefix}_shoulder_roll_link"/>
+      <child link="${prefix}_shoulder_pitch_link"/>
       <origin xyz="0.0 0.0 0.05095" rpy="0 0 0"/>
       <axis xyz="0 1 0"/>
       <limit velocity="4.8" effort="1" lower="${-M_PI/2}" upper="${M_PI/2}" />
     </joint>
-    <!--  Link 3: Upper Arm -->
-    <link name="${prefix}_2_link">
+    <!--  Act 2: Shoulder Pitch (right) -->
+    <link name="${prefix}_shoulder_pitch_link">
       <visual>
         <origin xyz="0 0 0" rpy="0 0 ${M_PI/2}"/>
@@ -108,5 +108,5 @@
           <mesh filename="file://$(find sobit_light_description)/meshes/arm/omx1_link3.stl" scale="0.001 0.001 0.001"/>
         </geometry>
-        <material name="grey"/>
+        <material name="black"/>
       </visual>
       <collision>
@@ -124,15 +124,15 @@
       </inertial>
     </link>
-    <!--  Joint 3: Upper Arm (SUB) -->
-    <joint name="${prefix}_2_sub_joint" type="revolute">
-      <parent link="${prefix}_1_link"/>
-      <child link="${prefix}_2_sub_link"/>
+    <!--  Act 3: Shoulder Pitch (left) -->
+    <joint name="${prefix}_shoulder_pitch_sub_joint" type="revolute">
+      <parent link="${prefix}_shoulder_roll_link"/>
+      <child link="${prefix}_shoulder_pitch_sub_link"/>
       <origin xyz="0.0 0.0 0.05095" rpy="0 0 0"/>
       <axis xyz="0 1 0"/>
       <limit velocity="4.8" effort="1" lower="${-M_PI/2}" upper="${M_PI/2}" />
-      <mimic joint="${prefix}_2_joint" multiplier="-1" offset="0"/>
-    </joint>
-    <!--  Link 3: Upper Arm (SUB) -->
-    <link name="${prefix}_2_sub_link">
+      <mimic joint="${prefix}_shoulder_pitch_joint" multiplier="-1" offset="0"/>
+    </joint>
+    <!--  Act 3: Shoulder Pitch (left) -->
+    <link name="${prefix}_shoulder_pitch_sub_link">
       <!-- <visual>
         <origin xyz="0 0 0" rpy="0 0 ${M_PI/2}"/>
@@ -140,12 +140,12 @@
           <mesh filename="file://$(find sobit_light_description)/meshes/arm/omx1_link3.stl" scale="0.001 0.001 0.001"/>
         </geometry>
-        <material name="grey"/>
-      </visual>
-      <collision>
+        <material name="black"/>
+      </visual> -->
+      <!-- <collision>
         <origin xyz="${0.03575-0.0585/2} 0.0 ${-0.016+(0.14475+0.016)/2}" rpy="0 0 0"/>
         <geometry>
           <box size="0.0585 0.0440 ${0.14475+0.016}"/>
         </geometry>
-      </collision>
+      </collision> -->
       <inertial>
         <origin xyz="${0.03575-0.0585/2} 0.0 ${-0.016+(0.14475+0.016)/2}" rpy="0 0 0"/>
@@ -154,16 +154,16 @@
                   iyy="${1/12*0.261*(0.0440**2+(0.14475+0.016)**2)}" iyz="0.0"
                   izz="${1/12*0.261*(0.0585**2+0.0440**2)}" />
-      </inertial> -->
-    </link>
-    <!--  Joint 4: Lower Arm -->
-    <joint name="${prefix}_3_joint" type="revolute">
-      <parent link="${prefix}_2_link"/>
-      <child link="${prefix}_3_link"/>
+      </inertial>
+    </link>
+    <!--  Act 4: Elbow Pitch -->
+    <joint name="${prefix}_elbow_pitch_joint" type="revolute">
+      <parent link="${prefix}_shoulder_pitch_link"/>
+      <child link="${prefix}_elbow_pitch_link"/>
       <origin xyz="0.022 -0.0 0.128" rpy="0 0 0"/>
       <axis xyz="0 1 0"/>
       <limit velocity="4.8" effort="1" lower="${-M_PI/2}" upper="${M_PI/2}" />
     </joint>
-    <!--  Link 4: Lower Arm -->
-    <link name="${prefix}_3_link">
+    <!--  Act 4: Elbow Pitch -->
+    <link name="${prefix}_elbow_pitch_link">
       <visual>
         <origin xyz="0 0 0" rpy="0 0 ${M_PI/2}"/>
@@ -171,5 +171,5 @@
           <mesh filename="file://$(find sobit_light_description)/meshes/arm/omx1_link4.stl" scale="0.001 0.001 0.001"/>
         </geometry>
-        <material name="grey"/>
+        <material name="black"/>
       </visual>
       <collision>
@@ -187,14 +187,14 @@
       </inertial>
     </link>
-    <!--  Joint 5: Forearm Upper -->
-    <joint name="${prefix}_4_joint" type="revolute">
-      <parent link="${prefix}_3_link"/>
-      <child link="${prefix}_4_link"/>
+    <!--  Act 5: Forearm Roll -->
+    <joint name="${prefix}_forearm_roll_joint" type="revolute">
+      <parent link="${prefix}_elbow_pitch_link"/>
+      <child link="${prefix}_forearm_roll_link"/>
       <origin xyz="0.0835 0.0 0.0" rpy="0 0 0"/>
       <axis xyz="1 0 0"/>
       <limit velocity="4.8" effort="1" lower="${-M_PI}" upper="${M_PI}" />
     </joint>
-    <!--  Link 5: Forearm Upper -->
-    <link name="${prefix}_4_link">
+    <!--  Act 5: Forearm Roll -->
+    <link name="${prefix}_forearm_roll_link">
       <visual>
         <origin xyz="0 0 0" rpy="0 0 ${M_PI/2}"/>
@@ -202,5 +202,5 @@
           <mesh filename="file://$(find sobit_light_description)/meshes/arm/omx1_link5.stl" scale="0.001 0.001 0.001"/>
         </geometry>
-        <material name="grey"/>
+        <material name="black"/>
       </visual>
       <collision>
@@ -218,14 +218,14 @@
       </inertial>
     </link>
-    <!--  Joint 6: Forearm Lower -->
-    <joint name="${prefix}_5_joint" type="revolute">
-      <parent link="${prefix}_4_link"/>
-      <child link="${prefix}_5_link"/>
+    <!--  Act 6: Wrist Pitch -->
+    <joint name="${prefix}_wrist_pitch_joint" type="revolute">
+      <parent link="${prefix}_forearm_roll_link"/>
+      <child link="${prefix}_wrist_pitch_link"/>
       <origin xyz="0.0405 0.0 0.0" rpy="0 0 0"/>
       <axis xyz="0 1 0"/>
       <limit velocity="4.8" effort="1" lower="${-M_PI/2}" upper="${M_PI/2}" />
     </joint>
-    <!--  Link 6: Forearm Lower -->
-    <link name="${prefix}_5_link">
+    <!--  Act 6: Wrist Pitch -->
+    <link name="${prefix}_wrist_pitch_link">
       <visual>
         <origin xyz="0 0 0" rpy="0 0 ${M_PI/2}"/>
@@ -233,5 +233,5 @@
           <mesh filename="file://$(find sobit_light_description)/meshes/arm/omx1_link6.stl" scale="0.001 0.001 0.001"/>
         </geometry>
-        <material name="grey"/>
+        <material name="black"/>
       </visual>
       <collision>
@@ -249,14 +249,14 @@
       </inertial>
     </link>
-    <!--  Joint 7: Wrist (Hand Base) -->
-    <joint name="${prefix}_6_joint" type="revolute">
-      <parent link="${prefix}_5_link"/>
-      <child link="${prefix}_6_link"/>
+    <!--  Act 7: Wrist Roll -->
+    <joint name="${prefix}_wrist_roll_joint" type="revolute">
+      <parent link="${prefix}_wrist_pitch_link"/>
+      <child link="${prefix}_wrist_roll_link"/>
       <origin xyz="0.064 0 0.0" rpy="0 0 0"/>
       <axis xyz="1 0 0"/>
       <limit velocity="4.8" effort="1" lower="${-M_PI}" upper="${M_PI}" />
     </joint>
-    <!--  Link 7: Wrist (Hand Base) -->
-    <link name="${prefix}_6_link">
+    <!--  Act 7: Wrist Roll -->
+    <link name="${prefix}_wrist_roll_link">
       <visual>
         <origin xyz="0 0 0" rpy="0 0 ${M_PI/2}"/>
@@ -264,5 +264,5 @@
           <mesh filename="file://$(find sobit_light_description)/meshes/arm/omx1_link7_hand_base.stl" scale="0.001 0.001 0.001"/>
         </geometry>
-        <material name="grey"/>
+        <material name="black"/>
       </visual>
       <collision>
@@ -280,11 +280,11 @@
       </inertial>
     </link>
-    <!--  Joint 8: Hand -->
+    <!--  Joint: Hand Base -->
     <joint name="${prefix}_hand_joint" type="fixed">
-      <parent link="${prefix}_6_link"/>
+      <parent link="${prefix}_wrist_roll_link"/>
       <child link="${prefix}_hand_link"/>
       <origin xyz="0.05 0.0 0.0" rpy="0 0 0"/>
     </joint>
-    <!--  Link 8: Hand -->
+    <!--  Link: Hand Base -->
     <link name="${prefix}_hand_link">
       <visual>
@@ -293,5 +293,5 @@
           <mesh filename="file://$(find sobit_light_description)/meshes/arm/omx1_link8_hand.stl" scale="0.001 0.001 0.001"/>
         </geometry>
-        <material name="grey"/>
+        <material name="black"/>
       </visual>
       <collision>

File: sobit_light_description/urdf/dxl_control.urdf.xacro (robot description, xacro)
@@ -11,5 +11,5 @@
         <!-- <param name="use_dummy">true</param> -->
       </hardware>
-      <joint name="arm_1_joint">
+      <joint name="arm_shoulder_roll_joint">
         <param name="id">1</param>
         <command_interface name="position"/>
@@ -19,5 +19,5 @@
         <state_interface name="effort"/>
       </joint>
-      <joint name="arm_2_sub_joint">
+      <joint name="arm_shoulder_pitch_sub_joint">
         <param name="id">2</param>
         <command_interface name="position"/>
@@ -27,5 +27,5 @@
         <state_interface name="effort"/>
       </joint>
-      <joint name="arm_2_joint">
+      <joint name="arm_shoulder_pitch_joint">
         <param name="id">3</param>
         <command_interface name="position"/>
@@ -35,5 +35,5 @@
         <state_interface name="effort"/>
       </joint>
-      <joint name="arm_3_joint">
+      <joint name="arm_elbow_pitch_joint">
         <param name="id">4</param>
         <command_interface name="position"/>
@@ -43,5 +43,5 @@
         <state_interface name="effort"/>
       </joint>
-      <joint name="arm_4_joint">
+      <joint name="arm_forearm_roll_joint">
         <param name="id">5</param>
         <command_interface name="position"/>
@@ -51,5 +51,5 @@
         <state_interface name="effort"/>
       </joint>
-      <joint name="arm_5_joint">
+      <joint name="arm_wrist_pitch_joint">
         <param name="id">6</param>
         <command_interface name="position"/>
@@ -59,5 +59,5 @@
         <state_interface name="effort"/>
       </joint>
-      <joint name="arm_6_joint">
+      <joint name="arm_wrist_roll_joint">
         <param name="id">7</param>
         <command_interface name="position"/>
@@ -67,5 +67,6 @@
         <state_interface name="effort"/>
       </joint>
-      <joint name="hand_finger_l_joint">
+      <joint name="hand_joint">
+      <!-- <joint name="hand_finger_l_joint"> -->
         <param name="id">8</param>
         <command_interface name="position"/>
@@ -75,5 +76,5 @@
         <state_interface name="effort"/>
       </joint>
-      <joint name="head_pan_joint">
+      <joint name="head_yaw_joint">
         <param name="id">11</param>
         <command_interface name="position"/>
@@ -83,5 +84,5 @@
         <state_interface name="effort"/>
       </joint>
-      <joint name="head_tilt_joint">
+      <joint name="head_pitch_joint">
         <param name="id">12</param>
         <command_interface name="position"/>

File: sobit_light_description/urdf/gazebo.urdf.xacro (robot description, xacro)
@@ -100,16 +100,16 @@
         <plugin>ign_ros2_control/IgnitionSystem</plugin>
       </hardware>
-      <joint name="arm_1_joint">
-        <command_interface name="position">
-          <param name="min">-3.141592654</param>
-          <param name="max">3.141592654</param>
-        </command_interface>
-        <state_interface name="position">
-          <param name="initial_value">0.0</param>
-        </state_interface>
-        <state_interface name="velocity"/>
-        <state_interface name="effort"/>
-      </joint>
-      <joint name="arm_2_joint">
+      <joint name="arm_shoulder_roll_joint">
+        <command_interface name="position">
+          <param name="min">-3.141592654</param>
+          <param name="max">3.141592654</param>
+        </command_interface>
+        <state_interface name="position">
+          <param name="initial_value">0.0</param>
+        </state_interface>
+        <state_interface name="velocity"/>
+        <state_interface name="effort"/>
+      </joint>
+      <joint name="arm_shoulder_pitch_joint">
         <command_interface name="position">
           <param name="min">-1.570796327</param>
@@ -122,5 +122,13 @@
         <state_interface name="effort"/>
       </joint>
-      <joint name="arm_3_joint">
+      <joint name="arm_shoulder_pitch_sub_joint">
+        <param name="mimic">arm_shoulder_pitch_joint</param>
+        <param name="multiplier">1</param>
+        <command_interface name="position"/>
+        <state_interface name="position"/>
+        <state_interface name="velocity"/>
+        <state_interface name="effort"/>
+      </joint>
+      <joint name="arm_elbow_pitch_joint">
         <command_interface name="position">
           <param name="min">-1.570796327</param>
@@ -133,16 +141,16 @@
         <state_interface name="effort"/>
       </joint>
-      <joint name="arm_4_joint">
-        <command_interface name="position">
-          <param name="min">-3.141592654</param>
-          <param name="max">3.141592654</param>
-        </command_interface>
-        <state_interface name="position">
-          <param name="initial_value">0.0</param>
-        </state_interface>
-        <state_interface name="velocity"/>
-        <state_interface name="effort"/>
-      </joint>
-      <joint name="arm_5_joint">
+      <joint name="arm_forearm_roll_joint">
+        <command_interface name="position">
+          <param name="min">-3.141592654</param>
+          <param name="max">3.141592654</param>
+        </command_interface>
+        <state_interface name="position">
+          <param name="initial_value">0.0</param>
+        </state_interface>
+        <state_interface name="velocity"/>
+        <state_interface name="effort"/>
+      </joint>
+      <joint name="arm_wrist_pitch_joint">
         <command_interface name="position">
           <param name="min">-1.570796327</param>
@@ -155,5 +163,5 @@
         <state_interface name="effort"/>
       </joint>
-      <joint name="arm_6_joint">
+      <joint name="arm_wrist_roll_joint">
         <command_interface name="position">
           <param name="min">-3.141592654</param>
@@ -172,5 +180,6 @@
         <plugin>ign_ros2_control/IgnitionSystem</plugin>
       </hardware>
-      <joint name="hand_finger_l_joint">
+      <!-- <joint name="hand_finger_l_joint"> -->
+      <joint name="hand_joint">
         <command_interface name="position"/>
         <state_interface name="position">
@@ -180,6 +189,8 @@
         <state_interface name="effort"/>
       </joint>
-      <joint name="hand_finger_r_joint">
-        <param name="mimic">hand_finger_l_joint</param>
+      <!-- <joint name="hand_finger_r_joint"> -->
+      <joint name="hand_sub_joint">
+        <!-- <param name="mimic">hand_finger_l_joint</param> -->
+        <param name="mimic">hand_joint</param>
         <param name="multiplier">1</param>
         <command_interface name="position"/>
@@ -194,16 +205,16 @@
         <plugin>ign_ros2_control/IgnitionSystem</plugin>
       </hardware>
-      <joint name="head_pan_joint">
-        <command_interface name="position">
-          <param name="min">-3.141592654</param>
-          <param name="max">3.141592654</param>
-        </command_interface>
-        <state_interface name="position">
-          <param name="initial_value">0.0</param>
-        </state_interface>
-        <state_interface name="velocity"/>
-        <state_interface name="effort"/>
-      </joint>
-      <joint name="head_tilt_joint">
+      <joint name="head_yaw_joint">
+        <command_interface name="position">
+          <param name="min">-3.141592654</param>
+          <param name="max">3.141592654</param>
+        </command_interface>
+        <state_interface name="position">
+          <param name="initial_value">0.0</param>
+        </state_interface>
+        <state_interface name="velocity"/>
+        <state_interface name="effort"/>
+      </joint>
+      <joint name="head_pitch_joint">
         <command_interface name="position">
           <param name="min">-3.141592654</param>

File: sobit_light_description/urdf/hand/hand.transmission.xacro (robot description, xacro)
@@ -2,6 +2,8 @@
 <robot name="hand_transmission" xmlns:xacro="http://ros.org/wiki/xacro">
   <xacro:macro name="hand_transmission" params="prefix_hand prefix_finger">
-    <effort_joint_transmission joint="${prefix_hand}_${prefix_finger}_l_joint" reduction="1" />
-    <effort_joint_transmission joint="${prefix_hand}_${prefix_finger}_r_joint" reduction="1" />
+    <effort_joint_transmission joint="${prefix_hand}_joint" reduction="1" />
+    <effort_joint_transmission joint="${prefix_hand}_sub_joint" reduction="1" />
+    <!-- <effort_joint_transmission joint="${prefix_hand}_${prefix_finger}_l_joint" reduction="1" /> -->
+    <!-- <effort_joint_transmission joint="${prefix_hand}_${prefix_finger}_r_joint" reduction="1" /> -->
   </xacro:macro>
 </robot>
