Commit message: [UPD] naming based on motion

File: sobit_light_description/urdf/hand/hand.urdf.xacro (robot description, xacro)
@@ -3,5 +3,5 @@
   <xacro:include filename="$(find sobit_light_description)/urdf/hand/hand.transmission.xacro" />
   <xacro:macro name="hand" params="prefix_hand prefix_finger parent">
-    <!--  Joint 9: Hand left sub -->
+    <!--  Joint: Hand left sub -->
     <joint name="${prefix_hand}_sub_l_joint" type="fixed">
       <parent link="${parent}"/>
@@ -9,5 +9,5 @@
       <origin xyz="0.009 0.015 0.0" rpy="0 0 0"/>
     </joint>
-    <!--  Link 9: Hand left sub -->
+    <!--  Link: Hand left sub -->
     <link name="${prefix_hand}_sub_l_link">
       <visual>
@@ -16,5 +16,5 @@
           <mesh filename="file://$(find sobit_light_description)/meshes/hand/omx1_link9-10_hand.stl" scale="0.001 0.001 0.001"/>
         </geometry>
-        <material name="grey"/>
+        <material name="black"/>
       </visual>
       <collision>
@@ -32,5 +32,5 @@
       </inertial>
     </link>
-    <!--  Joint 10: Hand right sub -->
+    <!--  Joint: Hand right sub -->
     <joint name="${prefix_hand}_sub_r_joint" type="fixed">
       <parent link="${parent}"/>
@@ -38,5 +38,5 @@
       <origin xyz="0.009 -0.015 0.0" rpy="0 0 0"/>
     </joint>
-    <!--  Link 10: Hand right sub -->
+    <!--  Link: Hand right sub -->
     <link name="${prefix_hand}_sub_r_link">
       <visual>
@@ -45,5 +45,5 @@
           <mesh filename="file://$(find sobit_light_description)/meshes/hand/omx1_link9-10_hand.stl" scale="0.001 0.001 0.001"/>
         </geometry>
-        <material name="grey"/>
+        <material name="black"/>
       </visual>
       <collision>
@@ -61,14 +61,17 @@
       </inertial>
     </link>
-    <!--  Joint 11: Hand Finger Left -->
-    <joint name="${prefix_hand}_${prefix_finger}_l_joint" type="prismatic">
+    <!--  Act 8: Hand Finger (left) -->
+    <!-- <joint name="${prefix_hand}_${prefix_finger}_l_joint" type="prismatic"> -->
+    <joint name="${prefix_hand}_joint" type="prismatic">
       <parent link="${prefix_hand}_sub_l_link"/>
-      <child link="${prefix_hand}_${prefix_finger}_l_link"/>
+      <!-- <child link="${prefix_hand}_${prefix_finger}_l_link"/> -->
+      <child link="${prefix_hand}_link"/>
       <origin xyz="0.0 0.04 0.0" rpy="0 0 0"/>
       <axis xyz="0 1 0"/>
       <limit velocity="4.8" effort="1" lower="${-0.055+0.02675}" upper="0.0" />
     </joint>
-    <!--  Link 11: Hand Finger Left -->
-    <link name="${prefix_hand}_${prefix_finger}_l_link">
+    <!--  Act 8: Hand Finger (left) -->
+    <!-- <link name="${prefix_hand}_${prefix_finger}_l_link"> -->
+    <link name="${prefix_hand}_link">
       <visual>
         <origin xyz="0.0 0.0 0" rpy="0 0 ${M_PI/2}"/>
@@ -76,5 +79,5 @@
           <mesh filename="file://$(find sobit_light_description)/meshes/hand/omx1_link11-12_finger.stl" scale="0.001 0.001 0.001"/>
         </geometry>
-        <material name="grey"/>
+        <material name="black"/>
       </visual>
       <collision>
@@ -92,15 +95,19 @@
       </inertial>
     </link>
-    <!--  Joint 12: Hand Finger Right -->
-    <joint name="${prefix_hand}_${prefix_finger}_r_joint" type="prismatic">
+    <!--  Act 8: Hand Finger (right) -->
+    <!-- <joint name="${prefix_hand}_${prefix_finger}_r_joint" type="prismatic"> -->
+    <joint name="${prefix_hand}_sub_joint" type="prismatic">
       <parent link="${prefix_hand}_sub_r_link"/>
-      <child link="${prefix_hand}_${prefix_finger}_r_link"/>
+      <!-- <child link="${prefix_hand}_${prefix_finger}_r_link"/> -->
+      <child link="${prefix_hand}_sub_link"/>
       <origin xyz="0.0 -0.04 0.0" rpy="0 0 0"/>
       <axis xyz="0 -1 0"/>
-      <limit velocity="4.8" effort="1" lower="0.0" upper="${-0.055+0.02675}" />
-      <mimic joint="${prefix_hand}_${prefix_finger}_l_joint" multiplier="1"/>
-    </joint>
-    <!--  Link 12: Hand Finger Right -->
-    <link name="${prefix_hand}_${prefix_finger}_r_link">
+      <limit velocity="4.8" effort="1" lower="${-0.055+0.02675}" upper="0.0" />
+      <!-- <mimic joint="${prefix_hand}_${prefix_finger}_l_joint" multiplier="1"/> -->
+      <mimic joint="${prefix_hand}_joint" multiplier="1"/>
+    </joint>
+    <!--  Act 8: Hand Finger (right) -->
+    <!-- <link name="${prefix_hand}_${prefix_finger}_r_link"> -->
+    <link name="${prefix_hand}_sub_link">
       <visual>
         <origin xyz="0.0 -0.0 0" rpy="0 ${M_PI} ${M_PI/2}"/>
@@ -108,5 +115,5 @@
           <mesh filename="file://$(find sobit_light_description)/meshes/hand/omx1_link11-12_finger.stl" scale="0.001 0.001 0.001"/>
         </geometry>
-        <material name="grey"/>
+        <material name="black"/>
       </visual>
       <collision>
@@ -124,11 +131,12 @@
       </inertial>
     </link>
-    <!--  Joint 13: Hand Tip Left -->
+    <!--  Joint: Hand Tip Left -->
     <joint name="${prefix_hand}_${prefix_finger}_tip_l_joint" type="fixed">
-      <parent link="${prefix_hand}_${prefix_finger}_l_link"/>
+      <!-- <parent link="${prefix_hand}_${prefix_finger}_l_link"/> -->
+      <parent link="${prefix_hand}_link"/>
       <child link="${prefix_hand}_${prefix_finger}_tip_l_link"/>
       <origin xyz="${0.0345+0.0375/2} -0.0145 0.0" rpy="0 0 0"/>
     </joint>
-    <!--  Link 13: Hand Tip Left -->
+    <!--  Link: Hand Tip Left -->
     <link name="${prefix_hand}_${prefix_finger}_tip_l_link">
       <visual>
@@ -137,5 +145,5 @@
           <mesh filename="file://$(find sobit_light_description)/meshes/hand/omx1_link13-14_finger.stl" scale="0.001 0.001 0.001"/>
         </geometry>
-        <material name="grey"/>
+        <material name="black"/>
       </visual>
       <collision>
@@ -153,11 +161,12 @@
       </inertial>
     </link>
-    <!--  Joint 14: Hand Tip Right -->
+    <!--  Joint: Hand Tip Right -->
     <joint name="${prefix_hand}_${prefix_finger}_tip_r_joint" type="fixed">
-      <parent link="${prefix_hand}_${prefix_finger}_r_link"/>
+      <!-- <parent link="${prefix_hand}_${prefix_finger}_r_link"/> -->
+      <parent link="${prefix_hand}_sub_link"/>
       <child link="${prefix_hand}_${prefix_finger}_tip_r_link"/>
       <origin xyz="${0.0345+0.0375/2} 0.0145 0.0" rpy="0 0 0"/>
     </joint>
-    <!--  Link 14: Hand Tip Right -->
+    <!--  Link: Hand Tip Right -->
     <link name="${prefix_hand}_${prefix_finger}_tip_r_link">
       <visual>
@@ -166,5 +175,5 @@
           <mesh filename="file://$(find sobit_light_description)/meshes/hand/omx1_link13-14_finger.stl" scale="0.001 0.001 0.001"/>
         </geometry>
-        <material name="grey"/>
+        <material name="black"/>
       </visual>
       <collision>
@@ -182,11 +191,11 @@
       </inertial>
     </link>
-    <!-- Joint 15: End Effector -->
+    <!-- Joint: End Effector -->
     <joint name="end_effector_joint" type="fixed">
       <origin xyz="${0.0935+0.0375/2} 0.0 0.0" rpy="0 0 0"/>
-      <parent link="arm_6_link"/>
+      <parent link="arm_wrist_roll_link"/>
       <child link="${prefix_hand}_end_effector_link"/>
     </joint>
-    <!-- Link 15: End Effector -->
+    <!-- Link: End Effector -->
     <link name="${prefix_hand}_end_effector_link">
       <visual>

File: sobit_light_description/urdf/head/head.transmission.xacro (robot description, xacro)
@@ -2,6 +2,8 @@
 <robot name="head_transmission" xmlns:xacro="http://ros.org/wiki/xacro">
   <xacro:macro name="head_transmission" params="prefix">
-    <position_joint_transmission joint="${prefix}_pan_joint"  reduction="1" />
-    <position_joint_transmission joint="${prefix}_tilt_joint" reduction="1" />
+    <position_joint_transmission joint="${prefix}_yaw_joint"  reduction="1" />
+    <position_joint_transmission joint="${prefix}_pitch_joint" reduction="1" />
+    <!-- <position_joint_transmission joint="${prefix}_yaw_joint"  reduction="1" /> -->
+    <!-- <position_joint_transmission joint="${prefix}_pitch_joint" reduction="1" /> -->
   </xacro:macro>
 </robot>

File: sobit_light_description/urdf/head/head.urdf.xacro (robot description, xacro)
@@ -33,16 +33,12 @@
       </inertial>
     </link>
-    <!-- <joint name="${prefix}_camera_pan_joint" type="revolute"> -->
-    <joint name="${prefix}_pan_joint" type="revolute">
+    <joint name="${prefix}_yaw_joint" type="revolute">
       <parent link="${prefix}_base_link" />
-      <!-- <parent link="${prefix}_camera_base_link" /> -->
-      <child link="${prefix}_pan_link" />
-      <!-- <child link="${prefix}_camera_pan_link" /> -->
+      <child link="${prefix}_yaw_link" />
       <origin xyz="0.012 0.0 0.041" rpy="0.0 0.0 0.0" />
       <axis xyz="0 0 1" />
       <limit effort="30" lower="${-M_PI}" upper="${M_PI}" velocity="${M_PI/2.0}" />
     </joint>
-    <link name="${prefix}_pan_link">
-    <!-- <link name="${prefix}_camera_pan_link"> -->
+    <link name="${prefix}_yaw_link">
       <visual>
         <origin xyz="0.0 0.0 0.0" rpy="0.0 0.0 ${M_PI/2.0}" />
@@ -66,16 +62,12 @@
       </inertial>
     </link>
-    <joint name="${prefix}_tilt_joint" type="revolute">
-    <!-- <joint name="${prefix}_camera_tilt_joint" type="revolute"> -->
-      <parent link="${prefix}_pan_link" />
-      <!-- <parent link="${prefix}_camera_pan_link" /> -->
-      <child link="${prefix}_tilt_link" />
-      <!-- <child link="${prefix}_camera_tilt_link" /> -->
+    <joint name="${prefix}_pitch_joint" type="revolute">
+      <parent link="${prefix}_yaw_link" />
+      <child link="${prefix}_pitch_link" />
       <origin xyz="0.0 0.0 0.0405" rpy="0.0 0.0 0.0" />
       <axis xyz="0 -1 0" />
       <limit effort="30" lower="${-M_PI/2.0}" upper="${M_PI/2.0}" velocity="${M_PI/2.0}" />
     </joint>
-    <link name="${prefix}_tilt_link">
-    <!-- <link name="${prefix}_camera_tilt_link"> -->
+    <link name="${prefix}_pitch_link">
       <visual>
         <origin xyz="0.0 0.0 0.0" rpy="0.0 0.0 ${M_PI/2.0}" />
