Commit message: [FIX] comments with collon are removed

File: sobit_light_description/urdf/arm/arm.transmission.xacro (robot description, xacro)
@@ -1,4 +1,4 @@
 <?xml version="1.0" encoding="UTF-8" ?>
-<!-- OpenManipulator X1000 (ROS Control: Transmission) -->
+<!-- OpenManipulator X1000 (ROS Control - Transmission) -->
 <robot name="arm_transmission" xmlns:xacro="http://ros.org/wiki/xacro">
   <xacro:macro name="arm_transmission" params="prefix">

File: sobit_light_description/urdf/arm/arm.urdf.xacro (robot description, xacro)
@@ -4,5 +4,5 @@
   <xacro:include filename="$(find sobit_light_description)/urdf/arm/arm.transmission.xacro" />
   <xacro:macro name="arm" params="prefix parent">
-    <!-- Joint: Platform -->
+    <!-- Joint - Platform -->
     <joint name="${prefix}_platform_joint" type="fixed">
       <parent link="${parent}"/>
@@ -10,5 +10,5 @@
       <origin xyz="0.122 0.0 0.0" rpy="0 0 0"/>
     </joint>
-    <!-- Link: Platform -->
+    <!-- Link - Platform -->
     <link name="${prefix}_platform_link">
       <visual>
@@ -33,5 +33,5 @@
       </inertial>
     </link>
-    <!-- Joint: Base -->
+    <!-- Joint - Base -->
     <joint name="${prefix}_base_joint" type="fixed">
       <parent link="${prefix}_platform_link"/>
@@ -39,5 +39,5 @@
       <origin xyz="${-0.0112-0.016/2} 0.0 0.008" rpy="0 0 0"/>
     </joint>
-    <!-- Link: Base -->
+    <!-- Link - Base -->
     <link name="${prefix}_base_link">
       <visual>
@@ -62,5 +62,5 @@
       </inertial>
     </link>
-    <!-- Act 1: Shoulder Roll -->
+    <!-- Act 1 - Shoulder Roll -->
     <joint name="${prefix}_shoulder_roll_joint" type="revolute">
       <parent link="${prefix}_base_link"/>
@@ -70,5 +70,5 @@
       <limit velocity="4.8" effort="25" lower="${-M_PI}" upper="${M_PI}" />
     </joint>
-    <!--  Act 1: Shoulder Roll -->
+    <!--  Act 1 - Shoulder Roll -->
     <link name="${prefix}_shoulder_roll_link">
       <visual>
@@ -93,5 +93,5 @@
       </inertial>
     </link>
-    <!--  Act 2: Shoulder Pitch (right) -->
+    <!--  Act 2 - Shoulder Pitch (right) -->
     <joint name="${prefix}_shoulder_pitch_joint" type="revolute">
       <parent link="${prefix}_shoulder_roll_link"/>
@@ -101,5 +101,5 @@
       <limit velocity="4.8" effort="25" lower="${-M_PI/2}" upper="${M_PI/2}" />
     </joint>
-    <!--  Act 2: Shoulder Pitch (right) -->
+    <!--  Act 2 - Shoulder Pitch (right) -->
     <link name="${prefix}_shoulder_pitch_link">
       <visual>
@@ -124,5 +124,5 @@
       </inertial>
     </link>
-    <!--  Act 3: Shoulder Pitch (left) -->
+    <!--  Act 3 - Shoulder Pitch (left) -->
     <joint name="${prefix}_shoulder_pitch_sub_joint" type="revolute">
       <parent link="${prefix}_shoulder_roll_link"/>
@@ -133,19 +133,6 @@
       <!-- <mimic joint="${prefix}_shoulder_pitch_joint" multiplier="-1" offset="0"/> -->
     </joint>
-    <!--  Act 3: Shoulder Pitch (left) -->
+    <!--  Act 3 - Shoulder Pitch (left) -->
     <link name="${prefix}_shoulder_pitch_sub_link">
-      <!-- <visual>
-        <origin xyz="0 0 0" rpy="0 0 ${M_PI/2}"/>
-        <geometry>
-          <mesh filename="file://$(find sobit_light_description)/meshes/arm/omx1_link3.stl" scale="0.001 0.001 0.001"/>
-        </geometry>
-        <material name="black"/>
-      </visual> -->
-      <!-- <collision>
-        <origin xyz="${0.03575-0.0585/2} 0.0 ${-0.016+(0.14475+0.016)/2}" rpy="0 0 0"/>
-        <geometry>
-          <box size="0.0585 0.0440 ${0.14475+0.016}"/>
-        </geometry>
-      </collision> -->
       <inertial>
         <origin xyz="${0.03575-0.0585/2} 0.0 ${-0.016+(0.14475+0.016)/2}" rpy="0 0 0"/>
@@ -156,5 +143,5 @@
       </inertial>
     </link>
-    <!--  Act 4: Elbow Pitch -->
+    <!--  Act 4 - Elbow Pitch -->
     <joint name="${prefix}_elbow_pitch_joint" type="revolute">
       <parent link="${prefix}_shoulder_pitch_link"/>
@@ -164,5 +151,5 @@
       <limit velocity="4.8" effort="25" lower="${-M_PI/2}" upper="${M_PI/2}" />
     </joint>
-    <!--  Act 4: Elbow Pitch -->
+    <!--  Act 4 - Elbow Pitch -->
     <link name="${prefix}_elbow_pitch_link">
       <visual>
@@ -187,5 +174,5 @@
       </inertial>
     </link>
-    <!--  Act 5: Forearm Roll -->
+    <!--  Act 5 - Forearm Roll -->
     <joint name="${prefix}_forearm_roll_joint" type="revolute">
       <parent link="${prefix}_elbow_pitch_link"/>
@@ -195,5 +182,5 @@
       <limit velocity="4.8" effort="25" lower="${-M_PI}" upper="${M_PI}" />
     </joint>
-    <!--  Act 5: Forearm Roll -->
+    <!--  Act 5 - Forearm Roll -->
     <link name="${prefix}_forearm_roll_link">
       <visual>
@@ -218,5 +205,5 @@
       </inertial>
     </link>
-    <!--  Act 6: Wrist Pitch -->
+    <!--  Act 6 - Wrist Pitch -->
     <joint name="${prefix}_wrist_pitch_joint" type="revolute">
       <parent link="${prefix}_forearm_roll_link"/>
@@ -226,5 +213,5 @@
       <limit velocity="4.8" effort="25" lower="${-M_PI/2}" upper="${M_PI/2}" />
     </joint>
-    <!--  Act 6: Wrist Pitch -->
+    <!--  Act 6 - Wrist Pitch -->
     <link name="${prefix}_wrist_pitch_link">
       <visual>
@@ -249,5 +236,5 @@
       </inertial>
     </link>
-    <!--  Act 7: Wrist Roll -->
+    <!--  Act 7 - Wrist Roll -->
     <joint name="${prefix}_wrist_roll_joint" type="revolute">
       <parent link="${prefix}_wrist_pitch_link"/>
@@ -257,5 +244,5 @@
       <limit velocity="4.8" effort="25" lower="${-M_PI}" upper="${M_PI}" />
     </joint>
-    <!--  Act 7: Wrist Roll -->
+    <!--  Act 7 - Wrist Roll -->
     <link name="${prefix}_wrist_roll_link">
       <visual>
@@ -280,5 +267,5 @@
       </inertial>
     </link>
-    <!--  Joint: Hand Base -->
+    <!--  Joint - Hand Base -->
     <joint name="${prefix}_hand_joint" type="fixed">
       <parent link="${prefix}_wrist_roll_link"/>
@@ -286,5 +273,5 @@
       <origin xyz="0.05 0.0 0.0" rpy="0 0 0"/>
     </joint>
-    <!--  Link: Hand Base -->
+    <!--  Link - Hand Base -->
     <link name="${prefix}_hand_link">
       <visual>

File: sobit_light_description/urdf/controllers.urdf.xacro (robot description, xacro)
@@ -8,5 +8,5 @@
         <xacro:if value="${$(arg enable_gz)}">
           <plugin>ign_ros2_control/IgnitionSystem</plugin>
-          <!-- <plugin>gazebo_ros2_control/GazeboHardware</plugin> -->
+          <!-- <plugin>gz_ros2_control/GazeboSimSystem</plugin> -->
         </xacro:if>
         <xacro:unless value="${$(arg enable_gz)}">
@@ -18,5 +18,5 @@
         </xacro:unless>
       </hardware>
-      <!-- Position Drive: Arm -->
+      <!-- Position Drive - Arm -->
       <joint name="arm_shoulder_roll_joint">
         <xacro:unless value="${$(arg enable_gz)}">
@@ -128,5 +128,5 @@
         <state_interface name="effort"/>
       </joint>
-      <!-- Position Drive: Hand -->
+      <!-- Position Drive - Hand -->
       <joint name="hand_joint">
         <xacro:unless value="${$(arg enable_gz)}">
@@ -152,5 +152,5 @@
         </joint>
       </xacro:if>
-      <!-- Position Drive: Head -->
+      <!-- Position Drive - Head -->
       <joint name="head_yaw_joint">
         <xacro:unless value="${$(arg enable_gz)}">
@@ -189,5 +189,5 @@
         <hardware>
           <plugin>ign_ros2_control/IgnitionSystem</plugin>
-          <!-- <plugin>gazebo_ros2_control/GazeboHardware</plugin> -->
+          <!-- <plugin>gz_ros2_control/GazeboSimSystem</plugin> -->
         </hardware>
         <joint name="base_l_drive_wheel_joint">
@@ -216,5 +216,4 @@
     <xacro:if value="${$(arg enable_gz)}">
       <gazebo>
-        <!-- <plugin filename="gz_ros2_control-system" name="gz_ros2_control::GazeboSimROS2ControlPlugin"> -->
         <plugin filename="ign_ros2_control-system" name="ign_ros2_control::IgnitionROS2ControlPlugin">
           <ros>

File: sobit_light_description/urdf/gazebo.urdf.xacro (robot description, xacro)
@@ -3,5 +3,5 @@
 <robot name="sobit_light_gazebo" xmlns:xacro="http://ros.org/wiki/xacro">
   <xacro:macro name="gazebo_sensors" params="robot_name enable_gz_front_cam_color:=True enable_gz_back_cam_color:=True enable_gz_head_cam_color:=True enable_gz_head_cam_depth:=True enable_gz_hand_cam_color:=True enable_gz_hand_cam_depth:=True enable_gz_lidar:=True enable_gz_imu:=True">
-    <!-- Sensor: Base Front Camera (Color) -->
+    <!-- Sensor - Base Front Camera (Color) -->
     <xacro:if value="${enable_gz_front_cam_color}">
       <gazebo reference="imu_link">
@@ -16,5 +16,5 @@
       </gazebo>
     </xacro:if>
-    <!-- [TODO] Sensor: Base Front Camera (Color) -->
+    <!-- [TODO] Sensor - Base Front Camera (Color) -->
     <!-- <gazebo reference="camera_front_link">
       <sensor name="base_front_camera_color" type="wideanglecamera">
@@ -50,5 +50,5 @@
       </sensor>
     </gazebo> -->
-    <!-- Sensor: Base Front Camera (Color) -->
+    <!-- Sensor - Base Front Camera (Color) -->
     <xacro:if value="${enable_gz_front_cam_color}">
       <gazebo reference="camera_front_link">
@@ -72,5 +72,5 @@
               <far>10</far>
             </clip>
-            <!-- TODO: adjust noise -->
+            <!-- TODO - adjust noise -->
             <!-- <noise>
               <type>gaussian</type>
@@ -82,5 +82,5 @@
       </gazebo>
     </xacro:if>
-    <!-- [TODO] Sensor: Base Back Camera (Color) -->
+    <!-- [TODO] Sensor - Base Back Camera (Color) -->
     <!-- <gazebo reference="camera_back_link">
       <sensor name="base_back_camera_color" type="wideanglecamera">
@@ -116,5 +116,5 @@
       </sensor>
     </gazebo> -->
-    <!-- Sensor: Base Back Camera (Color) -->
+    <!-- Sensor - Base Back Camera (Color) -->
     <xacro:if value="${enable_gz_back_cam_color}">
       <gazebo reference="camera_back_link">
@@ -138,5 +138,5 @@
               <far>10</far>
             </clip>
-            <!-- TODO: adjust noise -->
+            <!-- TODO - adjust noise -->
             <!-- <noise>
               <type>gaussian</type>
@@ -148,5 +148,5 @@
       </gazebo>
     </xacro:if>
-    <!-- Sensor: Head Camera (Color) -->
+    <!-- Sensor - Head Camera (Color) -->
     <xacro:if value="${enable_gz_head_cam_color}">
       <gazebo reference="head_camera_color_optical_frame">
@@ -170,5 +170,5 @@
               <far>10</far>
             </clip>
-            <!-- TODO: adjust noise -->
+            <!-- TODO - adjust noise -->
             <!-- <noise>
               <type>gaussian</type>
@@ -180,5 +180,5 @@
       </gazebo>
     </xacro:if>
-    <!-- Sensor: Head Camera (Depth) -->
+    <!-- Sensor - Head Camera (Depth) -->
     <xacro:if value="${enable_gz_head_cam_depth}">
       <gazebo reference="head_camera_depth_optical_frame">
@@ -201,5 +201,5 @@
               <far>10</far>
             </clip>
-            <!-- TODO: adjust noise -->
+            <!-- TODO - adjust noise -->
             <!-- <noise>
               <type>gaussian</type>
@@ -211,5 +211,5 @@
       </gazebo>
     </xacro:if>
-    <!-- Sensor: Hand Camera (Color) -->
+    <!-- Sensor - Hand Camera (Color) -->
     <xacro:if value="${enable_gz_hand_cam_color}">
       <gazebo reference="hand_camera_color_optical_frame">
@@ -233,5 +233,5 @@
               <far>10</far>
             </clip>
-            <!-- TODO: adjust noise -->
+            <!-- TODO - adjust noise -->
             <!-- <noise>
               <type>gaussian</type>
@@ -243,5 +243,5 @@
       </gazebo>
     </xacro:if>
-    <!-- Sensor: Hand Camera (Depth) -->
+    <!-- Sensor - Hand Camera (Depth) -->
     <xacro:if value="${enable_gz_hand_cam_depth}">
       <gazebo reference="hand_camera_depth_optical_frame">
@@ -264,5 +264,5 @@
               <far>10</far>
             </clip>
-            <!-- TODO: adjust noise -->
+            <!-- TODO - adjust noise -->
             <!-- <noise>
               <type>gaussian</type>
@@ -274,5 +274,5 @@
       </gazebo>
     </xacro:if>
-    <!-- Sensor: LiDAR -->
+    <!-- Sensor - LiDAR -->
     <xacro:if value="${enable_gz_lidar}">
       <gazebo reference="sim_laser_frame">
@@ -309,19 +309,6 @@
       </gazebo>
     </xacro:if>
-    <!-- Publish Pose -->
-    <!-- <gazebo>
-      <plugin
-          filename="gz-sim-pose-publisher-system"
-          name="gz::sim::systems::PosePublisher">
-        <publish_link_pose>true</publish_link_pose>
-        <publish_collision_pose>false</publish_collision_pose>
-        <publish_visual_pose>false</publish_visual_pose>
-        <publish_sensor_pose>false</publish_sensor_pose>
-        <publish_nested_model_pose>true</publish_nested_model_pose>
-      </plugin>
-    </gazebo> -->
     <!-- Publish Joint States -->
     <gazebo>
-      <!-- <plugin filename="ignition-gazebo-joint-state-publisher-system" name="ignition::gazebo::systems::JointStatePublisher"> -->
       <plugin filename="gz-sim-joint-state-publisher-system" name="gz::sim::systems::JointStatePublisher">
         <topic>${robot_name}/joint_states</topic>

File: sobit_light_description/urdf/hand/hand.urdf.xacro (robot description, xacro)
@@ -3,5 +3,5 @@
   <xacro:include filename="$(find sobit_light_description)/urdf/hand/hand.transmission.xacro" />
   <xacro:macro name="hand" params="prefix_hand prefix_finger parent">
-    <!--  Joint: Hand left sub -->
+    <!--  Joint - Hand left sub -->
     <joint name="${prefix_hand}_sub_l_joint" type="fixed">
       <parent link="${parent}"/>
@@ -9,5 +9,5 @@
       <origin xyz="0.009 0.015 0.0" rpy="0 0 0"/>
     </joint>
-    <!--  Link: Hand left sub -->
+    <!--  Link - Hand left sub -->
     <link name="${prefix_hand}_sub_l_link">
       <visual>
@@ -32,5 +32,5 @@
       </inertial>
     </link>
-    <!--  Joint: Hand right sub -->
+    <!--  Joint - Hand right sub -->
     <joint name="${prefix_hand}_sub_r_joint" type="fixed">
       <parent link="${parent}"/>
@@ -38,5 +38,5 @@
       <origin xyz="0.009 -0.015 0.0" rpy="0 0 0"/>
     </joint>
-    <!--  Link: Hand right sub -->
+    <!--  Link - Hand right sub -->
     <link name="${prefix_hand}_sub_r_link">
       <visual>
@@ -61,5 +61,5 @@
       </inertial>
     </link>
-    <!--  Act 8: Hand Finger (left) -->
+    <!--  Act 8 - Hand Finger (left) -->
     <joint name="${prefix_hand}_joint" type="prismatic">
       <parent link="${prefix_hand}_sub_l_link"/>
@@ -69,5 +69,5 @@
       <limit velocity="4.8" effort="1" lower="0.0" upper="${0.02675-0.055}" />
     </joint>
-    <!--  Act 8: Hand Finger (left) -->
+    <!--  Act 8 - Hand Finger (left) -->
     <link name="${prefix_hand}_link">
       <visual>
@@ -92,5 +92,5 @@
       </inertial>
     </link>
-    <!--  Act 8: Hand Finger (right) -->
+    <!--  Act 8 - Hand Finger (right) -->
     <joint name="${prefix_hand}_sub_joint" type="prismatic">
       <parent link="${prefix_hand}_sub_r_link"/>
@@ -101,5 +101,5 @@
       <mimic joint="${prefix_hand}_joint" multiplier="-1"/>
     </joint>
-    <!--  Act 8: Hand Finger (right) -->
+    <!--  Act 8 - Hand Finger (right) -->
     <link name="${prefix_hand}_sub_link">
       <visual>
@@ -124,5 +124,5 @@
       </inertial>
     </link>
-    <!--  Joint: Hand Tip Left -->
+    <!--  Joint - Hand Tip Left -->
     <joint name="${prefix_hand}_${prefix_finger}_tip_l_joint" type="fixed">
       <parent link="${prefix_hand}_link"/>
@@ -130,5 +130,5 @@
       <origin xyz="${0.0345+0.0375/2} -0.0145 0.0" rpy="0 0 0"/>
     </joint>
-    <!--  Link: Hand Tip Left -->
+    <!--  Link - Hand Tip Left -->
     <link name="${prefix_hand}_${prefix_finger}_tip_l_link">
       <visual>
@@ -153,5 +153,5 @@
       </inertial>
     </link>
-    <!--  Joint: Hand Tip Right -->
+    <!--  Joint - Hand Tip Right -->
     <joint name="${prefix_hand}_${prefix_finger}_tip_r_joint" type="fixed">
       <parent link="${prefix_hand}_sub_link"/>
@@ -159,5 +159,5 @@
       <origin xyz="${0.0345+0.0375/2} 0.0145 0.0" rpy="0 0 0"/>
     </joint>
-    <!--  Link: Hand Tip Right -->
+    <!--  Link - Hand Tip Right -->
     <link name="${prefix_hand}_${prefix_finger}_tip_r_link">
       <visual>
@@ -182,5 +182,5 @@
       </inertial>
     </link>
-    <!-- Joint: End Effector -->
+    <!-- Joint - End Effector -->
     <joint name="end_effector_joint" type="fixed">
       <origin xyz="${0.0935+0.0375/2} 0.0 0.0" rpy="0 0 0"/>
@@ -188,5 +188,5 @@
       <child link="${prefix_hand}_end_effector_link"/>
     </joint>
-    <!-- Link: End Effector -->
+    <!-- Link - End Effector -->
     <link name="${prefix_hand}_end_effector_link">
       <visual>

File: sobit_light_description/urdf/sensor/camera_hand.urdf.xacro (robot description, xacro)
@@ -3,5 +3,5 @@
   <xacro:include filename="$(find realsense2_description)/urdf/_d405.urdf.xacro" />
   <xacro:macro name="camera_hand" params="prefix parent">
-    <!-- Joint: Hand Camera Base -->
+    <!-- Joint - Hand Camera Base -->
     <joint name="${prefix}_base_joint" type="fixed">
       <origin xyz="0.03685 0.0 0.0408" rpy="0 0 0"/>
@@ -9,5 +9,5 @@
       <child link="${prefix}_base_link"/>
     </joint>
-    <!-- Link: Hand Camera Base -->
+    <!-- Link - Hand Camera Base -->
     <link name="${prefix}_base_link">
       <visual>

File: sobit_light_description/urdf/transmission.urdf.xacro (robot description, xacro)
@@ -2,5 +2,5 @@
 <!-- SOBIT Light (transmission) -->
 <robot name="sobit_light_transmission" xmlns:xacro="http://ros.org/wiki/xacro">
-  <!-- Transmission macro: Position -->
+  <!-- Transmission macro - Position -->
   <xacro:macro name="SimpleTransmissionPosition" params="joint reduction">
     <transmission name="${joint}_transmission">
@@ -14,5 +14,5 @@
     </transmission>
   </xacro:macro>
-  <!-- Transmission macro: Effort -->
+  <!-- Transmission macro - Effort -->
   <xacro:macro name="SimpleTransmissionEffort" params="joint reduction">
     <transmission name="${joint}_transmission">
@@ -26,5 +26,5 @@
     </transmission>
   </xacro:macro>
-  <!-- Transmission macro: Velocity -->
+  <!-- Transmission macro - Velocity -->
   <xacro:macro name="SimpleTransmissionVelocity" params="joint reduction">
     <transmission name="${joint}_transmission">
