Commit message: [UPD] arm and hand urdf (todo: inertia)

File: sobit_light_description/urdf/arm/arm.urdf.xacro (robot description, xacro)
@@ -2,4 +2,5 @@
 <!-- OpenManipulator X1000 (Arm) -->
 <robot name="arm" xmlns:xacro="http://ros.org/wiki/xacro">
+  <xacro:include filename="$(find sobit_light_description)/urdf/arm/arm.transmission.xacro" />
   <xacro:macro name="arm" params="prefix parent">
     <!-- Joint 0: Platform -->
@@ -7,5 +8,5 @@
       <parent link="${parent}"/>
       <child link="${prefix}_platform_link"/>
-      <origin xyz="-0.0105 -0.0135 0.006" rpy="0 0 0"/>
+      <origin xyz="0.122 0.0 0.0" rpy="0 0 0"/>
     </joint>
     <!-- Link 0: Platform -->
@@ -38,5 +39,5 @@
       <parent link="${prefix}_platform_link"/>
       <child link="${prefix}_base_link"/>
-      <origin xyz="-0.0105 -0.0135 0.006" rpy="0 0 0"/>
+      <origin xyz="${-0.0112-0.016/2} 0.0 0.008" rpy="0 0 0"/>
     </joint>
     <!-- Link 1: Base -->
@@ -64,13 +65,13 @@
     </link>
     <!-- Joint 2: Shoulder -->
-    <joint name="${prefix}_arm1_joint" type="revolute">
+    <joint name="${prefix}_1_joint" type="revolute">
       <parent link="${prefix}_base_link"/>
-      <child link="${prefix}_arm1_link"/>
-      <origin xyz="0.0 0.0 0.0465" rpy="0 0 0"/>
+      <child link="${prefix}_1_link"/>
+      <origin xyz="0.0 0.0 0.0465" rpy="0 ${M_PI/2} 0"/>
       <axis xyz="0 0 1"/>
       <limit velocity="4.8" effort="1" lower="${-M_PI}" upper="${M_PI}" />
     </joint>
     <!--  Link 2: Shoulder -->
-    <link name="${prefix}_arm1_link">
+    <link name="${prefix}_1_link">
       <visual>
         <origin xyz="0 0 0.0" rpy="0 0 ${M_PI/2}"/>
@@ -95,7 +96,7 @@
     </link>
     <!--  Joint 3: Upper Arm -->
-    <joint name="${prefix}_arm2_joint" type="revolute">
-      <parent link="${prefix}_arm1_link"/>
-      <child link="${prefix}_arm2_link"/>
+    <joint name="${prefix}_2_joint" type="revolute">
+      <parent link="${prefix}_1_link"/>
+      <child link="${prefix}_2_link"/>
       <origin xyz="0.0 0.0 0.05095" rpy="0 0 0"/>
       <axis xyz="0 1 0"/>
@@ -103,5 +104,5 @@
     </joint>
     <!--  Link 3: Upper Arm -->
-    <link name="${prefix}_arm2_link">
+    <link name="${prefix}_2_link">
       <visual>
         <origin xyz="0 0 0" rpy="0 0 ${M_PI/2}"/>
@@ -126,7 +127,7 @@
     </link>
     <!--  Joint 4: Lower Arm -->
-    <joint name="${prefix}_arm3_joint" type="revolute">
-      <parent link="${prefix}_arm2_link"/>
-      <child link="${prefix}_arm3_link"/>
+    <joint name="${prefix}_3_joint" type="revolute">
+      <parent link="${prefix}_2_link"/>
+      <child link="${prefix}_3_link"/>
       <origin xyz="0.022 -0.0 0.128" rpy="0 0 0"/>
       <axis xyz="0 1 0"/>
@@ -134,5 +135,5 @@
     </joint>
     <!--  Link 4: Lower Arm -->
-    <link name="${prefix}_arm3_link">
+    <link name="${prefix}_3_link">
       <visual>
         <origin xyz="0 0 0" rpy="0 0 ${M_PI/2}"/>
@@ -157,7 +158,7 @@
     </link>
     <!--  Joint 5: Forearm Upper -->
-    <joint name="${prefix}_arm4_joint" type="revolute">
-      <parent link="${prefix}_arm3_link"/>
-      <child link="${prefix}_arm4_link"/>
+    <joint name="${prefix}_4_joint" type="revolute">
+      <parent link="${prefix}_3_link"/>
+      <child link="${prefix}_4_link"/>
       <origin xyz="0.0835 0.0 0.0" rpy="0 0 0"/>
       <axis xyz="1 0 0"/>
@@ -165,5 +166,5 @@
     </joint>
     <!--  Link 5: Forearm Upper -->
-    <link name="${prefix}_arm4_link">
+    <link name="${prefix}_4_link">
       <visual>
         <origin xyz="0 0 0" rpy="0 0 ${M_PI/2}"/>
@@ -188,7 +189,7 @@
     </link>
     <!--  Joint 6: Forearm Lower -->
-    <joint name="${prefix}_arm5_joint" type="revolute">
-      <parent link="${prefix}_arm4_link"/>
-      <child link="${prefix}_arm5_link"/>
+    <joint name="${prefix}_5_joint" type="revolute">
+      <parent link="${prefix}_4_link"/>
+      <child link="${prefix}_5_link"/>
       <origin xyz="0.0405 0.0 0.0" rpy="0 0 0"/>
       <axis xyz="0 1 0"/>
@@ -196,5 +197,5 @@
     </joint>
     <!--  Link 6: Forearm Lower -->
-    <link name="${prefix}_arm5_link">
+    <link name="${prefix}_5_link">
       <visual>
         <origin xyz="0 0 0" rpy="0 0 ${M_PI/2}"/>
@@ -219,7 +220,7 @@
     </link>
     <!--  Joint 7: Wrist (Gripper Base) -->
-    <joint name="${prefix}_arm6_joint" type="revolute">
-      <parent link="${prefix}_arm5_link"/>
-      <child link="${prefix}_arm6_link"/>
+    <joint name="${prefix}_6_joint" type="revolute">
+      <parent link="${prefix}_5_link"/>
+      <child link="${prefix}_6_link"/>
       <origin xyz="0.064 0 0.0" rpy="0 0 0"/>
       <axis xyz="1 0 0"/>
@@ -227,5 +228,5 @@
     </joint>
     <!--  Link 7: Wrist (Gripper Base) -->
-    <link name="${prefix}_arm6_link">
+    <link name="${prefix}_6_link">
       <visual>
         <origin xyz="0 0 0" rpy="0 0 ${M_PI/2}"/>
@@ -251,5 +252,5 @@
     <!--  Joint 8: Gripper -->
     <joint name="${prefix}_gripper_joint" type="fixed">
-      <parent link="${prefix}_arm6_link"/>
+      <parent link="${prefix}_6_link"/>
       <child link="${prefix}_gripper_link"/>
       <origin xyz="0.05 0.0 0.0" rpy="0 0 0"/>

File: sobit_light_description/urdf/hand/hand.transmission.xacro (robot description, xacro)
@@ -1,12 +1,7 @@
 <?xml version="1.0" ?>
-<robot xmlns:xacro="http://ros.org/wiki/xacro">
+<robot name="hand_transmission" xmlns:xacro="http://ros.org/wiki/xacro">
   <xacro:macro name="hand_transmission" params="prefix_hand prefix_finger">
-    <position_joint_transmission joint="${prefix_hand}_joint"         reduction="1" />
-    <position_joint_transmission joint="${prefix_hand}_inner_l_joint" reduction="1" />
-    <position_joint_transmission joint="${prefix_hand}_inner_r_joint" reduction="1" />
-    <position_joint_transmission joint="${prefix_hand}_outer_l_joint" reduction="1" />
-    <position_joint_transmission joint="${prefix_hand}_outer_r_joint" reduction="1" />
-    <position_joint_transmission joint="${prefix_hand}_${prefix_finger}_l_joint" reduction="1" />
-    <position_joint_transmission joint="${prefix_hand}_${prefix_finger}_r_joint" reduction="1" />
+    <effort_joint_transmission joint="${prefix_hand}_${prefix_finger}_l_joint" reduction="1" />
+    <effort_joint_transmission joint="${prefix_hand}_${prefix_finger}_r_joint" reduction="1" />
   </xacro:macro>
 </robot>
