Commit message: [UPD] arm and hand urdf (todo: inertia)

File: sobit_light_description/urdf/hand/hand.urdf.xacro (robot description, xacro)
@@ -1,261 +1,209 @@
 <?xml version="1.0" encoding="UTF-8" ?>
 <robot name="hand" xmlns:xacro="http://ros.org/wiki/xacro">
-  <xacro:include filename="$(find sobit_pro_description)/urdf/hand/hand.transmission.xacro" />
+  <xacro:include filename="$(find sobit_light_description)/urdf/hand/hand.transmission.xacro" />
   <xacro:macro name="hand" params="prefix_hand prefix_finger parent">
-    <joint name="${prefix_hand}_base_joint" type="fixed">
-      <parent link="${parent}" />
-      <child link="${prefix_hand}_base_link" />
-      <origin xyz="0.0 0.0 0.0" rpy="0.0 0.0 0.0" />
-    </joint>
-    <link name="${prefix_hand}_base_link">
-      <visual>
-        <origin xyz="0.0 0.0 0.0" rpy="${M_PI/2.0} 0.0 ${M_PI/2.0}" />
-        <geometry>
-          <mesh filename="file://$(find sobit_light_description)/meshes/hand/hand_base.stl" scale="0.001 0.001 0.001" />
-        </geometry>
-        <material name="black" />
-      </visual>
-      <collision>
-        <origin xyz="${0.0215+(0.08251-0.0215)/2} 0.0 ${(0.0415-0.033)/2}" rpy="0.0 0.0 0.0" />
-        <!-- <origin xyz="0.0 0.0 0.0" rpy="${M_PI/2.0} 0.0 ${M_PI/2.0}" /> -->
-        <geometry>
-          <box size="0.06102 0.102 0.0745" />
-          <!-- <mesh filename="file://$(find sobit_light_description)/meshes/hand/hand_base.stl" scale="0.001 0.001 0.001" /> -->
-        </geometry>
-      </collision>
-      <inertial>
-        <origin xyz="${0.0215+(0.08251-0.0215)/2} 0.0 ${(0.0415-0.033)/2}" rpy="0.0 0.0 ${M_PI/2}" />
-        <mass value="0.08" />
-        <inertia ixx="${1/12*0.08*(0.06102**2+0.0745**2)}" ixy="0.0" ixz="0.0"
-                 iyy="${1/12*0.08*(0.102**2  +0.0745**2)}" iyz="0.0"
-                 izz="${1/12*0.08*(0.06102**2+0.102**2)}" />
-        <!-- <inertia ixx="1.0" ixy="0.0" ixz="0.0"
-                 iyy="1.0" iyz="0.0"
-                 izz="1.0" /> -->
-      </inertial>
-    </link>
-    <joint name="${prefix_hand}_joint" type="revolute">
-      <parent link="${prefix_hand}_base_link" />
-      <child link="${prefix_hand}_link" />
-      <origin xyz="0.0631932 -0.0151495 0.0222231" rpy="0.0 0.0 0.0" />
-      <axis xyz="0.0 0.0 1.0" />
-      <limit lower="${-M_PI/2.0}" upper="0" effort="1" velocity="1" />
-    </joint>
-    <link name="${prefix_hand}_link" />
-    <joint name="${prefix_hand}_inner_l_joint" type="revolute">
-      <parent link="${prefix_hand}_base_link" />
-      <child link="${prefix_hand}_inner_l_link" />
-      <origin xyz="0.0631932 0.0151495 0.0372231" rpy="0.0 0.0 0.0" />
-      <axis xyz="0.0 0.0 1.0" />
-      <mimic joint="${prefix_hand}_joint" multiplier="-1.0" offset="0" />
-      <limit lower="${-M_PI/2.0}" upper="0" effort="1" velocity="1" />
-    </joint>
-    <link name="${prefix_hand}_inner_l_link">
-      <visual>
-        <origin xyz="0.0 0.0 0.0" rpy="0.0 0.0 ${M_PI/2.0}" />
-        <geometry>
-          <mesh filename="file://$(find sobit_light_description)/meshes/hand/hand_inner_l.stl" scale="0.001 0.001 0.001" />
-        </geometry>
-        <material name="black" />
-      </visual>
-      <collision>
-        <origin xyz="${0.05408+(0.06006-0.00707)/2} 0.0 -${0.066/2}" rpy="0.0 0.0 0.0" />
-        <!-- <origin xyz="0.0 0.0 0.0" rpy="0.0 0.0 ${M_PI/2.0}" /> -->
-        <geometry>
-          <box size="${0.06006-0.0071} 0.01 0.066" />
-          <!-- <mesh filename="file://$(find sobit_light_description)/meshes/hand/hand_inner_l.stl" scale="0.001 0.001 0.001" /> -->
-        </geometry>
-      </collision>
-      <inertial>
-        <origin xyz="${0.05408+(0.06006-0.00707)/2} 0.0 -${0.066/2}" rpy="0.0 0.0 ${M_PI/2}" />
-        <mass value="0.08" />
-        <inertia ixx="${1/12*0.08*((0.06006-0.0071)**2+0.066**2)}" ixy="0.0" ixz="0.0"
-                 iyy="${1/12*0.08*(0.01**2+0.066**2)}"             iyz="0.0"
-                 izz="${1/12*0.08*((0.06006-0.0071)**2+0.01**2)}" />
-        <!-- <inertia ixx="1.0" ixy="0.0" ixz="0.0"
-                 iyy="1.0" iyz="0.0"
-                 izz="1.0" /> -->
-      </inertial>
-    </link>
-    <joint name="${prefix_hand}_inner_r_joint" type="revolute">
-      <parent link="${prefix_hand}_base_link" />
-      <child link="${prefix_hand}_inner_r_link" />
-      <origin xyz="0.0631932 -0.0151495 0.0372231" rpy="0.0 0.0 0.0" />
-      <axis xyz="0.0 0.0 1.0" />
-      <mimic joint="${prefix_hand}_joint" multiplier="1.0" offset="0" />
-      <limit lower="${-M_PI/2.0}" upper="0" effort="1" velocity="1" />
-    </joint>
-    <link name="${prefix_hand}_inner_r_link">
-      <visual>
-        <origin xyz="0.0 0.0 0.0" rpy="0.0 0.0 ${M_PI/2.0}" />
-        <geometry>
-          <mesh filename="file://$(find sobit_light_description)/meshes/hand/hand_inner_r.stl" scale="0.001 0.001 0.001" />
-        </geometry>
-        <material name="black" />
-      </visual>
-      <collision>
-        <origin xyz="${0.05408+(0.06006-0.00707)/2} 0.0 -${0.066/2}" rpy="0.0 0.0 0.0" />
-        <!-- <origin xyz="0.0 0.0 0.0" rpy="0.0 0.0 ${M_PI/2.0}" /> -->
-        <geometry>
-          <box size="${0.06006-0.0071} 0.01 0.066" />
-          <!-- <mesh filename="file://$(find sobit_light_description)/meshes/hand/hand_inner_r.stl" scale="0.001 0.001 0.001" /> -->
-        </geometry>
-      </collision>
-      <inertial>
-        <origin xyz="${0.05408+(0.06006-0.00707)/2} 0.0 -${0.066/2}" rpy="0.0 0.0 ${M_PI/2}" />
-        <mass value="0.08" />
-        <inertia ixx="${1/12*0.08*((0.06006-0.0071)**2+0.066**2)}" ixy="0.0" ixz="0.0"
-                 iyy="${1/12*0.08*(0.01**2+0.066**2)}"             iyz="0.0"
-                 izz="${1/12*0.08*((0.06006-0.0071)**2+0.01**2)}" />
-        <!-- <inertia ixx="1.0" ixy="0.0" ixz="0.0"
-                 iyy="1.0" iyz="0.0"
-                 izz="1.0" /> -->
-      </inertial>
-    </link>
-    <joint name="${prefix_hand}_outer_l_joint" type="revolute">
-      <!-- <parent link="${prefix_hand}_inner_l_link" /> -->
-      <parent link="${prefix_hand}_base_link" />
-      <child link="${prefix_hand}_outer_l_link" />
-      <!-- <origin xyz="-0.01988747 0.025 -0.01022197" rpy="0.0 0.0 0.0" /> -->
-      <origin xyz="0.043193 0.04015 0.0282231" rpy="0.0 0.0 0.0" />
-      <axis xyz="0.0 0.0 1.0" />
-      <mimic joint="${prefix_hand}_inner_l_joint" multiplier="1.0" offset="0" />
-      <limit lower="${-M_PI/2.0}" upper="0" effort="1" velocity="1" />
-    </joint>
-    <link name="${prefix_hand}_outer_l_link">
-      <visual>
-        <origin xyz="0.0 0.0 0.0" rpy="0.0 0.0 ${M_PI/2.0}" />
-        <geometry>
-          <mesh filename="file://$(find sobit_light_description)/meshes/hand/hand_outer_l.stl" scale="0.001 0.001 0.001" />
-        </geometry>
-        <material name="black" />
-      </visual>
-      <collision>
-        <origin xyz="${0.06123+0.04281/2} 0.0 -${0.056/2}" rpy="0.0 0.0 0.0" />
-        <!-- <origin xyz="0.0 0.0 0.0" rpy="0.0 0.0 ${M_PI/2.0}" /> -->
-        <geometry>
-          <box size="0.04281 0.01 0.056" />
-          <!-- <mesh filename="file://$(find sobit_light_description)/meshes/hand/hand_outer_l.stl" scale="0.001 0.001 0.001" /> -->
-        </geometry>
-      </collision>
-      <inertial>
-        <origin xyz="${0.06123+0.04281/2} 0.0 -${0.056/2}" rpy="0.0 0.0 ${M_PI/2}" />
-        <mass value="0.08" />
-        <inertia ixx="${1/12*0.08*(0.04281**2+0.056**2)}" ixy="0.0" ixz="0.0"
-                 iyy="${1/12*0.08*(0.01**2   +0.056**2)}" iyz="0.0"
-                 izz="${1/12*0.08*(0.04281**2+0.01**2)}" />
-        <!-- <inertia ixx="1.0" ixy="0.0" ixz="0.0"
-                 iyy="1.0" iyz="0.0"
-                 izz="1.0" /> -->
-      </inertial>
-    </link>
-    <joint name="${prefix_hand}_outer_r_joint" type="revolute">
-      <!-- <parent link="${prefix_hand}_inner_r_link" /> -->
-      <parent link="${prefix_hand}_base_link" />
-      <child link="${prefix_hand}_outer_r_link" />
-      <!-- <origin xyz="-0.01988747 -0.025 -0.01022197" rpy="0.0 0.0 0.0" /> -->
-      <origin xyz="0.043193 -0.04015 0.0282231" rpy="0.0 0.0 0.0" />
-      <axis xyz="0.0 0.0 1.0" />
-      <mimic joint="${prefix_hand}_joint" multiplier="1.0" offset="0" />
-      <limit lower="${-M_PI/2.0}" upper="0" effort="1" velocity="1" />
-    </joint>
-    <link name="${prefix_hand}_outer_r_link">
-      <visual>
-        <origin xyz="0.0 0.0 0.0" rpy="0.0 0.0 ${M_PI/2.0}" />
-        <geometry>
-          <mesh filename="file://$(find sobit_light_description)/meshes/hand/hand_outer_r.stl" scale="0.001 0.001 0.001" />
-        </geometry>
-        <material name="black" />
-      </visual>
-      <collision>
-        <origin xyz="${0.06123+0.04281/2} 0.0 -${0.056/2}" rpy="0.0 0.0 0.0" />
-        <!-- <origin xyz="0.0 0.0 0.0" rpy="0.0 0.0 ${M_PI/2.0}" /> -->
-        <geometry>
-          <box size="0.04281 0.01 0.056" />
-          <!-- <mesh filename="file://$(find sobit_light_description)/meshes/hand/hand_outer_r.stl" scale="0.001 0.001 0.001" /> -->
-        </geometry>
-      </collision>
-      <inertial>
-        <origin xyz="${0.06123+0.04281/2} 0.0 -${0.056/2}" rpy="0.0 0.0 ${M_PI/2}" />
-        <mass value="0.08" />
-        <inertia ixx="${1/12*0.08*(0.04281**2+0.056**2)}" ixy="0.0" ixz="0.0"
-                 iyy="${1/12*0.08*(0.01**2   +0.056**2)}" iyz="0.0"
-                 izz="${1/12*0.08*(0.04281**2+0.01**2)}" />
-        <!-- <inertia ixx="1.0" ixy="0.0" ixz="0.0"
-                 iyy="1.0" iyz="0.0"
-                 izz="1.0" /> -->
-      </inertial>
-    </link>
-    <joint name="${prefix_hand}_${prefix_finger}_l_joint" type="revolute">
-      <parent link="${prefix_hand}_inner_l_link" />
-      <child link="${prefix_hand}_${prefix_finger}_l_link" />
-      <origin xyz="0.114316 0.0 -0.027729" rpy="0.0 0.0 0.0" />
-      <axis xyz="0.0 0.0 1.0" />
-      <mimic joint="${prefix_hand}_joint" multiplier="1.0" offset="0" />
-      <limit lower="${-M_PI/2.0}" upper="0" effort="1" velocity="1" />
-    </joint>
-    <link name="${prefix_hand}_${prefix_finger}_l_link">
-      <visual>
-        <origin xyz="-0.029998 0.025 0.0" rpy="0.0 0.0 ${M_PI/2.0}" />
-        <geometry>
-          <mesh filename="file://$(find sobit_light_description)/meshes/hand/hand_finger_l.stl" scale="0.001 0.001 0.001" />
-        </geometry>
-        <material name="black" />
-      </visual>
-      <collision>
-        <origin xyz="${0.007071+(0.012042+0.061128)/2} 0.0 -${0.018/2}" rpy="0.0 0.0 0.0" />
-        <!-- <origin xyz="0.0 0.0 0.0" rpy="0.0 0.0 ${M_PI/2.0}" /> -->
-        <geometry>
-          <box size="${0.012042+0.061128} 0.01137 0.044" />
-          <!-- <mesh filename="file://$(find sobit_light_description)/meshes/hand/hand_finger_l.stl" scale="0.001 0.001 0.001" /> -->
-        </geometry>
-      </collision>
-      <inertial>
-        <origin xyz="${0.007071+(0.012042+0.061128)/2} 0.0 -${0.018/2}" rpy="0.0 0.0 ${M_PI/2}" />
-        <mass value="0.08" />
-        <inertia ixx="${1/12*0.08*((0.012042+0.061128)**2+0.044**2)}" ixy="0.0" ixz="0.0"
-                 iyy="${1/12*0.08*(0.01137**2+0.044**2)}"             iyz="0.0"
-                 izz="${1/12*0.08*((0.012042+0.061128)**2+0.01137**2)}" />
-        <!-- <inertia ixx="1.0" ixy="0.0" ixz="0.0"
-                 iyy="1.0" iyz="0.0"
-                 izz="1.0" /> -->
-      </inertial>
-    </link>
-    <joint name="${prefix_hand}_${prefix_finger}_r_joint" type="revolute">
-      <parent link="${prefix_hand}_inner_r_link" />
-      <child link="${prefix_hand}_${prefix_finger}_r_link" />
-      <origin xyz="0.114316 0.0 -0.027729" rpy="0.0 0.0 0.0" />
-      <axis xyz="0.0 0.0 1.0" />
-      <mimic joint="${prefix_hand}_joint" multiplier="-1.0" offset="0" />
-      <limit lower="${-M_PI/2.0}" upper="0" effort="1" velocity="1" />
-    </joint>
-    <link name="${prefix_hand}_${prefix_finger}_r_link">
-      <visual>
-        <origin xyz="-0.029998 -0.025 0.0" rpy="0.0 0.0 ${M_PI/2.0}" />
-        <geometry>
-          <mesh filename="file://$(find sobit_light_description)/meshes/hand/hand_finger_r.stl" scale="0.001 0.001 0.001" />
-        </geometry>
-        <material name="black" />
-      </visual>
-      <collision>
-        <origin xyz="${0.007071+(0.012042+0.061128)/2} 0.0 -${0.018/2}" rpy="0.0 0.0 0.0" />
-        <!-- <origin xyz="0.0 0.0 0.0" rpy="0.0 0.0 ${M_PI/2.0}" /> -->
-        <geometry>
-          <box size="${0.012042+0.061128} 0.01137 0.044" />
-          <!-- <mesh filename="file://$(find sobit_light_description)/meshes/hand/hand_finger_r.stl" scale="0.001 0.001 0.001" /> -->
-        </geometry>
-      </collision>
-      <inertial>
-        <origin xyz="${0.007071+(0.012042+0.061128)/2} 0.0 -${0.018/2}" rpy="0.0 0.0 ${M_PI/2}" />
-        <mass value="0.08" />
-        <inertia ixx="${1/12*0.08*((0.012042+0.061128)**2+0.044**2)}"   ixy="0.0" ixz="0.0"
-                 iyy="${1/12*0.08*(0.01137**2+0.044**2)}"               iyz="0.0"
-                 izz="${1/12*0.08*((0.012042+0.061128)**2+0.01137**2)}" />
-        <!-- <inertia ixx="1.0" ixy="0.0" ixz="0.0"
-                 iyy="1.0" iyz="0.0"
-                 izz="1.0" /> -->
-      </inertial>
-    </link>
-    <xacro:hand_transmission prefix_hand="${prefix_hand}" prefix_finger="${prefix_finger}" />
+    <!--  Joint 9: Gripper left sub -->
+    <joint name="${prefix_hand}_l_sub_joint" type="fixed">
+      <parent link="${parent}"/>
+      <child link="${prefix_hand}_l_sub_link"/>
+      <origin xyz="0.009 0.015 0.0" rpy="0 0 0"/>
+    </joint>
+    <!--  Link 9: Gripper left sub -->
+    <link name="${prefix_hand}_l_sub_link">
+      <visual>
+        <origin xyz="0 0 0" rpy="0 0 ${M_PI/2}"/>
+        <geometry>
+          <mesh filename="file://$(find sobit_light_description)/meshes/hand/omx1_link9-10_gripper.stl" scale="0.001 0.001 0.001"/>
+        </geometry>
+        <material name="grey"/>
+      </visual>
+      <collision>
+        <origin xyz="0 0 0" rpy="0 0 ${M_PI/2}"/>
+        <geometry>
+          <mesh filename="file://$(find sobit_light_description)/meshes/hand/omx1_link9-10_gripper.stl" scale="0.001 0.001 0.001"/>
+        </geometry>
+      </collision>
+      <inertial>
+        <origin xyz="0 0 0" rpy="0 0 ${M_PI/2}"/>
+        <mass value="0.2" />
+        <inertia ixx="1.0" ixy="0.0" ixz="1.0"
+                 iyy="1.0" iyz="0.0"
+                 izz="1.0" />
+      </inertial>
+    </link>
+    <!--  Joint 10: Gripper right sub -->
+    <joint name="${prefix_hand}_r_sub_joint" type="fixed">
+      <parent link="${parent}"/>
+      <child link="${prefix_hand}_r_sub_link"/>
+      <origin xyz="0.009 -0.015 0.0" rpy="0 0 0"/>
+    </joint>
+    <!--  Link 10: Gripper right sub -->
+    <link name="${prefix_hand}_r_sub_link">
+      <visual>
+        <origin xyz="0 0 0" rpy="0 ${M_PI} ${M_PI/2}"/>
+        <geometry>
+          <mesh filename="file://$(find sobit_light_description)/meshes/hand/omx1_link9-10_gripper.stl" scale="0.001 0.001 0.001"/>
+        </geometry>
+        <material name="grey"/>
+      </visual>
+      <collision>
+        <origin xyz="0 0 0" rpy="0 ${M_PI} ${M_PI/2}"/>
+        <geometry>
+          <mesh filename="file://$(find sobit_light_description)/meshes/hand/omx1_link9-10_gripper.stl" scale="0.001 0.001 0.001"/>
+        </geometry>
+      </collision>
+      <inertial>
+        <origin xyz="0 0 0" rpy="0 ${M_PI} ${M_PI/2}"/>
+        <mass value="0.2" />
+        <inertia ixx="1.0" ixy="0.0" ixz="1.0"
+                 iyy="1.0" iyz="0.0"
+                 izz="1.0" />
+      </inertial>
+    </link>
+    <!--  Joint 11: Gripper Finger Left -->
+    <joint name="${prefix_hand}_l_${prefix_finger}_joint" type="prismatic">
+      <parent link="${prefix_hand}_l_sub_link"/>
+      <child link="${prefix_hand}_l_${prefix_finger}_link"/>
+      <origin xyz="0.0 0.04 0.0" rpy="0 0 0"/>
+      <axis xyz="0 1 0"/>
+      <limit velocity="4.8" effort="1" lower="${-0.055+0.02675}" upper="0.0" />
+    </joint>
+    <!--  Link 11: Gripper Finger Left -->
+    <link name="${prefix_hand}_l_${prefix_finger}_link">
+      <visual>
+        <origin xyz="0.0 0.0 0" rpy="0 0 ${M_PI/2}"/>
+        <geometry>
+          <mesh filename="file://$(find sobit_light_description)/meshes/hand/omx1_link11-12_finger.stl" scale="0.001 0.001 0.001"/>
+        </geometry>
+        <material name="grey"/>
+      </visual>
+      <collision>
+        <origin xyz="0.0 0.0 0" rpy="0 0 ${M_PI/2}"/>
+        <geometry>
+          <mesh filename="file://$(find sobit_light_description)/meshes/hand/omx1_link11-12_finger.stl" scale="0.001 0.001 0.001"/>
+        </geometry>
+      </collision>
+      <inertial>
+        <origin xyz="0.0 0.0 0" rpy="0 0 ${M_PI/2}"/>
+        <mass value="0.2" />
+        <inertia ixx="1.0" ixy="0.0" ixz="1.0"
+                 iyy="1.0" iyz="0.0"
+                 izz="1.0" />
+      </inertial>
+    </link>
+    <!--  Joint 12: Gripper Finger Right -->
+    <joint name="${prefix_hand}_r_${prefix_finger}_joint" type="prismatic">
+      <parent link="${prefix_hand}_r_sub_link"/>
+      <child link="${prefix_hand}_r_${prefix_finger}_link"/>
+      <origin xyz="0.0 -0.04 0.0" rpy="0 0 0"/>
+      <axis xyz="0 -1 0"/>
+      <limit velocity="4.8" effort="1" lower="0.0" upper="${-0.055+0.02675}" />
+      <mimic joint="${prefix_hand}_l_${prefix_finger}_joint" multiplier="1"/>
+    </joint>
+    <!--  Link 12: Gripper Finger Right -->
+    <link name="${prefix_hand}_r_${prefix_finger}_link">
+      <visual>
+        <origin xyz="0.0 -0.0 0" rpy="0 ${M_PI} ${M_PI/2}"/>
+        <geometry>
+          <mesh filename="file://$(find sobit_light_description)/meshes/hand/omx1_link11-12_finger.stl" scale="0.001 0.001 0.001"/>
+        </geometry>
+        <material name="grey"/>
+      </visual>
+      <collision>
+        <origin xyz="0.0 -0.0 0" rpy="0 ${M_PI} ${M_PI/2}"/>
+        <geometry>
+          <mesh filename="file://$(find sobit_light_description)/meshes/hand/omx1_link11-12_finger.stl" scale="0.001 0.001 0.001"/>
+        </geometry>
+      </collision>
+      <inertial>
+        <origin xyz="0.0 -0.0 0" rpy="0 ${M_PI} ${M_PI/2}"/>
+        <mass value="0.2" />
+        <inertia ixx="1.0" ixy="0.0" ixz="1.0"
+                 iyy="1.0" iyz="0.0"
+                 izz="1.0" />
+      </inertial>
+    </link>
+    <!--  Joint 13: Gripper Tip Left -->
+    <joint name="${prefix_hand}_l_tip_joint" type="fixed">
+      <parent link="${prefix_hand}_l_${prefix_finger}_link"/>
+      <child link="${prefix_hand}_l_tip_link"/>
+      <origin xyz="${0.0345+0.0375/2} -0.0145 0.0" rpy="0 0 0"/>
+    </joint>
+    <!--  Link 13: Gripper Tip Left -->
+    <link name="${prefix_hand}_l_tip_link">
+      <visual>
+        <origin xyz="0.0 -0.0 0" rpy="0 0 ${M_PI/2}"/>
+        <geometry>
+          <mesh filename="file://$(find sobit_light_description)/meshes/hand/omx1_link13-14_finger.stl" scale="0.001 0.001 0.001"/>
+        </geometry>
+        <material name="grey"/>
+      </visual>
+      <collision>
+        <origin xyz="0.0 -0.0 0" rpy="0 0 ${M_PI/2}"/>
+        <geometry>
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