Commit message: [ADD] inertia for each joint

File: sobit_light_description/urdf/arm/arm.urdf.xacro (robot description, xacro)
@@ -19,18 +19,16 @@
         <material name="grey"/>
       </visual>
-      <!-- TODO: Collision with simple geometry -->
-      <collision>
-        <origin xyz="0 0 0" rpy="0 0 ${M_PI/2}"/>
-        <geometry>
-          <mesh filename="file://$(find sobit_light_description)/meshes/arm/omx1_link_base.stl" scale="0.001 0.001 0.001"/>
-        </geometry>
-      </collision>
-      <!-- TODO: Inertial with simple geometry -->
-      <inertial>
-        <origin xyz="0 0 0" rpy="0 0 ${M_PI/2}"/>
-        <mass value="0.2" />
-        <inertia ixx="1.0" ixy="0.0" ixz="1.0"
-                iyy="1.0" iyz="0.0"
-                izz="1.0" />
+      <collision>
+        <origin xyz="${0.005-0.1/2} 0.0 ${-0.0156+0.0686/2}" rpy="0 0 0"/>
+        <geometry>
+          <box size="0.1000 0.1200 0.0686"/>
+        </geometry>
+      </collision>
+      <inertial>
+        <origin xyz="${0.005-0.1/2} 0.0 ${-0.0156+0.0686/2}" rpy="0 0 0"/>
+        <mass value="0.336" />
+        <inertia  ixx="${1/12*0.336*(0.1000**2+0.0686**2)}" ixy="0.0" ixz="0.0"
+                  iyy="${1/12*0.336*(0.1200**2+0.0686**2)}" iyz="0.0"
+                  izz="${1/12*0.336*(0.1000**2+0.1200**2)}" />
       </inertial>
     </link>
@@ -51,15 +49,15 @@
       </visual>
       <collision>
-        <origin xyz="0 0 0" rpy="0 0 ${M_PI/2}"/>
-        <geometry>
-          <mesh filename="file://$(find sobit_light_description)/meshes/arm/omx1_link1.stl" scale="0.001 0.001 0.001"/>
-        </geometry>
-      </collision>
-      <inertial>
-        <origin xyz="0 0 0" rpy="0 0 ${M_PI/2}"/>
-        <mass value="0.2" />
-        <inertia ixx="1.0" ixy="0.0" ixz="1.0"
-                iyy="1.0" iyz="0.0"
-                izz="1.0" />
+        <origin xyz="0.0 0.0 ${0.0585/2}" rpy="0 0 0"/>
+        <geometry>
+          <box size="0.0440 0.0335 0.0585"/>
+        </geometry>
+      </collision>
+      <inertial>
+        <origin xyz="0.0 0.0 ${0.0585/2}" rpy="0 0 0"/>
+        <mass value="0.205" />
+        <inertia  ixx="${1/12*0.205*(0.0440**2+0.0585**2)}" ixy="0.0" ixz="0.0"
+                  iyy="${1/12*0.205*(0.0335**2+0.0585**2)}" iyz="0.0"
+                  izz="${1/12*0.205*(0.0440**2+0.0335**2)}" />
       </inertial>
     </link>
@@ -82,15 +80,15 @@
       </visual>
       <collision>
-        <origin xyz="0 0 0.0" rpy="0 0 ${M_PI/2}"/>
-        <geometry>
-          <mesh filename="file://$(find sobit_light_description)/meshes/arm/omx1_link2.stl" scale="0.001 0.001 0.001"/>
-        </geometry>
-      </collision>
-      <inertial>
-        <origin xyz="0 0 0.0" rpy="0 0 ${M_PI/2}"/>
-        <mass value="0.2" />
-        <inertia ixx="1.0" ixy="0.0" ixz="1.0"
-                iyy="1.0" iyz="0.0"
-                izz="1.0" />
+        <origin xyz="0.0 0.0 ${0.0647/2}" rpy="0 0 0"/>
+        <geometry>
+          <box size="0.0335 0.1130 0.0647"/>
+        </geometry>
+      </collision>
+      <inertial>
+        <origin xyz="0.0 0.0 ${0.0647/2}" rpy="0 0 0"/>
+        <mass value="0.392" />
+        <inertia  ixx="${1/12*0.392*(0.0335**2+0.0647**2)}" ixy="0.0" ixz="0.0"
+                  iyy="${1/12*0.392*(0.1130**2+0.0647**2)}" iyz="0.0"
+                  izz="${1/12*0.392*(0.0335**2+0.1130**2)}" />
       </inertial>
     </link>
@@ -113,15 +111,15 @@
       </visual>
       <collision>
-        <origin xyz="0 0 0" rpy="0 0 ${M_PI/2}"/>
-        <geometry>
-          <mesh filename="file://$(find sobit_light_description)/meshes/arm/omx1_link3.stl" scale="0.001 0.001 0.001"/>
-        </geometry>
-      </collision>
-      <inertial>
-        <origin xyz="0 0 0" rpy="0 0 ${M_PI/2}"/>
-        <mass value="0.2" />
-        <inertia ixx="1.0" ixy="0.0" ixz="1.0"
-                iyy="1.0" iyz="0.0"
-                izz="1.0" />
+        <origin xyz="${0.03575-0.0585/2} 0.0 ${-0.016+(0.14475+0.016)/2}" rpy="0 0 0"/>
+        <geometry>
+          <box size="0.0585 0.0440 ${0.14475+0.016}"/>
+        </geometry>
+      </collision>
+      <inertial>
+        <origin xyz="${0.03575-0.0585/2} 0.0 ${-0.016+(0.14475+0.016)/2}" rpy="0 0 0"/>
+        <mass value="0.261" />
+        <inertia  ixx="${1/12*0.261*(0.0585**2+(0.14475+0.016)**2)}" ixy="0.0" ixz="0.0"
+                  iyy="${1/12*0.261*(0.0440**2+(0.14475+0.016)**2)}" iyz="0.0"
+                  izz="${1/12*0.261*(0.0585**2+0.0440**2)}" />
       </inertial>
     </link>
@@ -144,15 +142,15 @@
       </visual>
       <collision>
-        <origin xyz="0 0 0" rpy="0 0 ${M_PI/2}"/>
-        <geometry>
-          <mesh filename="file://$(find sobit_light_description)/meshes/arm/omx1_link4.stl" scale="0.001 0.001 0.001"/>
-        </geometry>
-      </collision>
-      <inertial>
-        <origin xyz="0 0 0" rpy="0 0 ${M_PI/2}"/>
-        <mass value="0.2" />
-        <inertia ixx="1.0" ixy="0.0" ixz="1.0"
-                iyy="1.0" iyz="0.0"
-                izz="1.0" />
+        <origin xyz="${0.0835-0.0860/2} 0.0 ${0.03525-0.04875/2}" rpy="0 0 0"/>
+        <geometry>
+          <box size="0.0860 0.0530 0.04875"/>
+        </geometry>
+      </collision>
+      <inertial>
+        <origin xyz="${0.0835-0.0860/2} 0.0 ${0.03525-0.04875/2}" rpy="0 0 0"/>
+        <mass value="0.157" />
+        <inertia  ixx="${1/12*0.157*(0.0860**2+0.04875**2)}" ixy="0.0" ixz="0.0"
+                  iyy="${1/12*0.157*(0.0530**2+0.04875**2)}" iyz="0.0"
+                  izz="${1/12*0.157*(0.0860**2+0.0530**2)}" />
       </inertial>
     </link>
@@ -175,15 +173,15 @@
       </visual>
       <collision>
-        <origin xyz="0 0 0" rpy="0 0 ${M_PI/2}"/>
-        <geometry>
-          <mesh filename="file://$(find sobit_light_description)/meshes/arm/omx1_link5.stl" scale="0.001 0.001 0.001"/>
-        </geometry>
-      </collision>
-      <inertial>
-        <origin xyz="0 0 0" rpy="0 0 ${M_PI/2}"/>
-        <mass value="0.2" />
-        <inertia ixx="1.0" ixy="0.0" ixz="1.0"
-                iyy="1.0" iyz="0.0"
-                izz="1.0" />
+        <origin xyz="${0.05175/2} 0.0 0.0" rpy="0 0 0"/>
+        <geometry>
+          <box size="0.05175 0.03700 0.0285"/>
+        </geometry>
+      </collision>
+      <inertial>
+        <origin xyz="${0.05175/2} 0.0 0.0" rpy="0 0 0"/>
+        <mass value="0.093" />
+        <inertia  ixx="${1/12*0.093*(0.05175**2+0.0285**2)}" ixy="0.0" ixz="0.0"
+                  iyy="${1/12*0.093*(0.03700**2+0.0285**2)}" iyz="0.0"
+                  izz="${1/12*0.093*(0.05175**2+0.0370**2)}" />
       </inertial>
     </link>
@@ -206,18 +204,18 @@
       </visual>
       <collision>
-        <origin xyz="0 0 0" rpy="0 0 ${M_PI/2}"/>
-        <geometry>
-          <mesh filename="file://$(find sobit_light_description)/meshes/arm/omx1_link6.stl" scale="0.001 0.001 0.001"/>
-        </geometry>
-      </collision>
-      <inertial>
-        <origin xyz="0 0 0" rpy="0 0 ${M_PI/2}"/>
-        <mass value="0.2" />
-        <inertia ixx="1.0" ixy="0.0" ixz="1.0"
-                iyy="1.0" iyz="0.0"
-                izz="1.0" />
-      </inertial>
-    </link>
-    <!--  Joint 7: Wrist (Gripper Base) -->
+        <origin xyz="${0.064-0.0665/2} 0.0 ${0.03525-0.0465/2}" rpy="0 0 0"/>
+        <geometry>
+          <box size="0.0665 0.0410 0.0465"/>
+        </geometry>
+      </collision>
+      <inertial>
+        <origin xyz="${0.064-0.0665/2} 0.0 ${0.03525-0.0465/2}" rpy="0 0 0"/>
+        <mass value="0.106" />
+        <inertia  ixx="${1/12*0.106*(0.0665**2+0.0465**2)}" ixy="0.0" ixz="0.0"
+                  iyy="${1/12*0.106*(0.0410**2+0.0465**2)}" iyz="0.0"
+                  izz="${1/12*0.106*(0.0665**2+0.0410**2)}" />
+      </inertial>
+    </link>
+    <!--  Joint 7: Wrist (Hand Base) -->
     <joint name="${prefix}_6_joint" type="revolute">
       <parent link="${prefix}_5_link"/>
@@ -227,54 +225,54 @@
       <limit velocity="4.8" effort="1" lower="${-M_PI}" upper="${M_PI}" />
     </joint>
-    <!--  Link 7: Wrist (Gripper Base) -->
+    <!--  Link 7: Wrist (Hand Base) -->
     <link name="${prefix}_6_link">
       <visual>
         <origin xyz="0 0 0" rpy="0 0 ${M_PI/2}"/>
         <geometry>
-          <mesh filename="file://$(find sobit_light_description)/meshes/arm/omx1_link7_gripper_base.stl" scale="0.001 0.001 0.001"/>
-        </geometry>
-        <material name="grey"/>
-      </visual>
-      <collision>
-        <origin xyz="0 0 0" rpy="0 0 ${M_PI/2}"/>
-        <geometry>
-          <mesh filename="file://$(find sobit_light_description)/meshes/arm/omx1_link7_gripper_base.stl" scale="0.001 0.001 0.001"/>
-        </geometry>
-      </collision>
-      <inertial>
-        <origin xyz="0 0 0" rpy="0 0 ${M_PI/2}"/>
-        <mass value="0.2" />
-        <inertia ixx="1.0" ixy="0.0" ixz="1.0"
-                iyy="1.0" iyz="0.0"
-                izz="1.0" />
-      </inertial>
-    </link>
-    <!--  Joint 8: Gripper -->
-    <joint name="${prefix}_gripper_joint" type="fixed">
+          <mesh filename="file://$(find sobit_light_description)/meshes/arm/omx1_link7_hand_base.stl" scale="0.001 0.001 0.001"/>
+        </geometry>
+        <material name="grey"/>
+      </visual>
+      <collision>
+        <origin xyz="${0.0505/2} 0.0 ${0.03775-0.0495/2}" rpy="0 0 0"/>
+        <geometry>
+          <box size="0.0505 0.0335 0.0495"/>
+        </geometry>
+      </collision>
+      <inertial>
+        <origin xyz="${0.0505/2} 0.0 ${0.03775-0.0495/2}" rpy="0 0 0"/>
+        <mass value="0.134" />
+        <inertia  ixx="${1/12*0.134*(0.0505**2+0.0495**2)}" ixy="0.0" ixz="0.0"
+                  iyy="${1/12*0.134*(0.0335**2+0.0495**2)}" iyz="0.0"
+                  izz="${1/12*0.134*(0.0505**2+0.0335**2)}" />
+      </inertial>
+    </link>
+    <!--  Joint 8: Hand -->
+    <joint name="${prefix}_hand_joint" type="fixed">
       <parent link="${prefix}_6_link"/>
-      <child link="${prefix}_gripper_link"/>
+      <child link="${prefix}_hand_link"/>
       <origin xyz="0.05 0.0 0.0" rpy="0 0 0"/>
     </joint>
-    <!--  Link 8: Gripper -->
-    <link name="${prefix}_gripper_link">
-      <visual>
-        <origin xyz="0 0 0" rpy="0 0 ${M_PI/2}"/>
-        <geometry>
-          <mesh filename="file://$(find sobit_light_description)/meshes/arm/omx1_link8_gripper.stl" scale="0.001 0.001 0.001"/>
-        </geometry>
-        <material name="grey"/>
-      </visual>
-      <collision>
-        <origin xyz="0 0 0" rpy="0 0 ${M_PI/2}"/>
-        <geometry>
-          <mesh filename="file://$(find sobit_light_description)/meshes/arm/omx1_link8_gripper.stl" scale="0.001 0.001 0.001"/>
-        </geometry>
-      </collision>
-      <inertial>
-        <origin xyz="0 0 0" rpy="0 0 ${M_PI/2}"/>
-        <mass value="0.2" />
-        <inertia ixx="1.0" ixy="0.0" ixz="1.0"
-                iyy="1.0" iyz="0.0"
-                izz="1.0" />
+    <!--  Link 8: Hand -->
+    <link name="${prefix}_hand_link">
+      <visual>
+        <origin xyz="0 0 0" rpy="0 0 ${M_PI/2}"/>
+        <geometry>
+          <mesh filename="file://$(find sobit_light_description)/meshes/arm/omx1_link8_hand.stl" scale="0.001 0.001 0.001"/>
+        </geometry>
+        <material name="grey"/>
+      </visual>
+      <collision>
+        <origin xyz="${0.008/2} 0.0 0.0" rpy="0 ${M_PI/2} 0"/>
+        <geometry>
+          <cylinder radius="0.011" length="0.008"/>
+        </geometry>
+      </collision>
+      <inertial>
+        <origin xyz="${0.008/2} 0.0 0.0" rpy="0 ${M_PI/2} 0"/>
+        <mass value="0.003" />
+        <inertia  ixx="${1/12*0.003*(3*0.011**2+0.008**2)}" ixy="0.0" ixz="0.0"
+                  iyy="${1/12*0.003*(3*0.011**2+0.008**2)}" iyz="0.0"
+                  izz="${1/12*0.003*(3*0.011**2+0.008**2)}" />
       </inertial>
     </link>

File: sobit_light_description/urdf/back/back.urdf.xacro (robot description, xacro)
@@ -16,20 +16,15 @@
       </visual>
       <collision>
-        <origin xyz="0.0 0.0 ${0.517/2}" rpy="0.0 0.0 0.0" />
-        <!-- <origin xyz="0.0 0.0 0.0" rpy="0.0 0.0 ${M_PI}" /> -->
+        <origin xyz="0.0 0.0 ${0.60/2}" rpy="0 0 0"/>
         <geometry>
-          <box size="0.02 0.02 0.517"/>
-          <!-- <mesh filename="file://$(find sobit_light_description)/meshes/back/back_base.stl" scale="0.001 0.001 0.001" /> -->
+          <box size="0.02 0.02 0.60"/>
         </geometry>
       </collision>
       <inertial>
-        <origin xyz="0.0 0.0 ${0.517/2}" rpy="0.0 0.0 0.0" />
-        <mass value="0.5" />
-        <inertia ixx="${1/12*0.5*(0.02**2+0.517**2)}" ixy="0.0" ixz="0.0"
-                 iyy="${1/12*0.5*(0.02**2+0.517**2)}" iyz="0.0"
-                 izz="${1/12*0.5*(0.02**2+0.02**2)}" />
-        <!-- <inertia ixx="1.0" ixy="0.0" ixz="0.0"
-                 iyy="1.0" iyz="0.0"
-                 izz="1.0" /> -->
+        <origin xyz="0.0 0.0 ${0.60/2}" rpy="0 0 0"/>
+        <mass value="1.212" />
+        <inertia  ixx="${1/12*1.212*(0.02**2+0.60**2)}" ixy="0.0" ixz="0.0"
+                  iyy="${1/12*1.212*(0.02**2+0.60**2)}" iyz="0.0"
+                  izz="${1/12*1.212*(0.02**2+0.02**2)}" />
       </inertial>
     </link>

File: sobit_light_description/urdf/base/base.urdf.xacro (robot description, xacro)
@@ -16,5 +16,5 @@
         <material name="body" />
       </visual>
-      <collision>
+      <!-- <collision>
         <origin xyz="0.0435 0.0 0.0475"
                 rpy="0 0 0" />
@@ -23,5 +23,5 @@
         </geometry>
         <material name="body" />
-      </collision>
+      </collision> -->
       <inertial>
         <mass value="6.4" />

File: sobit_light_description/urdf/base/plate.urdf.xacro (robot description, xacro)
@@ -16,20 +16,15 @@
       </visual>
       <collision>
-        <origin xyz="0.0 0.0 -${0.009/2}" rpy="0.0 0.0 ${M_PI/2}" />
-        <!-- <origin xyz="0.0 0.0 0.0" rpy="0.0 0.0 0.0" /> -->
+        <origin xyz="0.0 0.0 -${0.1408/2}" rpy="0 0 0"/>
         <geometry>
-          <box size="0.3 0.3 0.009" />
-          <!-- <mesh filename="file://$(find sobit_light_description)/meshes/body/plate_bottom.stl" scale="0.001 0.001 0.001" /> -->
+          <box size="0.320 0.375 0.1408"/>
         </geometry>
       </collision>
       <inertial>
-        <origin xyz="0.0 0.0 -${0.009/2}" rpy="0.0 0.0 ${M_PI/2}" />
-        <mass value="0.08" />
-        <inertia ixx="${1/12*0.08*(0.3**2+0.009**2)}" ixy="0.0" ixz="0.0"
-                 iyy="${1/12*0.08*(0.3**2+0.009**2)}" iyz="0.0"
-                 izz="${1/12*0.08*(0.3**2+0.3**2)}" />
-        <!-- <inertia ixx="1.0" ixy="0.0" ixz="0.0"
-                 iyy="1.0" iyz="0.0"
-                 izz="1.0" /> -->
+        <origin xyz="0.0 0.0 -${0.1408/2}" rpy="0 0 0"/>
+        <mass value="2.343" />
+        <inertia  ixx="${1/12*2.343*(0.320**2+0.1408**2)}" ixy="0.0" ixz="0.0"
+                  iyy="${1/12*2.343*(0.375**2+0.1408**2)}" iyz="0.0"
+                  izz="${1/12*2.343*(0.320**2+0.375**2)}" />
       </inertial>
     </link>
@@ -48,20 +43,15 @@
       </visual>
       <collision>
-        <origin xyz="0.0 0.0 -${0.009/2}" rpy="0.0 0.0 ${M_PI/2}" />
-        <!-- <origin xyz="0.0 0.0 0.0" rpy="0.0 0.0 0.0" /> -->
+        <origin xyz="0.0 0.0 -${0.11875/2}" rpy="0 0 0"/>
         <geometry>
-          <box size="0.3 0.3 0.009" />
-          <!-- <mesh filename="file://$(find sobit_light_description)/meshes/body/plate_middle.stl" scale="0.001 0.001 0.001" /> -->
+          <box size="0.244 0.300 0.11875"/>
         </geometry>
       </collision>
       <inertial>
-        <origin xyz="0.0 0.0 -${0.009/2}" rpy="0.0 0.0 ${M_PI/2}" />
-        <mass value="0.08" />
-        <inertia ixx="${1/12*0.08*(0.3**2+0.009**2)}" ixy="0.0" ixz="0.0"
-                 iyy="${1/12*0.08*(0.3**2+0.009**2)}" iyz="0.0"
-                 izz="${1/12*0.08*(0.3**2+0.3**2)}" />
-        <!-- <inertia ixx="1.0" ixy="0.0" ixz="0.0"
-                 iyy="1.0" iyz="0.0"
-                 izz="1.0" /> -->
+        <origin xyz="0.0 0.0 -${0.11875/2}" rpy="0 0 0"/>
+        <mass value="1.255" />
+        <inertia  ixx="${1/12*1.255*(0.244**2+0.11875**2)}" ixy="0.0" ixz="0.0"
+                  iyy="${1/12*1.255*(0.300**2+0.11875**2)}" iyz="0.0"
+                  izz="${1/12*1.255*(0.244**2+0.300**2)}" />
       </inertial>
     </link>
