Commit message: [ADD] inertia for each joint

File: sobit_light_description/urdf/hand/hand.urdf.xacro (robot description, xacro)
@@ -3,72 +3,72 @@
   <xacro:include filename="$(find sobit_light_description)/urdf/hand/hand.transmission.xacro" />
   <xacro:macro name="hand" params="prefix_hand prefix_finger parent">
-    <!--  Joint 9: Gripper left sub -->
-    <joint name="${prefix_hand}_l_sub_joint" type="fixed">
+    <!--  Joint 9: Hand left sub -->
+    <joint name="${prefix_hand}_sub_l_joint" type="fixed">
       <parent link="${parent}"/>
-      <child link="${prefix_hand}_l_sub_link"/>
+      <child link="${prefix_hand}_sub_l_link"/>
       <origin xyz="0.009 0.015 0.0" rpy="0 0 0"/>
     </joint>
-    <!--  Link 9: Gripper left sub -->
-    <link name="${prefix_hand}_l_sub_link">
+    <!--  Link 9: Hand left sub -->
+    <link name="${prefix_hand}_sub_l_link">
       <visual>
         <origin xyz="0 0 0" rpy="0 0 ${M_PI/2}"/>
         <geometry>
-          <mesh filename="file://$(find sobit_light_description)/meshes/hand/omx1_link9-10_gripper.stl" scale="0.001 0.001 0.001"/>
-        </geometry>
-        <material name="grey"/>
-      </visual>
-      <collision>
-        <origin xyz="0 0 0" rpy="0 0 ${M_PI/2}"/>
-        <geometry>
-          <mesh filename="file://$(find sobit_light_description)/meshes/hand/omx1_link9-10_gripper.stl" scale="0.001 0.001 0.001"/>
-        </geometry>
-      </collision>
-      <inertial>
-        <origin xyz="0 0 0" rpy="0 0 ${M_PI/2}"/>
-        <mass value="0.2" />
-        <inertia ixx="1.0" ixy="0.0" ixz="1.0"
-                 iyy="1.0" iyz="0.0"
-                 izz="1.0" />
-      </inertial>
-    </link>
-    <!--  Joint 10: Gripper right sub -->
-    <joint name="${prefix_hand}_r_sub_joint" type="fixed">
+          <mesh filename="file://$(find sobit_light_description)/meshes/hand/omx1_link9-10_hand.stl" scale="0.001 0.001 0.001"/>
+        </geometry>
+        <material name="grey"/>
+      </visual>
+      <collision>
+        <origin xyz="${0.0035/2} ${0.04/2} 0.0" rpy="0 0 0"/>
+        <geometry>
+          <box size="0.0035 0.0520 0.0120"/>
+        </geometry>
+      </collision>
+      <inertial>
+        <origin xyz="${0.0035/2} ${0.04/2} 0.0" rpy="0 0 0"/>
+        <mass value="0.002" />
+        <inertia  ixx="${1/12*0.002*(0.0035**2+0.0120**2)}" ixy="0.0" ixz="0.0"
+                  iyy="${1/12*0.002*(0.0520**2+0.0120**2)}" iyz="0.0"
+                  izz="${1/12*0.002*(0.0035**2+0.0520**2)}" />
+      </inertial>
+    </link>
+    <!--  Joint 10: Hand right sub -->
+    <joint name="${prefix_hand}_sub_r_joint" type="fixed">
       <parent link="${parent}"/>
-      <child link="${prefix_hand}_r_sub_link"/>
+      <child link="${prefix_hand}_sub_r_link"/>
       <origin xyz="0.009 -0.015 0.0" rpy="0 0 0"/>
     </joint>
-    <!--  Link 10: Gripper right sub -->
-    <link name="${prefix_hand}_r_sub_link">
+    <!--  Link 10: Hand right sub -->
+    <link name="${prefix_hand}_sub_r_link">
       <visual>
         <origin xyz="0 0 0" rpy="0 ${M_PI} ${M_PI/2}"/>
         <geometry>
-          <mesh filename="file://$(find sobit_light_description)/meshes/hand/omx1_link9-10_gripper.stl" scale="0.001 0.001 0.001"/>
-        </geometry>
-        <material name="grey"/>
-      </visual>
-      <collision>
-        <origin xyz="0 0 0" rpy="0 ${M_PI} ${M_PI/2}"/>
-        <geometry>
-          <mesh filename="file://$(find sobit_light_description)/meshes/hand/omx1_link9-10_gripper.stl" scale="0.001 0.001 0.001"/>
-        </geometry>
-      </collision>
-      <inertial>
-        <origin xyz="0 0 0" rpy="0 ${M_PI} ${M_PI/2}"/>
-        <mass value="0.2" />
-        <inertia ixx="1.0" ixy="0.0" ixz="1.0"
-                 iyy="1.0" iyz="0.0"
-                 izz="1.0" />
-      </inertial>
-    </link>
-    <!--  Joint 11: Gripper Finger Left -->
-    <joint name="${prefix_hand}_l_${prefix_finger}_joint" type="prismatic">
-      <parent link="${prefix_hand}_l_sub_link"/>
-      <child link="${prefix_hand}_l_${prefix_finger}_link"/>
+          <mesh filename="file://$(find sobit_light_description)/meshes/hand/omx1_link9-10_hand.stl" scale="0.001 0.001 0.001"/>
+        </geometry>
+        <material name="grey"/>
+      </visual>
+      <collision>
+        <origin xyz="${0.0035/2} -${0.04/2} 0.0" rpy="0 0 0"/>
+        <geometry>
+          <box size="0.0035 0.0520 0.0120"/>
+        </geometry>
+      </collision>
+      <inertial>
+        <origin xyz="${0.0035/2} -${0.04/2} 0.0" rpy="0 0 0"/>
+        <mass value="0.002" />
+        <inertia  ixx="${1/12*0.002*(0.0035**2+0.0120**2)}" ixy="0.0" ixz="0.0"
+                  iyy="${1/12*0.002*(0.0520**2+0.0120**2)}" iyz="0.0"
+                  izz="${1/12*0.002*(0.0035**2+0.0520**2)}" />
+      </inertial>
+    </link>
+    <!--  Joint 11: Hand Finger Left -->
+    <joint name="${prefix_hand}_${prefix_finger}_l_joint" type="prismatic">
+      <parent link="${prefix_hand}_sub_l_link"/>
+      <child link="${prefix_hand}_${prefix_finger}_l_link"/>
       <origin xyz="0.0 0.04 0.0" rpy="0 0 0"/>
       <axis xyz="0 1 0"/>
       <limit velocity="4.8" effort="1" lower="${-0.055+0.02675}" upper="0.0" />
     </joint>
-    <!--  Link 11: Gripper Finger Left -->
-    <link name="${prefix_hand}_l_${prefix_finger}_link">
+    <!--  Link 11: Hand Finger Left -->
+    <link name="${prefix_hand}_${prefix_finger}_l_link">
       <visual>
         <origin xyz="0.0 0.0 0" rpy="0 0 ${M_PI/2}"/>
@@ -79,28 +79,28 @@
       </visual>
       <collision>
-        <origin xyz="0.0 0.0 0" rpy="0 0 ${M_PI/2}"/>
-        <geometry>
-          <mesh filename="file://$(find sobit_light_description)/meshes/hand/omx1_link11-12_finger.stl" scale="0.001 0.001 0.001"/>
-        </geometry>
-      </collision>
-      <inertial>
-        <origin xyz="0.0 0.0 0" rpy="0 0 ${M_PI/2}"/>
-        <mass value="0.2" />
-        <inertia ixx="1.0" ixy="0.0" ixz="1.0"
-                 iyy="1.0" iyz="0.0"
-                 izz="1.0" />
-      </inertial>
-    </link>
-    <!--  Joint 12: Gripper Finger Right -->
-    <joint name="${prefix_hand}_r_${prefix_finger}_joint" type="prismatic">
-      <parent link="${prefix_hand}_r_sub_link"/>
-      <child link="${prefix_hand}_r_${prefix_finger}_link"/>
+        <origin xyz="${0.0056+0.068/2} -${0.009+0.008/2} 0.0" rpy="0 0 0"/>
+        <geometry>
+          <box size="0.068 0.008 0.034"/>
+        </geometry>
+      </collision>
+      <inertial>
+        <origin xyz="${0.0056+0.068/2} -${0.009+0.008/2} 0.0" rpy="0 0 0"/>
+        <mass value="0.032" />
+        <inertia  ixx="${1/12*0.032*(0.068**2+0.034**2)}" ixy="0.0" ixz="0.0"
+                  iyy="${1/12*0.032*(0.008**2+0.034**2)}" iyz="0.0"
+                  izz="${1/12*0.032*(0.068**2+0.008**2)}" />
+      </inertial>
+    </link>
+    <!--  Joint 12: Hand Finger Right -->
+    <joint name="${prefix_hand}_${prefix_finger}_r_joint" type="prismatic">
+      <parent link="${prefix_hand}_sub_r_link"/>
+      <child link="${prefix_hand}_${prefix_finger}_r_link"/>
       <origin xyz="0.0 -0.04 0.0" rpy="0 0 0"/>
       <axis xyz="0 -1 0"/>
       <limit velocity="4.8" effort="1" lower="0.0" upper="${-0.055+0.02675}" />
-      <mimic joint="${prefix_hand}_l_${prefix_finger}_joint" multiplier="1"/>
-    </joint>
-    <!--  Link 12: Gripper Finger Right -->
-    <link name="${prefix_hand}_r_${prefix_finger}_link">
+      <mimic joint="${prefix_hand}_${prefix_finger}_l_joint" multiplier="1"/>
+    </joint>
+    <!--  Link 12: Hand Finger Right -->
+    <link name="${prefix_hand}_${prefix_finger}_r_link">
       <visual>
         <origin xyz="0.0 -0.0 0" rpy="0 ${M_PI} ${M_PI/2}"/>
@@ -111,28 +111,57 @@
       </visual>
       <collision>
+        <origin xyz="${0.0056+0.068/2} ${0.009+0.008/2} 0.0" rpy="0 0 0"/>
+        <geometry>
+          <box size="0.068 0.008 0.034"/>
+        </geometry>
+      </collision>
+      <inertial>
+        <origin xyz="${0.0056+0.068/2} ${0.009+0.008/2} 0.0" rpy="0 0 0"/>
+        <mass value="0.032" />
+        <inertia  ixx="${1/12*0.032*(0.068**2+0.034**2)}" ixy="0.0" ixz="0.0"
+                  iyy="${1/12*0.032*(0.008**2+0.034**2)}" iyz="0.0"
+                  izz="${1/12*0.032*(0.068**2+0.008**2)}" />
+      </inertial>
+    </link>
+    <!--  Joint 13: Hand Tip Left -->
+    <joint name="${prefix_hand}_${prefix_finger}_tip_l_joint" type="fixed">
+      <parent link="${prefix_hand}_${prefix_finger}_l_link"/>
+      <child link="${prefix_hand}_${prefix_finger}_tip_l_link"/>
+      <origin xyz="${0.0345+0.0375/2} -0.0145 0.0" rpy="0 0 0"/>
+    </joint>
+    <!--  Link 13: Hand Tip Left -->
+    <link name="${prefix_hand}_${prefix_finger}_tip_l_link">
+      <visual>
+        <origin xyz="0.0 -0.0 0" rpy="0 0 ${M_PI/2}"/>
+        <geometry>
+          <mesh filename="file://$(find sobit_light_description)/meshes/hand/omx1_link13-14_finger.stl" scale="0.001 0.001 0.001"/>
+        </geometry>
+        <material name="grey"/>
+      </visual>
+      <collision>
+        <origin xyz="0.0 -${0.0031/2} 0.0" rpy="0 0 0"/>
+        <geometry>
+          <box size="0.0370 0.0031 0.015"/>
+        </geometry>
+      </collision>
+      <inertial>
+        <origin xyz="0.0 -${0.0031/2} 0.0" rpy="0 0 0"/>
+        <mass value="0.002" />
+        <inertia  ixx="${1/12*0.002*(0.0370**2+0.015**2)}" ixy="0.0" ixz="0.0"
+                  iyy="${1/12*0.002*(0.0031**2+0.015**2)}" iyz="0.0"
+                  izz="${1/12*0.002*(0.0370**2+0.0031**2)}" />
+      </inertial>
+    </link>
+    <!--  Joint 14: Hand Tip Right -->
+    <joint name="${prefix_hand}_${prefix_finger}_tip_r_joint" type="fixed">
+      <parent link="${prefix_hand}_${prefix_finger}_r_link"/>
+      <child link="${prefix_hand}_${prefix_finger}_tip_r_link"/>
+      <origin xyz="${0.0345+0.0375/2} 0.0145 0.0" rpy="0 0 0"/>
+    </joint>
+    <!--  Link 14: Hand Tip Right -->
+    <link name="${prefix_hand}_${prefix_finger}_tip_r_link">
+      <visual>
         <origin xyz="0.0 -0.0 0" rpy="0 ${M_PI} ${M_PI/2}"/>
         <geometry>
-          <mesh filename="file://$(find sobit_light_description)/meshes/hand/omx1_link11-12_finger.stl" scale="0.001 0.001 0.001"/>
-        </geometry>
-      </collision>
-      <inertial>
-        <origin xyz="0.0 -0.0 0" rpy="0 ${M_PI} ${M_PI/2}"/>
-        <mass value="0.2" />
-        <inertia ixx="1.0" ixy="0.0" ixz="1.0"
-                 iyy="1.0" iyz="0.0"
-                 izz="1.0" />
-      </inertial>
-    </link>
-    <!--  Joint 13: Gripper Tip Left -->
-    <joint name="${prefix_hand}_l_tip_joint" type="fixed">
-      <parent link="${prefix_hand}_l_${prefix_finger}_link"/>
-      <child link="${prefix_hand}_l_tip_link"/>
-      <origin xyz="${0.0345+0.0375/2} -0.0145 0.0" rpy="0 0 0"/>
-    </joint>
-    <!--  Link 13: Gripper Tip Left -->
-    <link name="${prefix_hand}_l_tip_link">
-      <visual>
-        <origin xyz="0.0 -0.0 0" rpy="0 0 ${M_PI/2}"/>
-        <geometry>
           <mesh filename="file://$(find sobit_light_description)/meshes/hand/omx1_link13-14_finger.stl" scale="0.001 0.001 0.001"/>
         </geometry>
@@ -140,44 +169,15 @@
       </visual>
       <collision>
-        <origin xyz="0.0 -0.0 0" rpy="0 0 ${M_PI/2}"/>
-        <geometry>
-          <mesh filename="file://$(find sobit_light_description)/meshes/hand/omx1_link13-14_finger.stl" scale="0.001 0.001 0.001"/>
-        </geometry>
-      </collision>
-      <inertial>
-        <origin xyz="0.0 -0.0 0" rpy="0 0 ${M_PI/2}"/>
-        <mass value="0.2" />
-        <inertia ixx="1.0" ixy="0.0" ixz="1.0"
-                iyy="1.0" iyz="0.0"
-                izz="1.0" />
-      </inertial>
-    </link>
-    <!--  Joint 14: Gripper Tip Right -->
-    <joint name="${prefix_hand}_r_tip_joint" type="fixed">
-      <parent link="${prefix_hand}_r_${prefix_finger}_link"/>
-      <child link="${prefix_hand}_r_tip_link"/>
-      <origin xyz="${0.0345+0.0375/2} 0.0145 0.0" rpy="0 0 0"/>
-    </joint>
-    <!--  Link 14: Gripper Tip Right -->
-    <link name="${prefix_hand}_r_tip_link">
-      <visual>
-        <origin xyz="0.0 -0.0 0" rpy="0 ${M_PI} ${M_PI/2}"/>
-        <geometry>
-          <mesh filename="file://$(find sobit_light_description)/meshes/hand/omx1_link13-14_finger.stl" scale="0.001 0.001 0.001"/>
-        </geometry>
-        <material name="grey"/>
-      </visual>
-      <collision>
-        <origin xyz="0.0 -0.0 0" rpy="0 ${M_PI} ${M_PI/2}"/>
-        <geometry>
-          <mesh filename="file://$(find sobit_light_description)/meshes/hand/omx1_link13-14_finger.stl" scale="0.001 0.001 0.001"/>
-        </geometry>
-      </collision>
-      <inertial>
-        <origin xyz="0.0 -0.0 0" rpy="0 ${M_PI} ${M_PI/2}"/>
-        <mass value="0.2" />
-        <inertia ixx="1.0" ixy="0.0" ixz="1.0"
-                 iyy="1.0" iyz="0.0"
-                 izz="1.0" />
+        <origin xyz="0.0 ${0.0031/2} 0.0" rpy="0 0 0"/>
+        <geometry>
+          <box size="0.0370 0.0031 0.015"/>
+        </geometry>
+      </collision>
+      <inertial>
+        <origin xyz="0.0 ${0.0031/2} 0.0" rpy="0 0 0"/>
+        <mass value="0.002" />
+        <inertia  ixx="${1/12*0.002*(0.0370**2+0.015**2)}" ixy="0.0" ixz="0.0"
+                  iyy="${1/12*0.002*(0.0031**2+0.015**2)}" iyz="0.0"
+                  izz="${1/12*0.002*(0.0370**2+0.0031**2)}" />
       </inertial>
     </link>
@@ -191,5 +191,5 @@
     <link name="${prefix_hand}_end_effector_link">
       <visual>
-        <origin xyz="0 0 0" rpy="0 0 0"/>
+        <origin xyz="0.0 0.0 0.0" rpy="0 0 0"/>
         <geometry>
           <box size="0.01 0.01 0.01" />
@@ -198,9 +198,9 @@
       </visual>
       <inertial>
-        <origin xyz="0 0 0" />
-        <mass value="0.2" />
-        <inertia ixx="1.0" ixy="0.0" ixz="1.0"
-                 iyy="1.0" iyz="0.0"
-                 izz="1.0" />
+        <origin xyz="0.0 0.0 0.0" rpy="0 0 0"/>
+        <mass value="0.0001" />
+        <inertia  ixx="${1/12*0.0001*(0.01**2+0.01**2)}" ixy="0.0" ixz="0.0"
+                  iyy="${1/12*0.0001*(0.01**2+0.01**2)}" iyz="0.0"
+                  izz="${1/12*0.0001*(0.01**2+0.01**2)}" />
       </inertial>
     </link>

File: sobit_light_description/urdf/head/head.urdf.xacro (robot description, xacro)
@@ -20,20 +20,15 @@
       </visual>
       <collision>
-        <origin xyz="${0.05125-0.15125/2} 0.0 0.0" rpy="0.0 0.0 0.0" />
-        <!-- <origin xyz="0.0 0.0 0.0" rpy="${M_PI/2.0} 0.0 ${M_PI/2.0}" /> -->
+        <origin xyz="0.0 0.0 ${0.039-0.069/2}" rpy="0 0 0"/>
         <geometry>
-          <box size="0.15125 0.0285 0.044"/>
-          <!-- <mesh filename="file://$(find sobit_light_description)/meshes/head/head_camera_base.stl" scale="0.001 0.001 0.001" /> -->
+          <box size="0.0565 0.0385 0.0690"/>
         </geometry>
       </collision>
       <inertial>
-        <origin xyz="${0.05125-0.15125/2} 0.0 0.0" rpy="0.0 0.0 0.0" />
-        <mass value="0.08" />
-        <inertia ixx="${1/12*0.08*(0.15125**2+0.044**2)}" ixy="0.0" ixz="0.0"
-                 iyy="${1/12*0.08*(0.0285**2 +0.044**2)}" iyz="0.0"
-                 izz="${1/12*0.08*(0.15125**2+0.0285**2)}" />
-        <!-- <inertia ixx="1.0" ixy="0.0" ixz="0.0"
-                 iyy="1.0" iyz="0.0"
-                 izz="1.0" /> -->
+        <origin xyz="0.0 0.0 ${0.039-0.069/2}" rpy="0 0 0"/>
+        <mass value="0.145" />
+        <inertia  ixx="${1/12*0.145*(0.0565**2+0.0690**2)}" ixy="0.0" ixz="0.0"
+                  iyy="${1/12*0.145*(0.0385**2+0.0690**2)}" iyz="0.0"
+                  izz="${1/12*0.145*(0.0565**2+0.0385**2)}" />
       </inertial>
     </link>
@@ -58,20 +53,15 @@
       </visual>
       <collision>
-        <origin xyz="0.0 0.0 ${0.00525+0.03525/2}" rpy="0.0 0.0 0.0" />
-        <!-- <origin xyz="0.0 0.0 0.0" rpy="0.0 0.0 ${M_PI/2.0}" /> -->
+        <origin xyz="0.0 0.0 ${0.05175/2}" rpy="0 0 0"/>
         <geometry>
-          <box size="0.0285 0.037 0.03525"/>
-          <!-- <mesh filename="file://$(find sobit_light_description)/meshes/head/head_camera_pan.stl" scale="0.001 0.001 0.001" /> -->
+          <box size="0.0285 0.0370 0.05175"/>
         </geometry>
       </collision>
       <inertial>
-        <origin xyz="0.0 0.0 ${0.00525+0.03525/2}" rpy="0.0 0.0 ${M_PI/2}" />
-        <mass value="0.08" />
-        <inertia ixx="${1/12*0.08*(0.0285**2+0.03525**2)}" ixy="0.0" ixz="0.0"
-                 iyy="${1/12*0.08*(0.037**2 +0.03525**2)}" iyz="0.0"
-                 izz="${1/12*0.08*(0.0285**2+0.037**2)}" />
-        <!-- <inertia ixx="1.0" ixy="0.0" ixz="0.0"
-                 iyy="1.0" iyz="0.0"
-                 izz="1.0" /> -->
+        <origin xyz="0.0 0.0 ${0.05175/2}" rpy="0 0 0"/>
+        <mass value="0.089" />
+        <inertia  ixx="${1/12*0.089*(0.0285**2+0.05175**2)}" ixy="0.0" ixz="0.0"
+                  iyy="${1/12*0.089*(0.0370**2+0.05175**2)}" iyz="0.0"
+                  izz="${1/12*0.089*(0.0285**2+0.0370**2)}" />
       </inertial>
     </link>
@@ -96,20 +86,15 @@
       </visual>
       <collision>
-        <origin xyz="0.0 0.0 ${0.028+0.0115/2}" rpy="0.0 0.0 0.0" />
-        <!-- <origin xyz="0.0 0.0 0.0" rpy="0.0 0.0 ${M_PI/2.0}" /> -->
+        <origin xyz="${0.0725-0.150/2} 0.0 ${0.028+0.1275/2}" rpy="0 0 0"/>
         <geometry>
-          <box size="0.046 0.0466 0.0115"/>
-          <!-- <mesh filename="file://$(find sobit_light_description)/meshes/head/head_camera_tilt.stl" scale="0.001 0.001 0.001" /> -->
+          <box size="0.150 0.200 0.1275"/>
         </geometry>
       </collision>
       <inertial>
-        <origin xyz="0.0 0.0 ${0.028+0.0115/2}" rpy="0.0 0.0 0.0" />
-        <mass value="0.08" />
-        <inertia ixx="${1/12*0.08*(0.046**2 +0.0115**2)}" ixy="0.0" ixz="0.0"
-                 iyy="${1/12*0.08*(0.0466**2+0.0115**2)}" iyz="0.0"
-                 izz="${1/12*0.08*(0.046**2 +0.0466**2)}" />
-        <!-- <inertia ixx="1.0" ixy="0.0" ixz="0.0"
-                 iyy="1.0" iyz="0.0"
-                 izz="1.0" /> -->
+        <origin xyz="${0.0725-0.150/2} 0.0 ${0.028+0.1275/2}" rpy="0 0 0"/>
+        <mass value="0.904" />
+        <inertia  ixx="${1/12*0.904*(0.150**2+0.1275**2)}" ixy="0.0" ixz="0.0"
+                  iyy="${1/12*0.904*(0.200**2+0.1275**2)}" iyz="0.0"
+                  izz="${1/12*0.904*(0.150**2+0.200**2)}" />
       </inertial>
     </link>

File: sobit_light_description/urdf/sensor/speaker.urdf.xacro (robot description, xacro)
@@ -16,16 +16,15 @@
       </visual>
       <collision>
-        <origin xyz="0.0 0.0 0.0" rpy="0.0 0.0 ${M_PI/2.0}" />
+        <origin xyz="${0.037025/2} 0.0 0.0" rpy="0 ${M_PI/2-M_PI/9.0} 0"/>
         <geometry>
-          <mesh filename="file://$(find sobit_light_description)/meshes/sensor/speaker.stl" scale="0.001 0.001 0.001" />
+          <cylinder radius="0.065" length="0.037025"/>
         </geometry>
-        <material name="black" />
       </collision>
       <inertial>
-        <origin xyz="0.0 0.0 0.0" rpy="0.0 0.0 ${M_PI/2.0}" />
-        <mass value="0.09507172" />
-        <inertia ixx="${1/12*0.09507172*(0.078**2 + 0.157**2)}" ixy="0.0" ixz="0.0"
-                 iyy="${1/12*0.09507172*(0.026**2 + 0.078**2)}" iyz="0.0"
-                 izz="${1/12*0.09507172*(0.026**2 + 0.157**2)}" />
+        <origin xyz="${0.037025/2} 0.0 0.0" rpy="0 ${M_PI/2-M_PI/9.0} 0"/>
+        <mass value="0.298" />
+        <inertia  ixx="${1/12*0.298*(3*0.065**2+0.037025**2)}" ixy="0.0" ixz="0.0"
+                  iyy="${1/12*0.298*(3*0.065**2+0.037025**2)}" iyz="0.0"
+                  izz="${1/12*0.298*(3*0.065**2+0.037025**2)}" />
       </inertial>
     </link>

Commit message: [TEMP] add bigger effort

File: sobit_light_description/urdf/arm/arm.urdf.xacro (robot description, xacro)
@@ -68,5 +68,5 @@
       <origin xyz="0.0 0.0 0.0465" rpy="0 ${M_PI/2} 0"/>
       <axis xyz="0 0 1"/>
-      <limit velocity="4.8" effort="1" lower="${-M_PI}" upper="${M_PI}" />
+      <limit velocity="4.8" effort="25" lower="${-M_PI}" upper="${M_PI}" />
     </joint>
     <!--  Act 1: Shoulder Roll -->
@@ -99,5 +99,5 @@
       <origin xyz="0.0 0.0 0.05095" rpy="0 0 0"/>
       <axis xyz="0 1 0"/>
-      <limit velocity="4.8" effort="1" lower="${-M_PI/2}" upper="${M_PI/2}" />
+      <limit velocity="4.8" effort="25" lower="${-M_PI/2}" upper="${M_PI/2}" />
     </joint>
     <!--  Act 2: Shoulder Pitch (right) -->
@@ -130,5 +130,5 @@
       <origin xyz="0.0 0.0 0.05095" rpy="0 0 0"/>
       <axis xyz="0 1 0"/>
-      <limit velocity="4.8" effort="1" lower="${-M_PI/2}" upper="${M_PI/2}" />
+      <limit velocity="4.8" effort="25" lower="${-M_PI/2}" upper="${M_PI/2}" />
       <mimic joint="${prefix}_shoulder_pitch_joint" multiplier="-1" offset="0"/>
     </joint>
@@ -162,5 +162,5 @@
       <origin xyz="0.022 -0.0 0.128" rpy="0 0 0"/>
       <axis xyz="0 1 0"/>
-      <limit velocity="4.8" effort="1" lower="${-M_PI/2}" upper="${M_PI/2}" />
+      <limit velocity="4.8" effort="25" lower="${-M_PI/2}" upper="${M_PI/2}" />
     </joint>
     <!--  Act 4: Elbow Pitch -->
@@ -193,5 +193,5 @@
       <origin xyz="0.0835 0.0 0.0" rpy="0 0 0"/>
       <axis xyz="1 0 0"/>
-      <limit velocity="4.8" effort="1" lower="${-M_PI}" upper="${M_PI}" />
+      <limit velocity="4.8" effort="25" lower="${-M_PI}" upper="${M_PI}" />
     </joint>
     <!--  Act 5: Forearm Roll -->
@@ -224,5 +224,5 @@
       <origin xyz="0.0405 0.0 0.0" rpy="0 0 0"/>
       <axis xyz="0 1 0"/>
-      <limit velocity="4.8" effort="1" lower="${-M_PI/2}" upper="${M_PI/2}" />
+      <limit velocity="4.8" effort="25" lower="${-M_PI/2}" upper="${M_PI/2}" />
     </joint>
     <!--  Act 6: Wrist Pitch -->
@@ -255,5 +255,5 @@
       <origin xyz="0.064 0 0.0" rpy="0 0 0"/>
       <axis xyz="1 0 0"/>
-      <limit velocity="4.8" effort="1" lower="${-M_PI}" upper="${M_PI}" />
+      <limit velocity="4.8" effort="25" lower="${-M_PI}" upper="${M_PI}" />
     </joint>
     <!--  Act 7: Wrist Roll -->

Commit message: [FIX] no longer mimic

File: sobit_light_description/urdf/arm/arm.urdf.xacro (robot description, xacro)
@@ -131,5 +131,5 @@
       <axis xyz="0 1 0"/>
       <limit velocity="4.8" effort="25" lower="${-M_PI/2}" upper="${M_PI/2}" />
-      <mimic joint="${prefix}_shoulder_pitch_joint" multiplier="-1" offset="0"/>
+      <!-- <mimic joint="${prefix}_shoulder_pitch_joint" multiplier="-1" offset="0"/> -->
     </joint>
     <!--  Act 3: Shoulder Pitch (left) -->
