Commit message: [FIX] new model position

File: sobit_light_description/urdf/arm/arm.urdf.xacro (robot description, xacro)
@@ -256,5 +256,5 @@
         <origin xyz="${0.0505/2} 0.0 ${0.03775-0.0495/2}" rpy="0 0 0"/>
         <geometry>
-          <box size="0.0505 0.0335 0.0495"/>
+          <box size="0.0505 0.1886 0.0495"/>
         </geometry>
       </collision>
@@ -267,33 +267,4 @@
       </inertial>
     </link>
-    <!--  Joint - Hand Base -->
-    <joint name="${prefix}_hand_joint" type="fixed">
-      <parent link="${prefix}_wrist_roll_link"/>
-      <child link="${prefix}_hand_link"/>
-      <origin xyz="0.05 0.0 0.0" rpy="0 0 0"/>
-    </joint>
-    <!--  Link - Hand Base -->
-    <link name="${prefix}_hand_link">
-      <visual>
-        <origin xyz="0 0 0" rpy="0 0 ${M_PI/2}"/>
-        <geometry>
-          <mesh filename="file://$(find sobit_light_description)/meshes/arm/omx1_link8_hand.stl" scale="0.001 0.001 0.001"/>
-        </geometry>
-        <material name="black"/>
-      </visual>
-      <collision>
-        <origin xyz="${0.008/2} 0.0 0.0" rpy="0 ${M_PI/2} 0"/>
-        <geometry>
-          <cylinder radius="0.011" length="0.008"/>
-        </geometry>
-      </collision>
-      <inertial>
-        <origin xyz="${0.008/2} 0.0 0.0" rpy="0 ${M_PI/2} 0"/>
-        <mass value="0.003" />
-        <inertia  ixx="${1/12*0.003*(3*0.011**2+0.008**2)}" ixy="0.0" ixz="0.0"
-                  iyy="${1/12*0.003*(3*0.011**2+0.008**2)}" iyz="0.0"
-                  izz="${1/12*0.003*(3*0.011**2+0.008**2)}" />
-      </inertial>
-    </link>
     <xacro:arm_transmission prefix="${prefix}" />
   </xacro:macro>

File: sobit_light_description/urdf/hand/hand.urdf.xacro (robot description, xacro)
@@ -3,62 +3,4 @@
   <xacro:include filename="$(find sobit_light_description)/urdf/hand/hand.transmission.xacro" />
   <xacro:macro name="hand" params="prefix_hand prefix_finger parent">
-    <!--  Joint - Hand left sub -->
-    <joint name="${prefix_hand}_sub_l_joint" type="fixed">
-      <parent link="${parent}"/>
-      <child link="${prefix_hand}_sub_l_link"/>
-      <origin xyz="0.009 0.015 0.0" rpy="0 0 0"/>
-    </joint>
-    <!--  Link - Hand left sub -->
-    <link name="${prefix_hand}_sub_l_link">
-      <visual>
-        <origin xyz="0 0 0" rpy="0 0 ${M_PI/2}"/>
-        <geometry>
-          <mesh filename="file://$(find sobit_light_description)/meshes/hand/omx1_link9-10_hand.stl" scale="0.001 0.001 0.001"/>
-        </geometry>
-        <material name="black"/>
-      </visual>
-      <collision>
-        <origin xyz="${0.0035/2} ${0.04/2} 0.0" rpy="0 0 0"/>
-        <geometry>
-          <box size="0.0035 0.0520 0.0120"/>
-        </geometry>
-      </collision>
-      <inertial>
-        <origin xyz="${0.0035/2} ${0.04/2} 0.0" rpy="0 0 0"/>
-        <mass value="0.002" />
-        <inertia  ixx="${1/12*0.002*(0.0035**2+0.0120**2)}" ixy="0.0" ixz="0.0"
-                  iyy="${1/12*0.002*(0.0520**2+0.0120**2)}" iyz="0.0"
-                  izz="${1/12*0.002*(0.0035**2+0.0520**2)}" />
-      </inertial>
-    </link>
-    <!--  Joint - Hand right sub -->
-    <joint name="${prefix_hand}_sub_r_joint" type="fixed">
-      <parent link="${parent}"/>
-      <child link="${prefix_hand}_sub_r_link"/>
-      <origin xyz="0.009 -0.015 0.0" rpy="0 0 0"/>
-    </joint>
-    <!--  Link - Hand right sub -->
-    <link name="${prefix_hand}_sub_r_link">
-      <visual>
-        <origin xyz="0 0 0" rpy="0 ${M_PI} ${M_PI/2}"/>
-        <geometry>
-          <mesh filename="file://$(find sobit_light_description)/meshes/hand/omx1_link9-10_hand.stl" scale="0.001 0.001 0.001"/>
-        </geometry>
-        <material name="black"/>
-      </visual>
-      <collision>
-        <origin xyz="${0.0035/2} -${0.04/2} 0.0" rpy="0 0 0"/>
-        <geometry>
-          <box size="0.0035 0.0520 0.0120"/>
-        </geometry>
-      </collision>
-      <inertial>
-        <origin xyz="${0.0035/2} -${0.04/2} 0.0" rpy="0 0 0"/>
-        <mass value="0.002" />
-        <inertia  ixx="${1/12*0.002*(0.0035**2+0.0120**2)}" ixy="0.0" ixz="0.0"
-                  iyy="${1/12*0.002*(0.0520**2+0.0120**2)}" iyz="0.0"
-                  izz="${1/12*0.002*(0.0035**2+0.0520**2)}" />
-      </inertial>
-    </link>
     <!--  Act 8 - Hand Finger (left) -->
     <joint name="${prefix_hand}_joint" type="prismatic">
@@ -66,17 +8,14 @@
       <parent link="${parent}"/>
       <child link="${prefix_hand}_link"/>
-      <!-- <origin xyz="0.0 0.04 0.0" rpy="0 0 0"/> -->
-      <origin xyz="0.0093 0.021 0.0" rpy="0 0 0"/>
+      <origin xyz="0.059 0.05498805 0.0" rpy="0 0 0"/>
       <axis xyz="0 1 0"/>
-      <limit velocity="4.8" effort="1" lower="-0.01" upper="0.019" />
+      <limit velocity="4.8" effort="1" lower="-0.01791787" upper="0.02901195" />
     </joint>
     <!--  Act 8 - Hand Finger (left) -->
     <link name="${prefix_hand}_link">
       <visual>
-        <!-- <origin xyz="0.0 0.0 0.0" rpy="0 0 ${M_PI/2}"/> -->
-        <origin xyz="0.0 0.0 0.0" rpy="0 0 0"/>
+        <origin xyz="0.0 0.0 0.0" rpy="0 0 ${M_PI/2}"/>
         <geometry>
-          <!-- <mesh filename="file://$(find sobit_light_description)/meshes/hand/omx1_link11-12_finger.stl" scale="0.001 0.001 0.001"/> -->
-          <mesh filename="file://$(find sobit_light_description)/meshes/hand/omx1_link11-12_finger_new.stl" scale="0.001 0.001 0.001"/>
+          <mesh filename="file://$(find sobit_light_description)/meshes/hand/omx1_link11-12_finger.stl" scale="0.001 0.001 0.001"/>
         </geometry>
         <material name="black"/>
@@ -98,9 +37,7 @@
     <!--  Act 8 - Hand Finger (right) -->
     <joint name="${prefix_hand}_sub_joint" type="prismatic">
-      <!-- <parent link="${prefix_hand}_sub_r_link"/> -->
       <parent link="${parent}"/>
       <child link="${prefix_hand}_sub_link"/>
-      <!-- <origin xyz="0.0 -0.04 0.0" rpy="0 0 0"/> -->
-      <origin xyz="0.0093 -0.021 0.0" rpy="0 0 0"/>
+      <origin xyz="0.059 -0.05498805 0.0" rpy="0 0 0"/>
       <axis xyz="0 -1 0"/>
       <limit velocity="4.8" effort="1" lower="-1.57" upper="1.57"/>
@@ -110,9 +47,7 @@
     <link name="${prefix_hand}_sub_link">
       <visual>
-        <!-- <origin xyz="0.0 0.0 0.0" rpy="0 ${M_PI} ${M_PI/2}"/> -->
-        <origin xyz="0.0 0.0 0.0" rpy="${M_PI} 0 0"/>
+        <origin xyz="0.0 0.0 0.0" rpy="0 ${M_PI} ${M_PI/2}"/>
         <geometry>
-          <!-- <mesh filename="file://$(find sobit_light_description)/meshes/hand/omx1_link11-12_finger.stl" scale="0.001 0.001 0.001"/> -->
-          <mesh filename="file://$(find sobit_light_description)/meshes/hand/omx1_link11-12_finger_new.stl" scale="0.001 0.001 0.001"/>
+          <mesh filename="file://$(find sobit_light_description)/meshes/hand/omx1_link11-12_finger.stl" scale="0.001 0.001 0.001"/>
         </geometry>
         <material name="black"/>
@@ -193,5 +128,5 @@
     <joint name="end_effector_joint" type="fixed">
       <origin xyz="${0.0935+0.0375/2} 0.0 0.0" rpy="0 0 0"/>
-      <parent link="arm_wrist_roll_link"/>
+      <parent link="${parent}"/>
       <child link="${prefix_hand}_end_effector_link"/>
     </joint>

File: sobit_light_description/urdf/sensor/camera_hand.urdf.xacro (robot description, xacro)
@@ -5,5 +5,5 @@
     <!-- Joint - Hand Camera Base -->
     <joint name="${prefix}_base_joint" type="fixed">
-      <origin xyz="0.03685 0.0 0.0438" rpy="0 0 0"/>
+      <origin xyz="0.03341 0.0 0.0504366" rpy="0 ${25*M_PI/180} 0"/>
       <parent link="${parent}"/>
       <child link="${prefix}_base_link"/>
@@ -33,5 +33,5 @@
     </link>
     <xacro:sensor_d405 parent="${prefix}_base_link" name="${prefix}" use_nominal_extrinsics="true" >
-      <origin xyz="0.0 0.0 0.0" rpy="0.0 0.0 0.0" />
+      <origin xyz="0.0 0.0 0.0" rpy="0 0 0" />
     </xacro:sensor_d405>
   </xacro:macro>

Commit message: [UPD] mimic joint for shoulder pitch (dynamixel hardware update)

File: sobit_light_description/urdf/arm/arm.urdf.xacro (robot description, xacro)
@@ -131,5 +131,5 @@
       <axis xyz="0 1 0"/>
       <limit velocity="4.8" effort="25" lower="${-M_PI/2}" upper="${M_PI/2}" />
-      <!-- <mimic joint="${prefix}_shoulder_pitch_joint" multiplier="-1" offset="0"/> -->
+      <mimic joint="${prefix}_shoulder_pitch_joint" multiplier="-1" offset="0"/>
     </joint>
     <!--  Act 3 - Shoulder Pitch (left) -->

Commit message: [UPD] rotation direction for sub joint

File: sobit_light_description/urdf/arm/arm.urdf.xacro (robot description, xacro)
@@ -129,6 +129,6 @@
       <child link="${prefix}_shoulder_pitch_sub_link"/>
       <origin xyz="0.0 0.0 0.05095" rpy="0 0 0"/>
-      <axis xyz="0 1 0"/>
-      <limit velocity="4.8" effort="25" lower="${-M_PI/2}" upper="${M_PI/2}" />
+      <axis xyz="0 -1 0"/>
+      <limit velocity="4.8" effort="25" lower="${-M_PI}" upper="${M_PI}" />
       <mimic joint="${prefix}_shoulder_pitch_joint" multiplier="-1" offset="0"/>
     </joint>

Commit message: [ADD] moveit_config

File: sobit_light_description/urdf/arm/arm.urdf.xacro (robot description, xacro)
@@ -66,5 +66,5 @@
       <parent link="${prefix}_base_link"/>
       <child link="${prefix}_shoulder_roll_link"/>
-      <origin xyz="0.0 0.0 0.0465" rpy="0 ${M_PI/2} 0"/>
+      <origin xyz="0.02495 0.0 0.0465" rpy="0 ${M_PI/2} 0"/>
       <axis xyz="0 0 1"/>
       <limit velocity="4.8" effort="25" lower="${-M_PI}" upper="${M_PI}" />

Commit message: Update shoulder roll joint origin calculation
Arm shoulder was colliding with base

File: sobit_light_description/urdf/arm/arm.urdf.xacro (robot description, xacro)
@@ -66,5 +66,5 @@
       <parent link="${prefix}_base_link"/>
       <child link="${prefix}_shoulder_roll_link"/>
-      <origin xyz="0.0 0.0 0.0465" rpy="0 ${M_PI/2} 0"/>
+      <origin xyz="${(44/2+2.5)/1000} 0.0 0.0465" rpy="0 ${M_PI/2} 0"/>
       <axis xyz="0 0 1"/>
       <limit velocity="4.8" effort="25" lower="${-M_PI}" upper="${M_PI}" />
