Commit message: feat(description): joint velocity and effort limits from actuator datasheets
Define each Dynamixel model's stall torque and no-load speed once in
values.urdf.xacro (XM540-W270, XM540-W150, XM430-W350) and reference them
from the arm, hand and head limits, replacing the flat velocity=4.8 and
effort=25/30/1 placeholders. Effort follows the sobit_home convention
(datasheet torque x effort_ratio). The shoulder pitch effort is doubled for
its paired actuator. The hand prismatic joint converts through a shared
HAND_GEAR_RATIO property that controllers.urdf.xacro now uses for
gear_ratio as well.

File: sobit_light_description/urdf/arm/arm.urdf.xacro (robot description, xacro)
@@ -68,5 +68,5 @@
       <origin xyz="${(44/2+2.5)/1000} 0.0 0.0465" rpy="0 ${M_PI/2} 0"/>
       <axis xyz="0 0 1"/>
-      <limit velocity="4.8" effort="25" lower="${-M_PI}" upper="${M_PI}" />
+      <limit velocity="${XM430_W350_VELOCITY}" effort="${XM430_W350_TORQUE * effort_ratio}" lower="${-M_PI}" upper="${M_PI}" />
     </joint>
     <!--  Act 1 - Shoulder Roll -->
@@ -99,5 +99,5 @@
       <origin xyz="0.0 0.0 0.05095" rpy="0 0 0"/>
       <axis xyz="0 1 0"/>
-      <limit velocity="4.8" effort="25" lower="${-M_PI/2}" upper="${M_PI/2}" />
+      <limit velocity="${XM540_W150_VELOCITY}" effort="${2 * XM540_W150_TORQUE * effort_ratio}" lower="${-M_PI/2}" upper="${M_PI/2}" />
     </joint>
     <!--  Act 2 - Shoulder Pitch (right) -->
@@ -130,5 +130,5 @@
       <origin xyz="0.0 0.0 0.05095" rpy="0 0 0"/>
       <axis xyz="0 -1 0"/>
-      <limit velocity="4.8" effort="25" lower="${-M_PI}" upper="${M_PI}" />
+      <limit velocity="${XM540_W150_VELOCITY}" effort="${XM540_W150_TORQUE * effort_ratio}" lower="${-M_PI}" upper="${M_PI}" />
       <mimic joint="${prefix}_shoulder_pitch_joint" multiplier="-1" offset="0"/>
     </joint>
@@ -149,5 +149,5 @@
       <origin xyz="0.022 -0.0 0.128" rpy="0 0 0"/>
       <axis xyz="0 1 0"/>
-      <limit velocity="4.8" effort="25" lower="${-M_PI/2}" upper="${M_PI/2}" />
+      <limit velocity="${XM540_W270_VELOCITY}" effort="${XM540_W270_TORQUE * effort_ratio}" lower="${-M_PI/2}" upper="${M_PI/2}" />
     </joint>
     <!--  Act 4 - Elbow Pitch -->
@@ -180,5 +180,5 @@
       <origin xyz="0.0835 0.0 0.0" rpy="0 0 0"/>
       <axis xyz="1 0 0"/>
-      <limit velocity="4.8" effort="25" lower="${-M_PI}" upper="${M_PI}" />
+      <limit velocity="${XM540_W150_VELOCITY}" effort="${XM540_W150_TORQUE * effort_ratio}" lower="${-M_PI}" upper="${M_PI}" />
     </joint>
     <!--  Act 5 - Forearm Roll -->
@@ -211,5 +211,5 @@
       <origin xyz="0.0405 0.0 0.0" rpy="0 0 0"/>
       <axis xyz="0 1 0"/>
-      <limit velocity="4.8" effort="25" lower="${-M_PI/2}" upper="${M_PI/2}" />
+      <limit velocity="${XM430_W350_VELOCITY}" effort="${XM430_W350_TORQUE * effort_ratio}" lower="${-M_PI/2}" upper="${M_PI/2}" />
     </joint>
     <!--  Act 6 - Wrist Pitch -->
@@ -242,5 +242,5 @@
       <origin xyz="0.064 0 0.0" rpy="0 0 0"/>
       <axis xyz="1 0 0"/>
-      <limit velocity="4.8" effort="25" lower="${-M_PI}" upper="${M_PI}" />
+      <limit velocity="${XM430_W350_VELOCITY}" effort="${XM430_W350_TORQUE * effort_ratio}" lower="${-M_PI}" upper="${M_PI}" />
     </joint>
     <!--  Act 7 - Wrist Roll -->

File: sobit_light_description/urdf/controllers.urdf.xacro (robot description, xacro)
@@ -208,5 +208,5 @@
         <param name="Goal_Current">50</param>
         <param name="interface">rs</param>
-        <param name="gear_ratio">-59.504383354</param>
+        <param name="gear_ratio">-${HAND_GEAR_RATIO}</param>
         <param name="Return_Delay_Time">0</param>
       </xacro:unless>

File: sobit_light_description/urdf/hand/hand.urdf.xacro (robot description, xacro)
@@ -10,5 +10,5 @@
       <origin xyz="0.059 0.05498805 0.0" rpy="0 0 0"/>
       <axis xyz="0 1 0"/>
-      <limit velocity="4.8" effort="1" lower="-0.01791787" upper="0.02901195" />
+      <limit velocity="${XM430_W350_VELOCITY / HAND_GEAR_RATIO}" effort="${XM430_W350_TORQUE * HAND_GEAR_RATIO * effort_ratio}" lower="-0.01791787" upper="0.02901195" />
     </joint>
     <!--  Act 8 - Hand Finger (left) -->
@@ -41,5 +41,5 @@
       <origin xyz="0.059 -0.05498805 0.0" rpy="0 0 0"/>
       <axis xyz="0 -1 0"/>
-      <limit velocity="4.8" effort="1" lower="-1.57" upper="1.57"/>
+      <limit velocity="${XM430_W350_VELOCITY / HAND_GEAR_RATIO}" effort="${XM430_W350_TORQUE * HAND_GEAR_RATIO * effort_ratio}" lower="-1.57" upper="1.57"/>
       <mimic joint="${prefix_hand}_joint" multiplier="1"/>
     </joint>

File: sobit_light_description/urdf/head/head.urdf.xacro (robot description, xacro)
@@ -38,5 +38,5 @@
       <origin xyz="0.012 0.0 0.041" rpy="0.0 0.0 0.0" />
       <axis xyz="0 0 1" />
-      <limit effort="30" lower="${-M_PI}" upper="${M_PI}" velocity="${M_PI/2.0}" />
+      <limit effort="${XM430_W350_TORQUE * effort_ratio}" lower="${-M_PI}" upper="${M_PI}" velocity="${XM430_W350_VELOCITY}" />
     </joint>
     <link name="${prefix}_yaw_link">
@@ -67,5 +67,5 @@
       <origin xyz="0.0 0.0 0.0405" rpy="0.0 0.0 0.0" />
       <axis xyz="0 1 0" />
-      <limit effort="30" lower="${-M_PI/2.0}" upper="${M_PI/2.0}" velocity="${M_PI/2.0}" />
+      <limit effort="${XM430_W350_TORQUE * effort_ratio}" lower="${-M_PI/2.0}" upper="${M_PI/2.0}" velocity="${XM430_W350_VELOCITY}" />
     </joint>
     <link name="${prefix}_pitch_link">

File: sobit_light_description/urdf/values.urdf.xacro (robot description, xacro)
@@ -3,3 +3,15 @@
 <robot name="sobit_light_values" xmlns:xacro="http://ros.org/wiki/xacro">
   <xacro:property name="M_PI" value="3.14159265359" />
+  <!-- Dynamixel datasheet values @ 12V: stall torque [N·m], no-load speed [rad/s] -->
+  <xacro:property name="XM540_W270_TORQUE"   value="10.6" />
+  <xacro:property name="XM540_W270_VELOCITY" value="3.14" /> <!-- 30 rpm -->
+  <xacro:property name="XM540_W150_TORQUE"   value="7.1" />
+  <xacro:property name="XM540_W150_VELOCITY" value="5.24" /> <!-- 50 rpm -->
+  <xacro:property name="XM430_W350_TORQUE"   value="4.1" />
+  <xacro:property name="XM430_W350_VELOCITY" value="4.82" /> <!-- 46 rpm -->
+  <!-- Hand: XM430-W350 drives the prismatic finger through this ratio [rad/m].
+       Same value as gear_ratio in controllers.urdf.xacro (sign handled there). -->
+  <xacro:property name="HAND_GEAR_RATIO" value="59.504383354" />
+  <!-- Scale applied to datasheet torque for URDF effort limits (same convention as sobit_home) -->
+  <xacro:property name="effort_ratio" value="100.0" />
 </robot>

Commit message: feat(description): pitch joint ranges from measured Dynamixel limits
Replace the +-pi/2 placeholders on the arm and head pitch joints with the
Min/Max Position Limit registers read from the robot (ID2/3 450-3000,
ID4 700-2850, ID6 1000-3400, ID12 1200-3150 ticks), expressed in
values.urdf.xacro as tick-to-rad properties. The shoulder pitch mimic gets
the mirrored range, and the ros2_control position command min/max in
controllers.urdf.xacro reference the same properties so URDF and hardware
clamp cannot drift. Roughly doubles the well-conditioned workspace for
MoveIt Servo tracking.

File: sobit_light_description/urdf/arm/arm.urdf.xacro (robot description, xacro)
@@ -99,5 +99,5 @@
       <origin xyz="0.0 0.0 0.05095" rpy="0 0 0"/>
       <axis xyz="0 1 0"/>
-      <limit velocity="${XM540_W150_VELOCITY}" effort="${2 * XM540_W150_TORQUE * effort_ratio}" lower="${-M_PI/2}" upper="${M_PI/2}" />
+      <limit velocity="${XM540_W150_VELOCITY}" effort="${2 * XM540_W150_TORQUE * effort_ratio}" lower="${SHOULDER_PITCH_MIN}" upper="${SHOULDER_PITCH_MAX}" />
     </joint>
     <!--  Act 2 - Shoulder Pitch (right) -->
@@ -130,5 +130,5 @@
       <origin xyz="0.0 0.0 0.05095" rpy="0 0 0"/>
       <axis xyz="0 -1 0"/>
-      <limit velocity="${XM540_W150_VELOCITY}" effort="${XM540_W150_TORQUE * effort_ratio}" lower="${-M_PI}" upper="${M_PI}" />
+      <limit velocity="${XM540_W150_VELOCITY}" effort="${XM540_W150_TORQUE * effort_ratio}" lower="${-SHOULDER_PITCH_MAX}" upper="${-SHOULDER_PITCH_MIN}" />
       <mimic joint="${prefix}_shoulder_pitch_joint" multiplier="-1" offset="0"/>
     </joint>
@@ -149,5 +149,5 @@
       <origin xyz="0.022 -0.0 0.128" rpy="0 0 0"/>
       <axis xyz="0 1 0"/>
-      <limit velocity="${XM540_W270_VELOCITY}" effort="${XM540_W270_TORQUE * effort_ratio}" lower="${-M_PI/2}" upper="${M_PI/2}" />
+      <limit velocity="${XM540_W270_VELOCITY}" effort="${XM540_W270_TORQUE * effort_ratio}" lower="${ELBOW_PITCH_MIN}" upper="${ELBOW_PITCH_MAX}" />
     </joint>
     <!--  Act 4 - Elbow Pitch -->
@@ -211,5 +211,5 @@
       <origin xyz="0.0405 0.0 0.0" rpy="0 0 0"/>
       <axis xyz="0 1 0"/>
-      <limit velocity="${XM430_W350_VELOCITY}" effort="${XM430_W350_TORQUE * effort_ratio}" lower="${-M_PI/2}" upper="${M_PI/2}" />
+      <limit velocity="${XM430_W350_VELOCITY}" effort="${XM430_W350_TORQUE * effort_ratio}" lower="${WRIST_PITCH_MIN}" upper="${WRIST_PITCH_MAX}" />
     </joint>
     <!--  Act 6 - Wrist Pitch -->

File: sobit_light_description/urdf/controllers.urdf.xacro (robot description, xacro)
@@ -67,6 +67,6 @@
       </xacro:unless>
       <command_interface name="position">
-        <param name="min">-${M_PI/2}</param>
-        <param name="max">${M_PI/2}</param>
+        <param name="min">${HEAD_PITCH_MIN}</param>
+        <param name="max">${HEAD_PITCH_MAX}</param>
       </command_interface>
       <state_interface name="position">
@@ -122,6 +122,6 @@
       </xacro:unless>
       <command_interface name="position">
-        <param name="min">-${M_PI/2}</param>
-        <param name="max">${M_PI/2}</param>
+        <param name="min">${SHOULDER_PITCH_MIN}</param>
+        <param name="max">${SHOULDER_PITCH_MAX}</param>
       </command_interface>
       <state_interface name="position">
@@ -139,6 +139,6 @@
       </xacro:unless>
       <command_interface name="position">
-        <param name="min">-${M_PI/2}</param>
-        <param name="max">${M_PI/2}</param>
+        <param name="min">${ELBOW_PITCH_MIN}</param>
+        <param name="max">${ELBOW_PITCH_MAX}</param>
       </command_interface>
       <state_interface name="position">
@@ -173,6 +173,6 @@
       </xacro:unless>
       <command_interface name="position">
-        <param name="min">-${M_PI/2}</param>
-        <param name="max">${M_PI/2}</param>
+        <param name="min">${WRIST_PITCH_MIN}</param>
+        <param name="max">${WRIST_PITCH_MAX}</param>
       </command_interface>
       <state_interface name="position">

File: sobit_light_description/urdf/head/head.urdf.xacro (robot description, xacro)
@@ -67,5 +67,5 @@
       <origin xyz="0.0 0.0 0.0405" rpy="0.0 0.0 0.0" />
       <axis xyz="0 1 0" />
-      <limit effort="${XM430_W350_TORQUE * effort_ratio}" lower="${-M_PI/2.0}" upper="${M_PI/2.0}" velocity="${XM430_W350_VELOCITY}" />
+      <limit effort="${XM430_W350_TORQUE * effort_ratio}" lower="${HEAD_PITCH_MIN}" upper="${HEAD_PITCH_MAX}" velocity="${XM430_W350_VELOCITY}" />
     </joint>
     <link name="${prefix}_pitch_link">

File: sobit_light_description/urdf/values.urdf.xacro (robot description, xacro)
@@ -13,4 +13,17 @@
        Same value as gear_ratio in controllers.urdf.xacro (sign handled there). -->
   <xacro:property name="HAND_GEAR_RATIO" value="59.504383354" />
+  <!-- Dynamixel position register -> rad (4096 ticks/rev, 2048 = 0 rad). Joint
+       ranges below are the Min/Max Position Limit registers measured on the
+       real robot (2026-09-10): ID2/3 450-3000, ID4 700-2850, ID6 1000-3400,
+       ID12 1200-3150. Rolls (ID1/5/7), head yaw (ID11) and hand (ID8) are full range. -->
+  <xacro:property name="DXL_TICK" value="${2*M_PI/4096}" />
+  <xacro:property name="SHOULDER_PITCH_MIN" value="${(450-2048)*DXL_TICK}" />
+  <xacro:property name="SHOULDER_PITCH_MAX" value="${(3000-2048)*DXL_TICK}" />
+  <xacro:property name="ELBOW_PITCH_MIN"    value="${(700-2048)*DXL_TICK}" />
+  <xacro:property name="ELBOW_PITCH_MAX"    value="${(2850-2048)*DXL_TICK}" />
+  <xacro:property name="WRIST_PITCH_MIN"    value="${(1000-2048)*DXL_TICK}" />
+  <xacro:property name="WRIST_PITCH_MAX"    value="${(3400-2048)*DXL_TICK}" />
+  <xacro:property name="HEAD_PITCH_MIN"     value="${(1200-2048)*DXL_TICK}" />
+  <xacro:property name="HEAD_PITCH_MAX"     value="${(3150-2048)*DXL_TICK}" />
   <!-- Scale applied to datasheet torque for URDF effort limits (same convention as sobit_home) -->
   <xacro:property name="effort_ratio" value="100.0" />

Commit message: refactor(description): shoulder_pitch_sub_joint is a slave, model it as fixed
Dynamixel ID2 runs as a drive-mode slave of ID3, so it is never commanded
by ros2_control. The second shoulder bracket shares the pitch joint origin
and, with its old axis (0 -1 0) and mimic multiplier -1, always had the
same orientation as the shoulder pitch link; attach it there with a fixed
joint instead of a mimic revolute joint, keeping its inertia. Drop the
commented-out ros2_control block and the sub-joint mirroring (negated
target, extra trajectory entry) from the dualshock and keyboard teleop
scripts.

File: sobit_light_description/urdf/arm/arm.urdf.xacro (robot description, xacro)
@@ -124,12 +124,13 @@
       </inertial>
     </link>
-    <!--  Act 3 - Shoulder Pitch (left) -->
-    <joint name="${prefix}_shoulder_pitch_sub_joint" type="revolute">
-      <parent link="${prefix}_shoulder_roll_link"/>
+    <!--  Act 3 - Shoulder Pitch (left): Dynamixel ID2 runs as a drive-mode
+          slave of ID3, so the second bracket is rigid with the shoulder pitch
+          link. It shares the pitch joint's origin and, with its former axis
+          (0 -1 0) and mimic multiplier -1, always had the same orientation, so
+          a fixed joint at the identity is kinematically identical. -->
+    <joint name="${prefix}_shoulder_pitch_sub_joint" type="fixed">
+      <parent link="${prefix}_shoulder_pitch_link"/>
       <child link="${prefix}_shoulder_pitch_sub_link"/>
-      <origin xyz="0.0 0.0 0.05095" rpy="0 0 0"/>
-      <axis xyz="0 -1 0"/>
-      <limit velocity="${XM540_W150_VELOCITY}" effort="${XM540_W150_TORQUE * effort_ratio}" lower="${-SHOULDER_PITCH_MAX}" upper="${-SHOULDER_PITCH_MIN}" />
-      <mimic joint="${prefix}_shoulder_pitch_joint" multiplier="-1" offset="0"/>
+      <origin xyz="0.0 0.0 0.0" rpy="0 0 0"/>
     </joint>
     <!--  Act 3 - Shoulder Pitch (left) -->

File: sobit_light_description/urdf/controllers.urdf.xacro (robot description, xacro)
@@ -96,22 +96,4 @@
       <!-- <state_interface name="effort"/> -->
     </joint>
-    <!-- <joint name="${prefix}_shoulder_pitch_sub_joint">
-      <xacro:unless value="${$(arg enable_gz)}">
-        <param name="id">2</param>
-        <param name="control_mode">0</param>
-        <param name="interface">rs</param>
-        <param name="Return_Delay_Time">0</param>
-      </xacro:unless>
-      <state_interface name="position">
-        <param name="initial_value">${M_PI/2}</param>
-      </state_interface>
-      <state_interface name="velocity"/>
-      <state_interface name="effort"/>
-      <xacro:unless value="${$(arg enable_gz)}">
-        <command_interface name="position"/>
-      </xacro:unless>
-      <param name="mimic">${prefix}_shoulder_pitch_joint</param>
-      <param name="multiplier">-1</param>
-    </joint> -->
     <joint name="${prefix}_shoulder_pitch_joint">
       <xacro:unless value="${$(arg enable_gz)}">

Commit message: refactor(description): remove arm_shoulder_pitch_sub joint and link
Dynamixel ID2 is a drive-mode slave of ID3; the second shoulder bracket is
rigid with arm_shoulder_pitch_link and needs no joint or link of its own.
Delete both and fold the bracket's mass and inertia (identical origin and
values) into arm_shoulder_pitch_link, and drop the link from the saved
rviz link lists.

File: sobit_light_description/urdf/arm/arm.urdf.xacro (robot description, xacro)
@@ -116,30 +116,13 @@
         </geometry>
       </collision>
+      <!-- Mass covers both shoulder pitch brackets: Dynamixel ID2 is a
+           drive-mode slave of ID3, so the second bracket is rigid with this
+           link and is not modelled as its own link (same origin and inertia). -->
       <inertial>
         <origin xyz="${0.03575-0.0585/2} 0.0 ${-0.016+(0.14475+0.016)/2}" rpy="0 0 0"/>
-        <mass value="0.261" />
-        <inertia  ixx="${1/12*0.261*(0.0585**2+(0.14475+0.016)**2)}" ixy="0.0" ixz="0.0"
-                  iyy="${1/12*0.261*(0.0440**2+(0.14475+0.016)**2)}" iyz="0.0"
-                  izz="${1/12*0.261*(0.0585**2+0.0440**2)}" />
-      </inertial>
-    </link>
-    <!--  Act 3 - Shoulder Pitch (left): Dynamixel ID2 runs as a drive-mode
-          slave of ID3, so the second bracket is rigid with the shoulder pitch
-          link. It shares the pitch joint's origin and, with its former axis
-          (0 -1 0) and mimic multiplier -1, always had the same orientation, so
-          a fixed joint at the identity is kinematically identical. -->
-    <joint name="${prefix}_shoulder_pitch_sub_joint" type="fixed">
-      <parent link="${prefix}_shoulder_pitch_link"/>
-      <child link="${prefix}_shoulder_pitch_sub_link"/>
-      <origin xyz="0.0 0.0 0.0" rpy="0 0 0"/>
-    </joint>
-    <!--  Act 3 - Shoulder Pitch (left) -->
-    <link name="${prefix}_shoulder_pitch_sub_link">
-      <inertial>
-        <origin xyz="${0.03575-0.0585/2} 0.0 ${-0.016+(0.14475+0.016)/2}" rpy="0 0 0"/>
-        <mass value="0.261" />
-        <inertia  ixx="${1/12*0.261*(0.0585**2+(0.14475+0.016)**2)}" ixy="0.0" ixz="0.0"
-                  iyy="${1/12*0.261*(0.0440**2+(0.14475+0.016)**2)}" iyz="0.0"
-                  izz="${1/12*0.261*(0.0585**2+0.0440**2)}" />
+        <mass value="${2*0.261}" />
+        <inertia  ixx="${2*1/12*0.261*(0.0585**2+(0.14475+0.016)**2)}" ixy="0.0" ixz="0.0"
+                  iyy="${2*1/12*0.261*(0.0440**2+(0.14475+0.016)**2)}" iyz="0.0"
+                  izz="${2*1/12*0.261*(0.0585**2+0.0440**2)}" />
       </inertial>
     </link>
