Commit message: [UPD] all urdf and transmissions (todo: inertia)

File: sobit_light_description/urdf/back/back.urdf.xacro (robot description, xacro)
@@ -5,9 +5,9 @@
       <parent link="${parent}" />
       <child link="${prefix}_base_link" />
-      <origin xyz="0.0 0.0 0.0" rpy="0.0 0.0 0.0" />
+      <origin xyz="${0.320/2-0.197} 0.0 0.0" rpy="0.0 0.0 0.0" />
     </joint>
     <link name="${prefix}_base_link" >
       <visual>
-        <origin xyz="0.0 0.0 0.0" rpy="0.0 0.0 ${M_PI}" />
+        <origin xyz="0.0 0.0 0.0" rpy="0.0 0.0 ${M_PI/2}" />
         <geometry>
           <mesh filename="file://$(find sobit_light_description)/meshes/back/back_base.stl" scale="0.001 0.001 0.001" />

File: sobit_light_description/urdf/head/head.transmission.xacro (robot description, xacro)
@@ -1,4 +1,4 @@
 <?xml version="1.0" ?>
-<robot xmlns:xacro="http://ros.org/wiki/xacro">
+<robot name="head_transmission" xmlns:xacro="http://ros.org/wiki/xacro">
   <xacro:macro name="head_transmission" params="prefix">
     <position_joint_transmission joint="${prefix}_pan_joint"  reduction="1" />

File: sobit_light_description/urdf/head/head.urdf.xacro (robot description, xacro)
@@ -1,5 +1,5 @@
 <?xml version="1.0" encoding="UTF-8" ?>
 <robot name="head" xmlns:xacro="http://ros.org/wiki/xacro">
-  <xacro:include filename="$(find sobit_pro_description)/urdf/head/head.transmission.xacro" />
+  <xacro:include filename="$(find sobit_light_description)/urdf/head/head.transmission.xacro" />
   <xacro:macro name="head" params="prefix parent">
     <joint name="${prefix}_base_joint" type="fixed">
@@ -8,12 +8,12 @@
       <!-- <child link="${prefix}_camera_base_link" /> -->
       <child link="${prefix}_base_link" />
-      <origin xyz="0.0900 0.0 0.5270" rpy="0.0 0.0 0.0" />
+      <origin xyz="0.0 0.0 0.605" rpy="0.0 0.0 0.0" />
     </joint>
     <link name="${prefix}_base_link">
     <!-- <link name="${prefix}_camera_base_link"> -->
       <visual>
-        <origin xyz="0.0 0.0 0.0" rpy="${M_PI/2.0} 0.0 ${M_PI/2.0}" />
+        <origin xyz="0.0 0.0 0.0" rpy="0.0 0.0 ${M_PI/2.0}" />
         <geometry>
-          <mesh filename="file://$(find sobit_light_description)/meshes/head/head_camera_base.stl" scale="0.001 0.001 0.001" />
+          <mesh filename="file://$(find sobit_light_description)/meshes/head/head_base.stl" scale="0.001 0.001 0.001" />
         </geometry>
         <material name="black" />
@@ -44,7 +44,7 @@
       <child link="${prefix}_pan_link" />
       <!-- <child link="${prefix}_camera_pan_link" /> -->
-      <origin xyz="0.03985 0.0 0.0190" rpy="0.0 0.0 0.0" />
+      <origin xyz="0.012 0.0 0.041" rpy="0.0 0.0 0.0" />
       <axis xyz="0 0 1" />
-      <limit effort="30" lower="${-M_PI/2.0}" upper="${M_PI/2.0}" velocity="${M_PI/2.0}" />
+      <limit effort="30" lower="${-M_PI}" upper="${M_PI}" velocity="${M_PI/2.0}" />
     </joint>
     <link name="${prefix}_pan_link">
@@ -53,5 +53,5 @@
         <origin xyz="0.0 0.0 0.0" rpy="0.0 0.0 ${M_PI/2.0}" />
         <geometry>
-          <mesh filename="file://$(find sobit_light_description)/meshes/head/head_camera_pan.stl" scale="0.001 0.001 0.001" />
+          <mesh filename="file://$(find sobit_light_description)/meshes/head/head_pan.stl" scale="0.001 0.001 0.001" />
         </geometry>
         <material name="black" />
@@ -91,5 +91,5 @@
         <origin xyz="0.0 0.0 0.0" rpy="0.0 0.0 ${M_PI/2.0}" />
         <geometry>
-          <mesh filename="file://$(find sobit_light_description)/meshes/head/head_camera_tilt.stl" scale="0.001 0.001 0.001" />
+          <mesh filename="file://$(find sobit_light_description)/meshes/head/head_tilt.stl" scale="0.001 0.001 0.001" />
         </geometry>
         <material name="black" />

File: sobit_light_description/urdf/sensor/camera_back.urdf.xacro (robot description, xacro)
@@ -1,14 +1,20 @@
-<?xml version="1.0"?>
+<?xml version="1.0" encoding="UTF-8" ?>
 <robot name="camera_back" xmlns:xacro="http://ros.org/wiki/xacro">
   <xacro:macro name="camera_back" params="prefix parent">
-    <joint name="${prefix}_base_joint" type="fixed">
-      <origin xyz="0.0045 0.0 0.169655" rpy="0.0 0.0 0.0" />
+    <joint name="${prefix}_joint" type="fixed">
       <parent link="${parent}" />
-      <child link="${prefix}_base_link" />
+      <child link="${prefix}_link" />
+      <origin xyz="${-0.150 + 0.01} 0 0.070"
+              rpy="-${M_PI / 2.0} 0 ${M_PI / 2.0}" />
     </joint>
-    <link name="${prefix}_base_link" />
-    <xacro:sensor_d435 parent="${prefix}_base_link" name="${prefix}" topics_ns="head_camera" >
-      <origin xyz="0.0 0.0 0.0" rpy="0.0 0.0 0.0" />
-    </xacro:sensor_d435>
+    <link name="${prefix}_link">
+      <inertial>
+        <origin xyz="0 0 0" rpy="0 0 0" />
+        <mass value="0.2" />
+        <inertia ixx="0.001" ixy="0" ixz="0"
+                 iyy="0.001" iyz="0"
+                 izz="0.001" />
+      </inertial>
+    </link>
   </xacro:macro>
 </robot>

File: sobit_light_description/urdf/sensor/camera_front.urdf.xacro (robot description, xacro)
@@ -1,14 +1,20 @@
-<?xml version="1.0"?>
+<?xml version="1.0" encoding="UTF-8" ?>
 <robot name="camera_front" xmlns:xacro="http://ros.org/wiki/xacro">
   <xacro:macro name="camera_front" params="prefix parent">
-    <joint name="${prefix}_base_joint" type="fixed">
-      <origin xyz="0.0045 0.0 0.169655" rpy="0.0 0.0 0.0" />
+    <joint name="${prefix}_joint" type="fixed">
       <parent link="${parent}" />
-      <child link="${prefix}_base_link" />
+      <child link="${prefix}_link" />
+      <origin xyz="${0.2196 - 0.01} 0 0.070"
+              rpy="-${M_PI / 2.0} 0 -${M_PI / 2.0}" />
     </joint>
-    <link name="${prefix}_base_link" />
-    <xacro:sensor_d435 parent="${prefix}_base_link" name="${prefix}" topics_ns="head_camera" >
-      <origin xyz="0.0 0.0 0.0" rpy="0.0 0.0 0.0" />
-    </xacro:sensor_d435>
+    <link name="${prefix}_link">
+      <inertial>
+        <origin xyz="0 0 0" rpy="0 0 0" />
+        <mass value="0.2" />
+        <inertia ixx="0.001" ixy="0" ixz="0"
+                 iyy="0.001" iyz="0"
+                 izz="0.001" />
+      </inertial>
+    </link>
   </xacro:macro>
 </robot>

File: sobit_light_description/urdf/sensor/camera_head.urdf.xacro (robot description, xacro)
@@ -1,12 +1,13 @@
-<?xml version="1.0"?>
+<?xml version="1.0" encoding="UTF-8" ?>
 <robot name="camera_head" xmlns:xacro="http://ros.org/wiki/xacro">
+  <xacro:include filename="$(find realsense2_description)/urdf/_d435.urdf.xacro" />
   <xacro:macro name="camera_head" params="prefix parent">
     <joint name="${prefix}_base_joint" type="fixed">
-      <origin xyz="0.0045 0.0 0.169655" rpy="0.0 0.0 0.0" />
+      <origin xyz="0.05815 0.0 0.12050335" rpy="0.0 0.0 0.0" />
       <parent link="${parent}" />
       <child link="${prefix}_base_link" />
     </joint>
     <link name="${prefix}_base_link" />
-    <xacro:sensor_d435 parent="${prefix}_base_link" name="${prefix}" topics_ns="head_camera" >
+    <xacro:sensor_d435 parent="${prefix}_base_link" name="${prefix}" >
       <origin xyz="0.0 0.0 0.0" rpy="0.0 0.0 0.0" />
     </xacro:sensor_d435>

File: sobit_light_description/urdf/sensor/imu.urdf.xacro (robot description, xacro)
@@ -2,39 +2,12 @@
 <robot name="imu" xmlns:xacro="http://ros.org/wiki/xacro">
   <xacro:macro name="imu" params="prefix parent">
-    <joint name="${prefix}_base_joint" type="fixed">
+    <joint name="${prefix}_joint"
+          type="fixed">
       <parent link="${parent}" />
-      <child link="${prefix}_base_link" />
-      <origin xyz="0.1500 0.0 0.0" rpy="0.0 0.0 0.0" />
+      <child link="${prefix}_link" />
+      <origin rpy="0 0 0"
+              xyz="0.0756 -0.0655 0.05146" />
     </joint>
-    <link name="${prefix}_base_link">
-      <visual>
-        <origin xyz="0.0 0.0 0.0" rpy="${M_PI/2} 0.0 ${M_PI}" />
-        <geometry>
-          <mesh filename="file://$(find sobit_light_description)/meshes/sensor/lidar_base.stl" scale="0.001 0.001 0.001" />
-        </geometry>
-        <material name="black" />
-      </visual>
-      <collision>
-        <origin xyz="${0.092/2} 0.0 -${0.007/2}" rpy="0.0 0.0 0.0" />
-        <!-- <origin xyz="0.0 0.0 0.0" rpy="${M_PI/2} 0.0 ${M_PI}" /> -->
-        <geometry>
-          <box size="0.092 0.184 0.007"/>
-          <!-- <mesh filename="file://$(find sobit_light_description)/meshes/sensor/lidar_base.stl" scale="0.001 0.001 0.001" /> -->
-        </geometry>
-      </collision>
-      <inertial>
-        <origin xyz="${0.092/2} 0.0 -${0.007/2}" rpy="0.0 0.0 0.0" />
-        <mass value="0.08" />
-        <inertia ixx="${1/12*0.08*(0.092**2+0.007**2)}" ixy="0.0" ixz="0.0"
-                 iyy="${1/12*0.08*(0.184**2+0.007**2)}" iyz="0.0"
-                 izz="${1/12*0.08*(0.092**2+0.184**2)}" />
-        <!-- <inertia ixx="1.0" ixy="0.0" ixz="0.0"
-                 iyy="1.0" iyz="0.0"
-                 izz="1.0" /> -->
-      </inertial>
-    </link>
-    <xacro:hokuyo_ust_mount prefix="${prefix}" parent="${prefix}_base_link" topic="scan" >
-      <origin xyz="0.067 0.0 0.0" rpy="0.0 0.0 0.0" />
-    </xacro:hokuyo_ust_mount>
+    <link name="${prefix}_link" />
   </xacro:macro>
 </robot>

File: sobit_light_description/urdf/sensor/lidar.urdf.xacro (robot description, xacro)
@@ -2,39 +2,18 @@
 <robot name="lidar" xmlns:xacro="http://ros.org/wiki/xacro">
   <xacro:macro name="lidar" params="prefix parent">
-    <joint name="${prefix}_base_joint" type="fixed">
+    <joint name="${prefix}_joint" type="fixed">
       <parent link="${parent}" />
-      <child link="${prefix}_base_link" />
-      <origin xyz="0.1500 0.0 0.0" rpy="0.0 0.0 0.0" />
+      <child link="laser_frame" />
+      <origin xyz="0.156 0 0.1049" rpy="0 0 ${M_PI / 2.0}" />
     </joint>
-    <link name="${prefix}_base_link">
-      <visual>
-        <origin xyz="0.0 0.0 0.0" rpy="${M_PI/2} 0.0 ${M_PI}" />
-        <geometry>
-          <mesh filename="file://$(find sobit_light_description)/meshes/sensor/lidar_base.stl" scale="0.001 0.001 0.001" />
-        </geometry>
-        <material name="black" />
-      </visual>
-      <collision>
-        <origin xyz="${0.092/2} 0.0 -${0.007/2}" rpy="0.0 0.0 0.0" />
-        <!-- <origin xyz="0.0 0.0 0.0" rpy="${M_PI/2} 0.0 ${M_PI}" /> -->
-        <geometry>
-          <box size="0.092 0.184 0.007"/>
-          <!-- <mesh filename="file://$(find sobit_light_description)/meshes/sensor/lidar_base.stl" scale="0.001 0.001 0.001" /> -->
-        </geometry>
-      </collision>
+    <link name="laser_frame">
       <inertial>
-        <origin xyz="${0.092/2} 0.0 -${0.007/2}" rpy="0.0 0.0 0.0" />
-        <mass value="0.08" />
-        <inertia ixx="${1/12*0.08*(0.092**2+0.007**2)}" ixy="0.0" ixz="0.0"
-                 iyy="${1/12*0.08*(0.184**2+0.007**2)}" iyz="0.0"
-                 izz="${1/12*0.08*(0.092**2+0.184**2)}" />
-        <!-- <inertia ixx="1.0" ixy="0.0" ixz="0.0"
-                 iyy="1.0" iyz="0.0"
-                 izz="1.0" /> -->
+        <origin xyz="0 0 0" rpy="0 0 0" />
+        <mass value="0.2" />
+        <inertia ixx="0.001" ixy="0" ixz="0"
+                 iyy="0.001" iyz="0"
+                 izz="0.001" />
       </inertial>
     </link>
-    <xacro:hokuyo_ust_mount prefix="${prefix}" parent="${prefix}_base_link" topic="scan" >
-      <origin xyz="0.067 0.0 0.0" rpy="0.0 0.0 0.0" />
-    </xacro:hokuyo_ust_mount>
   </xacro:macro>
 </robot>

File: sobit_light_description/urdf/sensor/mic.urdf.xacro (robot description, xacro)
@@ -5,5 +5,5 @@
       <parent link="${parent}" />
       <child link="${prefix}_base_link" />
-      <origin xyz="-0.039589 0.0 0.169655" rpy="0.0 0.0 0.0" />
+      <origin xyz="0.0 0.0 0.0" rpy="0.0 0.0 0.0" />
     </joint>
     <link name="${prefix}_base_link">
@@ -11,5 +11,5 @@
         <origin xyz="0.0 0.0 0.0" rpy="0.0 0.0 ${M_PI/2.0}" />
         <geometry>
-          <mesh filename="package://sobit_mini_description/meshes/sensor/mic.stl"/>
+          <mesh filename="file://$(find sobit_light_description)/meshes/sensor/mic.stl"/>
         </geometry>
         <material name="black" />
@@ -18,5 +18,5 @@
         <origin xyz="0.0 0.0 0.0" rpy="0.0 0.0 ${M_PI/2.0}" />
         <geometry>
-          <mesh filename="package://sobit_mini_description/meshes/sensor/mic.stl" />
+          <mesh filename="file://$(find sobit_light_description)/meshes/sensor/mic.stl" />
         </geometry>
         <material name="black" />
@@ -30,7 +30,7 @@
       </inertial>
     </link>
-    <gazebo reference="${prefix}_base_link">
+    <!-- <gazebo reference="${prefix}_base_link">
       <material>Gazebo/Black</material>
-    </gazebo>
+    </gazebo> -->
   </xacro:macro>
 </robot>

File: sobit_light_description/urdf/sensor/speaker.urdf.xacro (robot description, xacro)
@@ -5,11 +5,11 @@
       <parent link="${parent}" />
       <child link="${prefix}_base_link" />
-      <origin xyz="-0.039589 0.0 0.169655" rpy="0.0 0.0 0.0" />
+      <origin xyz="0.050 0.0 0.510" rpy="0.0 0.0 0.0" />
     </joint>
     <link name="${prefix}_base_link">
       <visual>
-        <origin xyz="0.0 0.0 0.0" rpy="0.0 0.0 ${M_PI/2.0}" />
+        <origin xyz="0.0 0.0 0.0" rpy="-${M_PI/9.0} 0.0 ${M_PI/2.0}" />
         <geometry>
-          <mesh filename="package://sobit_mini_description/meshes/sensor/mic.stl"/>
+          <mesh filename="file://$(find sobit_light_description)/meshes/sensor/speaker.stl" scale="0.001 0.001 0.001" />
         </geometry>
         <material name="black" />
@@ -18,5 +18,5 @@
         <origin xyz="0.0 0.0 0.0" rpy="0.0 0.0 ${M_PI/2.0}" />
         <geometry>
-          <mesh filename="package://sobit_mini_description/meshes/sensor/mic.stl" />
+          <mesh filename="file://$(find sobit_light_description)/meshes/sensor/speaker.stl" scale="0.001 0.001 0.001" />
         </geometry>
         <material name="black" />
@@ -30,7 +30,7 @@
       </inertial>
     </link>
-    <gazebo reference="${prefix}_base_link">
+    <!-- <gazebo reference="${prefix}_base_link">
       <material>Gazebo/Black</material>
-    </gazebo>
+    </gazebo> -->
   </xacro:macro>
 </robot>

File: sobit_light_description/urdf/sensor/tof.urdf.xacro (robot description, xacro)
@@ -2,39 +2,19 @@
 <robot name="tof" xmlns:xacro="http://ros.org/wiki/xacro">
   <xacro:macro name="tof" params="prefix parent">
-    <joint name="${prefix}_base_joint" type="fixed">
+    <joint name="${prefix}_joint" type="fixed">
       <parent link="${parent}" />
-      <child link="${prefix}_base_link" />
-      <origin xyz="0.1500 0.0 0.0" rpy="0.0 0.0 0.0" />
+      <child link="${prefix}_link" />
+      <origin xyz="0.221 0.0 0.0418"
+              rpy="-${M_PI / 4.0} 0 -${M_PI / 2.0}" />
     </joint>
-    <link name="${prefix}_base_link">
-      <visual>
-        <origin xyz="0.0 0.0 0.0" rpy="${M_PI/2} 0.0 ${M_PI}" />
-        <geometry>
-          <mesh filename="file://$(find sobit_light_description)/meshes/sensor/lidar_base.stl" scale="0.001 0.001 0.001" />
-        </geometry>
-        <material name="black" />
-      </visual>
-      <collision>
-        <origin xyz="${0.092/2} 0.0 -${0.007/2}" rpy="0.0 0.0 0.0" />
-        <!-- <origin xyz="0.0 0.0 0.0" rpy="${M_PI/2} 0.0 ${M_PI}" /> -->
-        <geometry>
-          <box size="0.092 0.184 0.007"/>
-          <!-- <mesh filename="file://$(find sobit_light_description)/meshes/sensor/lidar_base.stl" scale="0.001 0.001 0.001" /> -->
-        </geometry>
-      </collision>
+    <link name="${prefix}_link">
       <inertial>
-        <origin xyz="${0.092/2} 0.0 -${0.007/2}" rpy="0.0 0.0 0.0" />
-        <mass value="0.08" />
-        <inertia ixx="${1/12*0.08*(0.092**2+0.007**2)}" ixy="0.0" ixz="0.0"
-                 iyy="${1/12*0.08*(0.184**2+0.007**2)}" iyz="0.0"
-                 izz="${1/12*0.08*(0.092**2+0.184**2)}" />
-        <!-- <inertia ixx="1.0" ixy="0.0" ixz="0.0"
-                 iyy="1.0" iyz="0.0"
-                 izz="1.0" /> -->
+        <origin xyz="0 0 0" rpy="0 0 0" />
+        <mass value="0.2" />
+        <inertia ixx="0.001" ixy="0" ixz="0"
+                 iyy="0.001" iyz="0"
+                 izz="0.001" />
       </inertial>
     </link>
-    <xacro:hokuyo_ust_mount prefix="${prefix}" parent="${prefix}_base_link" topic="scan" >
-      <origin xyz="0.067 0.0 0.0" rpy="0.0 0.0 0.0" />
-    </xacro:hokuyo_ust_mount>
   </xacro:macro>
 </robot>
