Commit message: [UPD] all urdf and transmissions (todo: inertia)

File: sobit_light_description/urdf/wheel/wheel.urdf.xacro (robot description, xacro)
@@ -1,126 +1,67 @@
 <?xml version="1.0" encoding="UTF-8" ?>
 <robot name="wheel" xmlns:xacro="http://ros.org/wiki/xacro">
-  <xacro:macro name="stack_wheel_steer_base" params="parent prefix number x_loc y_loc z_loc roll=0.0 pitch=0.0 yaw=0.0">
-    <joint name="wheel_${prefix}_steer_base_joint" type="fixed">
-      <origin xyz="${x_loc} ${y_loc} ${z_loc}" rpy="${roll} ${pitch} ${(number-1)*M_PI/2.0+M_PI/4.0}" />
+  <xacro:macro name="wheel" params="parent prefix">
+    <!-- Left wheel -->
+    <joint name="${prefix}_l_drive_wheel_joint" type="continuous">
       <parent link="${parent}" />
-      <child link="wheel_${prefix}_steer_base_link" />
+      <child link="${prefix}_l_drive_wheel_link" />
+      <origin xyz="0.0 0.100 0.045" rpy="0 0 0" />
+      <axis xyz="0 1 0" />
+      <limit velocity="10" effort="100" />
     </joint>
-    <link name="wheel_${prefix}_steer_base_link">
+    <link name="${prefix}_l_drive_wheel_link">
       <visual>
-        <origin xyz="0.0 0.0 0.0" rpy="${M_PI/2.0} 0.0 ${M_PI/2.0}" />
+        <origin xyz="0 0 0" rpy="${M_PI / 2.0} 0 0" />
         <geometry>
-          <mesh filename="file://$(find sobit_light_description)/meshes/wheel/wheel_base.stl" scale="0.001 0.001 0.001" />
+          <cylinder length="0.025" radius="0.045" />
         </geometry>
-        <material name="black" />
+        <material name="tire" />
       </visual>
       <collision>
-        <origin xyz="${0.01388-0.05525/2} 0.0 -${0.005+0.034/2+0.02/2}" rpy="0.0 0.0 0.0" />
-        <!-- <origin xyz="0.0 0.0 0.0" rpy="${M_PI/2.0} 0.0 ${M_PI/2.0}" /> -->
+        <origin xyz="0 0 0" rpy="${M_PI / 2.0} 0 0" />
         <geometry>
-          <box size="0.05525 0.0285 0.084" />
-          <!-- <mesh filename="file://$(find sobit_light_description)/meshes/wheel/wheel_base.stl" scale="0.001 0.001 0.001" /> -->
+          <cylinder length="0.025" radius="0.045" />
         </geometry>
+        <material name="tire" />
       </collision>
       <inertial>
-        <origin xyz="${0.01388-0.05525/2} 0.0 -${0.005+0.034/2+0.02/2}" rpy="0.0 0.0 0.0" />
-        <!-- <origin xyz="0.0 0.0 0.0" rpy="${M_PI/2.0} 0.0 ${M_PI/2.0}" /> -->
-        <mass value="1" />
-        <inertia ixx="${1/12*1*(0.05525**2+0.084**2)}" ixy="0.0" ixz="0.0"
-                 iyy="${1/12*1*(0.0285**2 +0.084**2)}" iyz="0.0"
-                 izz="${1/12*1*(0.05525**2+0.0285**2)}" />
-        <!-- <inertia ixx="1.0" ixy="0.0" ixz="0.0"
-                 iyy="1.0" iyz="0.0"
-                 izz="1.0" /> -->
+        <origin xyz="0 0 0" rpy="0 0 0" />
+        <mass value="0.2" />
+        <inertia ixx="0.001" ixy="0" ixz="0"
+                 iyy="0.001" iyz="0"
+                 izz="0.001" />
+      </inertial>
+    </link>
+    <!-- Right wheel -->
+    <joint name="${prefix}_r_drive_wheel_joint" type="continuous">
+      <parent link="${parent}" />
+      <child link="${prefix}_r_drive_wheel_link" />
+      <origin xyz="0.0 -0.100 0.045" rpy="0 0 0" />
+      <axis xyz="0 1 0" />
+      <limit velocity="10" effort="100" />
+    </joint>
+    <link name="${prefix}_r_drive_wheel_link">
+      <visual>
+        <origin xyz="0 0 0" rpy="${M_PI / 2.0} 0 0" />
+        <geometry>
+          <cylinder length="0.025" radius="0.045" />
+        </geometry>
+        <material name="tire" />
+      </visual>
+      <collision>
+        <origin xyz="0 0 0" rpy="${M_PI / 2.0} 0 0" />
+        <geometry>
+          <cylinder length="0.025" radius="0.045" />
+        </geometry>
+        <material name="tire" />
+      </collision>
+      <inertial>
+        <origin xyz="0 0 0" rpy="0 0 0" />
+        <mass value="0.2" />
+        <inertia ixx="0.001" ixy="0" ixz="0"
+                 iyy="0.001" iyz="0"
+                 izz="0.001" />
       </inertial>
     </link>
   </xacro:macro>
-  <xacro:macro name="stack_wheel_steer" params="parent prefix number x_loc y_loc z_loc roll=0.0 pitch=0.0 yaw=0.0">
-    <joint name="wheel_${prefix}_steer_joint" type="revolute">
-      <origin xyz="${x_loc} ${y_loc} ${z_loc}" rpy="${roll} ${pitch} ${yaw}" />
-      <parent link="${parent}" />
-      <child link="wheel_${prefix}_steer_link" />
-      <axis xyz="0.0 0.0 1.0 " />
-      <limit lower="${-M_PI / 2}" upper="${M_PI/2}" effort="10" velocity="10" />
-      <!-- <dynamics damping="0.2" friction="0" /> -->
-    </joint>
-    <link name="wheel_${prefix}_steer_link">
-      <visual>
-        <origin xyz="0.0 0.0 0.0" rpy="${M_PI/2} 0.0 ${M_PI/2}" />
-        <geometry>
-          <mesh filename="file://$(find sobit_light_description)/meshes/wheel/wheel_steer.stl" scale="0.001 0.001 0.001" />
-        </geometry>
-        <material name="black" />
-      </visual>
-      <collision>
-        <origin xyz="${0.0244+0.0436/2} 0.0 ${0.034/2+0.0149-0.1766/2}" rpy="0.0 0.0 0.0" />
-        <!-- <origin xyz="0.0 0.0 0.0" rpy="${M_PI/2} 0.0 ${M_PI/2}" /> -->
-        <geometry>
-          <!-- <box size="0.0495 0.1766 0.0436" /> -->
-          <box size="0.0436 0.0495 0.1766" />
-          <!-- <mesh filename="file://$(find sobit_light_description)/meshes/wheel/wheel_steer.stl" scale="0.001 0.001 0.001" /> -->
-        </geometry>
-      </collision>
-      <inertial>
-        <origin xyz="${0.0244+0.0436/2} 0.0 ${0.034/2+0.0149-0.1766/2}" rpy="0.0 0.0 0.0" />
-        <mass value="1" />
-        <inertia ixx="${1/12*1*(0.0436**2+0.1766**2)}" ixy="0.0" ixz="0.0"
-                 iyy="${1/12*1*(0.0495**2+0.1766**2)}" iyz="0.0"
-                 izz="${1/12*1*(0.0436**2+0.0495**2)}" />
-        <!-- <inertia ixx="1.0" ixy="0.0" ixz="0.0"
-                 iyy="1.0" iyz="0.0"
-                 izz="1.0" /> -->
-      </inertial>
-    </link>
-  </xacro:macro>
-  <xacro:macro name="stack_wheel_drive" params="parent prefix number x_loc y_loc z_loc roll=0.0 pitch=0.0 yaw=0.0">
-    <joint name="wheel_${prefix}_drive_joint" type="continuous">
-      <origin xyz="${x_loc+0.0019} ${y_loc} ${z_loc}" rpy="${roll} ${pitch} ${yaw}" />
-      <parent link="${parent}" />
-      <child link="wheel_${prefix}_drive_link" />
-      <axis xyz="-1.0 0.0 0.0 " />
-      <limit effort="10" velocity="10" />
-    </joint>
-    <link name="wheel_${prefix}_drive_link">
-      <visual>
-        <origin xyz="0.0 0.0 0.0" rpy="${M_PI/2} 0.0 ${M_PI+M_PI/2.0}" />
-        <geometry>
-          <mesh filename="file://$(find sobit_light_description)/meshes/wheel/wheel_drive.stl" scale="0.001 0.001 0.001" />
-        </geometry>
-        <material name="wheel" />
-      </visual>
-      <collision>
-        <origin xyz="-${0.0055+0.029/2} 0.0 0.0" rpy="${M_PI/2} 0.0 ${M_PI+M_PI/2.0}" />
-        <!-- <origin xyz="0.0 0.0 0.0" rpy="${M_PI/2} 0.0 ${M_PI+M_PI/2.0}" /> -->
-        <geometry>
-          <cylinder radius="${0.144/2}" length="0.029"/>
-          <!-- <mesh filename="file://$(find sobit_light_description)/meshes/wheel/wheel_drive.stl" scale="0.001 0.001 0.001" /> -->
-        </geometry>
-      </collision>
-      <inertial>
-        <origin xyz="-${0.0055+0.029/2} 0.0 0.0" rpy="0.0 0.0 0.0" />
-        <mass value="1" />
-        <inertia ixx="${1/2 *1*(0.144/2)**2}"              ixy="0.0" ixz="0.0"
-                 iyy="${1/12*1*(3*(0.144/2)**2+0.029**2)}" iyz="0.0"
-                 izz="${1/12*1*(3*(0.144/2)**2+0.029**2)}" />
-        <!-- <inertia ixx="1.0" ixy="0.0" ixz="0.0"
-                 iyy="1.0" iyz="0.0"
-                 izz="1.0" /> -->
-      </inertial>
-    </link>
-  </xacro:macro>
-  <xacro:macro name="wheel" params="parent prefix">
-    <xacro:stack_wheel_steer_base parent="${parent}" prefix="f_l" number="1" x_loc= " ${0.210*cos(radians(45.))}" y_loc= " ${0.210*cos(radians(45.))}" z_loc="-0.019" />
-    <xacro:stack_wheel_steer_base parent="${parent}" prefix="b_l" number="2" x_loc= "-${0.210*cos(radians(45.))}" y_loc= " ${0.210*cos(radians(45.))}" z_loc="-0.019" />
-    <xacro:stack_wheel_steer_base parent="${parent}" prefix="b_r" number="3" x_loc= "-${0.210*cos(radians(45.))}" y_loc= "-${0.210*cos(radians(45.))}" z_loc="-0.019" />
-    <xacro:stack_wheel_steer_base parent="${parent}" prefix="f_r" number="4" x_loc= " ${0.210*cos(radians(45.))}" y_loc= "-${0.210*cos(radians(45.))}" z_loc="-0.019" />
-    <xacro:stack_wheel_steer parent="wheel_f_l_steer_base_link" prefix="f_l" number="1" x_loc= "0.013875" y_loc= "0.0" z_loc="-0.032" />
-    <xacro:stack_wheel_steer parent="wheel_b_l_steer_base_link" prefix="b_l" number="2" x_loc= "0.013875" y_loc= "0.0" z_loc="-0.032" />
-    <xacro:stack_wheel_steer parent="wheel_b_r_steer_base_link" prefix="b_r" number="3" x_loc= "0.013875" y_loc= "0.0" z_loc="-0.032" />
-    <xacro:stack_wheel_steer parent="wheel_f_r_steer_base_link" prefix="f_r" number="4" x_loc= "0.013875" y_loc= "0.0" z_loc="-0.032" />
-    <xacro:stack_wheel_drive parent="wheel_f_l_steer_link" prefix="f_l" number="1" x_loc= "0.02" y_loc= "0.0" z_loc="-0.118" />
-    <xacro:stack_wheel_drive parent="wheel_b_l_steer_link" prefix="b_l" number="2" x_loc= "0.02" y_loc= "0.0" z_loc="-0.118" />
-    <xacro:stack_wheel_drive parent="wheel_b_r_steer_link" prefix="b_r" number="3" x_loc= "0.02" y_loc= "0.0" z_loc="-0.118" />
-    <xacro:stack_wheel_drive parent="wheel_f_r_steer_link" prefix="f_r" number="4" x_loc= "0.02" y_loc= "0.0" z_loc="-0.118" />
-  </xacro:macro>
 </robot>
