Commit message: [FIX] lidar sensor with dummy link

File: sobit_light_description/urdf/sensor/lidar.urdf.xacro (robot description, xacro)
@@ -16,4 +16,18 @@
       </inertial>
     </link>
+    <joint name="${prefix}_sim_joint" type="fixed">
+      <parent link="laser_frame" />
+      <child link="sim_laser_frame" />
+      <origin xyz="0.0 0 0.0" rpy="0 0 -${M_PI / 2.0}" />
+    </joint>
+    <link name="sim_laser_frame">
+      <inertial>
+        <origin xyz="0 0 0" rpy="0 0 0" />
+        <mass value="0.2" />
+        <inertia ixx="0.001" ixy="0" ixz="0"
+                 iyy="0.001" iyz="0"
+                 izz="0.001" />
+      </inertial>
+    </link>
   </xacro:macro>
 </robot>
