Commit message: [UPD] del not used tags

File: sobit_light_description/urdf/sensor/mic.urdf.xacro (robot description, xacro)
@@ -29,7 +29,4 @@
       </inertial>
     </link>
-    <!-- <gazebo reference="${prefix}_base_link">
-      <material>Gazebo/Black</material>
-    </gazebo> -->
   </xacro:macro>
 </robot>

File: sobit_light_description/urdf/sensor/speaker.urdf.xacro (robot description, xacro)
@@ -29,7 +29,4 @@
       </inertial>
     </link>
-    <!-- <gazebo reference="${prefix}_base_link">
-      <material>Gazebo/Black</material>
-    </gazebo> -->
   </xacro:macro>
 </robot>
