Commit message: [UPD] upd height of cam

File: sobit_light_description/urdf/sensor/camera_hand.urdf.xacro (robot description, xacro)
@@ -5,5 +5,5 @@
     <!-- Joint - Hand Camera Base -->
     <joint name="${prefix}_base_joint" type="fixed">
-      <origin xyz="0.03685 0.0 0.0408" rpy="0 0 0"/>
+      <origin xyz="0.03685 0.0 0.0438" rpy="0 0 0"/>
       <parent link="${parent}"/>
       <child link="${prefix}_base_link"/>
