Commit message: [UPD] add required base_link

File: sobit_light_description/robots/sobit_light_real_robot.urdf.xacro (robot description, xacro)
@@ -26,4 +26,5 @@
   <xacro:include filename="$(find sobit_light_description)/urdf/gazebo.urdf.xacro" />
   <!-- <link name="base_footprint"/> -->
+  <link name="base_link"/>
   <!-- Connect the previous Links and Joints -->
   <!-- <xacro:base    prefix="base"      parent="base_footprint" /> -->
