Commit message: [UPD] main urdf file

File: sobit_light_description/robots/sobit_light_robot.urdf.xacro (robot description, xacro)
@@ -1,34 +1,43 @@
-<?xml version="1.0" ?>
-<robot name="sobit_light"
-       xmlns:controller="http://playerstage.sourceforge.net/gazebo/xmlschema/#controller"
-       xmlns:interface="http://playerstage.sourceforge.net/gazebo/xmlschema/#interface"
-       xmlns:sensor="http://playerstage.sourceforge.net/gazebo/xmlschema/#sensor"
-       xmlns:xacro="http://www.ros.org/wiki/xacro">
+<?xml version="1.0" encoding="UTF-8" ?>
+<robot name="sobit_light" xmlns:xacro="http://www.ros.org/wiki/xacro">
   <!-- Add Common Xacro: transmissions, colors -->
-  <xacro:include filename="$(find sobit_light_description)/urdf/common.xacro" />
+  <xacro:include filename="$(find sobit_light_description)/urdf/values.urdf.xacro" />
   <xacro:include filename="$(find sobit_light_description)/urdf/materials.urdf.xacro" />
+  <xacro:include filename="$(find sobit_light_description)/urdf/transmission.urdf.xacro" />
   <!-- Add URDF: links, joints -->
   <xacro:include filename="$(find sobit_light_description)/urdf/base/base.urdf.xacro" />
+  <xacro:include filename="$(find sobit_light_description)/urdf/base/plate.urdf.xacro" />
   <xacro:include filename="$(find sobit_light_description)/urdf/arm/arm.urdf.xacro" />
   <xacro:include filename="$(find sobit_light_description)/urdf/hand/hand.urdf.xacro" />
   <xacro:include filename="$(find sobit_light_description)/urdf/back/back.urdf.xacro" />
   <xacro:include filename="$(find sobit_light_description)/urdf/head/head.urdf.xacro" />
-  <xacro:include filename="$(find sobit_light_description)/urdf/sensor/head_camera.urdf.xacro" />
-  <!-- <xacro:include filename="$(find sobit_light_description)/urdf/sensor/hand_camera.urdf.xacro" /> -->
+  <xacro:include filename="$(find sobit_light_description)/urdf/wheel/wheel.urdf.xacro" />
+  <xacro:include filename="$(find sobit_light_description)/urdf/sensor/camera_front.urdf.xacro" />
+  <xacro:include filename="$(find sobit_light_description)/urdf/sensor/camera_back.urdf.xacro" />
+  <xacro:include filename="$(find sobit_light_description)/urdf/sensor/camera_head.urdf.xacro" />
+  <xacro:include filename="$(find sobit_light_description)/urdf/sensor/lidar.urdf.xacro" />
+  <xacro:include filename="$(find sobit_light_description)/urdf/sensor/tof.urdf.xacro" />
+  <xacro:include filename="$(find sobit_light_description)/urdf/sensor/imu.urdf.xacro" />
   <xacro:include filename="$(find sobit_light_description)/urdf/sensor/mic.urdf.xacro" />
   <xacro:include filename="$(find sobit_light_description)/urdf/sensor/speaker.urdf.xacro" />
-  <!-- <xacro:include filename="$(find sobit_light_description)/urdf/sensor/lidar.urdf.xacro" /> -->
-  <xacro:include filename="$(find realsense2_description)/urdf/_d435.urdf.xacro" />
+  <!-- Add URDF: gazebo -->
+  <xacro:include filename="$(find sobit_light_description)/urdf/gazebo.urdf.xacro" />
+  <link name="base_footprint"/>
   <!-- Connect the previous Links and Joints -->
-  <xacro:base/>
-  <!-- <xacro:stack_hexagons parent="base_link" /> -->
-  <!-- <xacro:cover  prefix="cover"  parent="plate_top_link" /> -->
-  <xacro:arm    prefix="arm"     parent="plate_top_link" />
-  <xacro:hand   prefix_hand="hand" prefix_finger="finger" parent="arm_wrist_tilt_link" />
-  <xacro:back   prefix="back"    parent="plate_top_link" />
-  <xacro:head   prefix="head"    parent="back_base_link" />
-  <xacro:head_camera prefix="head_camera" parent="head_camera_tilt_link" />
-  <xacro:mic    prefix="mic"     parent="back_base_link" />
-  <xacro:mic    prefix="speaker" parent="back_base_link" />
-  <!-- <xacro:lidar  prefix="lidar"  parent="plate_bottom_link" /> -->
+  <xacro:base    prefix="base"      parent="base_footprint" />
+  <xacro:plate   prefix="plate"     parent="base_link" />
+  <xacro:arm     prefix="arm"       parent="plate_middle_link" />
+  <xacro:hand    prefix_hand="hand" prefix_finger="finger" parent="arm_gripper_link" />
+  <xacro:back    prefix="back"      parent="plate_bottom_link" />
+  <xacro:head    prefix="head"      parent="back_base_link" />
+  <xacro:wheel   prefix="base"      parent="base_link" />
+  <xacro:lidar   prefix="lidar"     parent="base_link" />
+  <xacro:tof     prefix="tof"       parent="base_link" />
+  <xacro:imu     prefix="imu"       parent="base_link" />
+  <!-- <xacro:mic     prefix="mic"       parent="head_tilt_link" /> -->
+  <xacro:speaker prefix="speaker"   parent="back_base_link" />
+  <xacro:camera_head  prefix="head_camera"  parent="head_tilt_link" />
+  <xacro:camera_front prefix="camera_front" parent="base_link" />
+  <xacro:camera_back  prefix="camera_back"  parent="base_link" />
+  <xacro:gazebo_ros2_control prefix="base" />
 </robot>

Commit message: [ADD] mic

File: sobit_light_description/robots/sobit_light_robot.urdf.xacro (robot description, xacro)
@@ -37,5 +37,5 @@
   <xacro:tof     prefix="tof"       parent="base_link" />
   <xacro:imu     prefix="imu"       parent="base_link" />
-  <!-- <xacro:mic     prefix="mic"       parent="head_pitch_link" /> -->
+  <xacro:mic     prefix="mic"       parent="head_pitch_link" />
   <xacro:speaker prefix="speaker"   parent="back_base_link" />
   <xacro:camera_hand  prefix="hand_camera"  parent="arm_wrist_roll_link" />

File: sobit_light_description/urdf/sensor/mic.urdf.xacro (robot description, xacro)
@@ -2,30 +2,29 @@
 <robot name="mic" xmlns:xacro="http://ros.org/wiki/xacro">
   <xacro:macro name="mic" params="prefix parent">
-    <joint name="${prefix}_base_joint" type="fixed">
+    <joint name="${prefix}_joint" type="fixed">
       <parent link="${parent}" />
-      <child link="${prefix}_base_link" />
-      <origin xyz="0.0 0.0 0.0" rpy="0.0 0.0 0.0" />
+      <child link="${prefix}_link" />
+      <origin xyz="-0.003202 0.0 0.12025" rpy="0.0 0.0 0.0" />
     </joint>
-    <link name="${prefix}_base_link">
+    <link name="${prefix}_link">
       <visual>
-        <origin xyz="0.0 0.0 0.0" rpy="0.0 0.0 ${M_PI/2.0}" />
+        <origin xyz="0.0 0.0 0.0" rpy="-${5.*M_PI/36.} 0.0 ${M_PI/2.0}" />
         <geometry>
-          <mesh filename="file://$(find sobit_light_description)/meshes/sensor/mic.stl"/>
+          <mesh filename="file://$(find sobit_light_description)/meshes/sensor/mic.stl" scale="0.001 0.001 0.001" />
         </geometry>
         <material name="black" />
       </visual>
       <collision>
-        <origin xyz="0.0 0.0 0.0" rpy="0.0 0.0 ${M_PI/2.0}" />
+        <origin xyz="0.0 0.0 0.065" rpy="0.0 -${M_PI/2.+5.*M_PI/36.} 0.0"/>
         <geometry>
-          <mesh filename="file://$(find sobit_light_description)/meshes/sensor/mic.stl" />
+          <cylinder radius="0.0256" length="0.118"/>
         </geometry>
-        <material name="black" />
       </collision>
       <inertial>
-        <origin xyz="0.0 0.0 0.0" rpy="0.0 0.0 ${M_PI/2.0}" />
-        <mass value="0.09507172" />
-        <inertia ixx="${1/12*0.09507172*(0.078**2 + 0.157**2)}" ixy="0.0" ixz="0.0"
-                 iyy="${1/12*0.09507172*(0.026**2 + 0.078**2)}" iyz="0.0"
-                 izz="${1/12*0.09507172*(0.026**2 + 0.157**2)}" />
+        <origin xyz="0.0 0.0 0.065" rpy="0.0 -${M_PI/2.+5.*M_PI/36.} 0.0"/>
+        <mass value="0.0935" />
+        <inertia  ixx="${1/12*0.0935*(3*0.0256**2+0.118**2)}" ixy="0.0" ixz="0.0"
+                  iyy="${1/12*0.0935*(3*0.0256**2+0.118**2)}" iyz="0.0"
+                  izz="${1/12*0.0935*(3*0.0256**2+0.118**2)}" />
       </inertial>
     </link>

Commit message: [UPD] gz support

File: sobit_light_description/robots/sobit_light_robot.urdf.xacro (robot description, xacro)
@@ -25,25 +25,31 @@
   <!-- Add URDF: gazebo -->
   <xacro:include filename="$(find sobit_light_description)/urdf/gazebo.urdf.xacro" />
-  <link name="base_footprint"/>
-  <!-- Connect the previous Links and Joints -->
-  <xacro:base    prefix="base"      parent="base_footprint" />
-  <xacro:plate   prefix="plate"     parent="base_link" />
-  <xacro:arm     prefix="arm"       parent="plate_middle_link" />
-  <xacro:hand    prefix_hand="hand" prefix_finger="finger" parent="arm_hand_link" />
-  <xacro:back    prefix="back"      parent="plate_bottom_link" />
-  <xacro:head    prefix="head"      parent="back_base_link" />
-  <xacro:wheel   prefix="base"      parent="base_link" />
-  <xacro:lidar   prefix="lidar"     parent="base_link" />
-  <xacro:tof     prefix="tof"       parent="base_link" />
-  <xacro:imu     prefix="imu"       parent="base_link" />
-  <xacro:mic     prefix="mic"       parent="head_pitch_link" />
-  <xacro:speaker prefix="speaker"   parent="back_base_link" />
-  <xacro:camera_hand  prefix="hand_camera"  parent="arm_wrist_roll_link" />
-  <xacro:camera_head  prefix="head_camera"  parent="head_pitch_link" />
-  <xacro:camera_front prefix="camera_front" parent="base_link" />
-  <xacro:camera_back  prefix="camera_back"  parent="base_link" />
+  <!-- Add variables -->
+  <xacro:arg name="enable_gz"       default="False" />
+  <!-- Connect the Links and Joints -->
+  <xacro:if value="${$(arg enable_gz)}">
+    <link               name="base_footprint"/>
+    <xacro:base         prefix="base"         parent="base_footprint" />
+    <xacro:wheel        prefix="base"         parent="base_link" />
+    <xacro:lidar        prefix="lidar"        parent="base_link" />
+    <xacro:tof          prefix="tof"          parent="base_link" />
+    <xacro:imu          prefix="imu"          parent="base_link" />
+    <xacro:camera_front prefix="camera_front" parent="base_link" />
+    <xacro:camera_back  prefix="camera_back"  parent="base_link" />
+  </xacro:if>
+  <xacro:plate          prefix="plate"        parent="base_link" />
+  <xacro:arm            prefix="arm"          parent="plate_middle_link" />
+  <xacro:hand           prefix_hand="hand"    prefix_finger="finger" parent="arm_hand_link" />
+  <xacro:back           prefix="back"         parent="plate_bottom_link" />
+  <xacro:head           prefix="head"         parent="back_base_link" />
+  <xacro:mic            prefix="mic"          parent="head_pitch_link" />
+  <xacro:speaker        prefix="speaker"      parent="back_base_link" />
+  <xacro:camera_hand    prefix="hand_camera"  parent="arm_wrist_roll_link" />
+  <xacro:camera_head    prefix="head_camera"  parent="head_pitch_link" />
   <!-- Add Dynamixel: plugins -->
-  <!-- <xacro:dxl_control name="dxl_control" /> -->
+  <xacro:dxl_control name="joints_control" enable_gz="$(arg enable_gz)" />
   <!-- Add Gazebo: plugins -->
-  <xacro:gazebo_ros2_control prefix="base" />
+  <xacro:if value="${$(arg enable_gz)}">
+    <xacro:gazebo_ros2_control prefix="base" />
+  </xacro:if>
 </robot>

Commit message: [UPD] controllers urdf

File: sobit_light_description/robots/sobit_light_robot.urdf.xacro (robot description, xacro)
@@ -5,5 +5,5 @@
   <xacro:include filename="$(find sobit_light_description)/urdf/materials.urdf.xacro" />
   <xacro:include filename="$(find sobit_light_description)/urdf/transmission.urdf.xacro" />
-  <xacro:include filename="$(find sobit_light_description)/urdf/dxl_control.urdf.xacro" />
+  <xacro:include filename="$(find sobit_light_description)/urdf/controllers.urdf.xacro" />
   <!-- Add URDF: links, joints -->
   <xacro:include filename="$(find sobit_light_description)/urdf/base/base.urdf.xacro" />
@@ -48,5 +48,5 @@
   <xacro:camera_head    prefix="head_camera"  parent="head_pitch_link" />
   <!-- Add Dynamixel: plugins -->
-  <xacro:dxl_control name="joints_control" enable_gz="$(arg enable_gz)" />
+  <xacro:controllers name="joints_control" enable_gz="$(arg enable_gz)" />
   <!-- Add Gazebo: plugins -->
   <xacro:if value="${$(arg enable_gz)}">

File: sobit_light_description/urdf/dxl_control.urdf.xacro (robot description, xacro)
@@ -1,7 +1,7 @@
 <?xml version="1.0" encoding="UTF-8" ?>
 <!-- SOBIT Light (Dynamixel Control) -->
-<robot name="sobit_light_dxl_control" xmlns:xacro="http://www.ros.org/wiki/xacro">
-  <xacro:macro name="dxl_control" params="name enable_gz:=False">
-    <ros2_control name="${name}" type="system">
+<robot name="sobit_light_controllers" xmlns:xacro="http://www.ros.org/wiki/xacro">
+  <xacro:macro name="controllers" params="name enable_gz:=False">
+    <ros2_control name="${name}_arm" type="system">
     <!-- <ros2_control name="joints_control" type="system"> -->
       <hardware>
@@ -178,5 +178,5 @@
     <!-- Differential Drive -->
     <xacro:if value="${$(arg enable_gz)}">
-      <ros2_control name="base_control" type="system">
+      <ros2_control name="${name}_base" type="system">
         <hardware>
           <plugin>ign_ros2_control/IgnitionSystem</plugin>
