Commit message: [UPD] toggle gz sensors

File: sobit_light_description/robots/sobit_light_robot.urdf.xacro (robot description, xacro)
@@ -26,6 +26,14 @@
   <xacro:include filename="$(find sobit_light_description)/urdf/gazebo.urdf.xacro" />
   <!-- Add variables -->
-  <xacro:arg name="enable_gz"       default="False" />
-  <xacro:arg name="robot_name"      default="sobit_light" />
+  <xacro:arg name="enable_gz"                 default="False" />
+  <xacro:arg name="enable_gz_front_cam_color" default="True" />
+  <xacro:arg name="enable_gz_back_cam_color"  default="True" />
+  <xacro:arg name="enable_gz_head_cam_color"  default="True" />
+  <xacro:arg name="enable_gz_head_cam_depth"  default="True" />
+  <xacro:arg name="enable_gz_hand_cam_color"  default="True" />
+  <xacro:arg name="enable_gz_hand_cam_depth"  default="True" />
+  <xacro:arg name="enable_gz_lidar"           default="True" />
+  <xacro:arg name="enable_gz_imu"             default="True" />
+  <xacro:arg name="robot_name"                default="sobit_light" />
   <!-- Connect the Links and Joints -->
   <xacro:if value="${$(arg enable_gz)}">
@@ -52,5 +60,14 @@
   <!-- Add Gazebo: plugins -->
   <xacro:if value="${$(arg enable_gz)}">
-    <xacro:gazebo_sensors prefix="base" robot_name="$(arg robot_name)" />
+    <xacro:gazebo_sensors robot_name="$(arg robot_name)"
+      enable_gz_front_cam_color="$(arg enable_gz_front_cam_color)"
+      enable_gz_back_cam_color="$(arg enable_gz_back_cam_color)"
+      enable_gz_head_cam_color="$(arg enable_gz_head_cam_color)"
+      enable_gz_head_cam_depth="$(arg enable_gz_head_cam_depth)"
+      enable_gz_hand_cam_color="$(arg enable_gz_hand_cam_color)"
+      enable_gz_hand_cam_depth="$(arg enable_gz_hand_cam_depth)"
+      enable_gz_lidar="$(arg enable_gz_lidar)"
+      enable_gz_imu="$(arg enable_gz_imu)"
+    />
   </xacro:if>
 </robot>

File: sobit_light_description/urdf/gazebo.urdf.xacro (robot description, xacro)
@@ -2,16 +2,18 @@
 <!-- SOBIT Light (Gazebo) -->
 <robot name="sobit_light_gazebo" xmlns:xacro="http://ros.org/wiki/xacro">
-  <xacro:macro name="gazebo_sensors" params="prefix robot_name">
+  <xacro:macro name="gazebo_sensors" params="robot_name enable_gz_front_cam_color:=True enable_gz_back_cam_color:=True enable_gz_head_cam_color:=True enable_gz_head_cam_depth:=True enable_gz_hand_cam_color:=True enable_gz_hand_cam_depth:=True enable_gz_lidar:=True enable_gz_imu:=True">
     <!-- Sensor: Base Front Camera (Color) -->
-    <gazebo reference="imu_link">
-      <sensor name="imu_sensor" type="imu">
-        <pose>0 0 0 0 0 0</pose>
-        <gz_frame_id>${robot_name}/camera_front_link</gz_frame_id>
-        <topic>${robot_name}/imu</topic>
-        <always_on>1</always_on>
-        <visualize>true</visualize>
-        <update_rate>1</update_rate>
-      </sensor>
-    </gazebo>
+    <xacro:if value="${enable_gz_front_cam_color}">
+      <gazebo reference="imu_link">
+        <sensor name="imu_sensor" type="imu">
+          <pose>0 0 0 0 0 0</pose>
+          <gz_frame_id>${robot_name}/camera_front_link</gz_frame_id>
+          <topic>${robot_name}/imu</topic>
+          <always_on>1</always_on>
+          <visualize>true</visualize>
+          <update_rate>1</update_rate>
+        </sensor>
+      </gazebo>
+    </xacro:if>
     <!-- [TODO] Sensor: Base Front Camera (Color) -->
     <!-- <gazebo reference="camera_front_link">
@@ -49,33 +51,35 @@
     </gazebo> -->
     <!-- Sensor: Base Front Camera (Color) -->
-    <gazebo reference="camera_front_link">
-      <sensor name="base_front_camera_color" type="camera">
-        <pose>0 0 ${0.0175/2} ${M_PI/2} -${M_PI/2} 0 </pose>
-        <ignition_frame_id>${robot_name}/base_front_camera_color</ignition_frame_id>
-        <!-- <gz_frame_id>${robot_name}/base_front_camera_color</gz_frame_id> -->
-        <topic>${robot_name}/base_front_camera/color</topic>
-        <always_on>1</always_on>
-        <visualize>true</visualize>
-        <update_rate>1</update_rate>
-        <camera name="base_front_camera">
-          <horizontal_fov>1.21126</horizontal_fov>
-          <image>
-            <width>640</width>
-            <height>480</height>
-            <format>RGB_INT8</format>
-          </image>
-          <clip>
-            <near>0.1</near>
-            <far>10</far>
-          </clip>
-          <!-- TODO: adjust noise -->
-          <!-- <noise>
-            <type>gaussian</type>
-            <mean>0</mean>
-            <stddev>0.007</stddev>
-          </noise> -->
-        </camera>
-      </sensor>
-    </gazebo>
+    <xacro:if value="${enable_gz_front_cam_color}">
+      <gazebo reference="camera_front_link">
+        <sensor name="base_front_camera_color" type="camera">
+          <pose>0 0 ${0.0175/2} ${M_PI/2} -${M_PI/2} 0 </pose>
+          <ignition_frame_id>${robot_name}/base_front_camera_color</ignition_frame_id>
+          <!-- <gz_frame_id>${robot_name}/base_front_camera_color</gz_frame_id> -->
+          <topic>${robot_name}/base_front_camera/color</topic>
+          <always_on>1</always_on>
+          <visualize>true</visualize>
+          <update_rate>1</update_rate>
+          <camera name="base_front_camera">
+            <horizontal_fov>1.21126</horizontal_fov>
+            <image>
+              <width>640</width>
+              <height>480</height>
+              <format>RGB_INT8</format>
+            </image>
+            <clip>
+              <near>0.1</near>
+              <far>10</far>
+            </clip>
+            <!-- TODO: adjust noise -->
+            <!-- <noise>
+              <type>gaussian</type>
+              <mean>0</mean>
+              <stddev>0.007</stddev>
+            </noise> -->
+          </camera>
+        </sensor>
+      </gazebo>
+    </xacro:if>
     <!-- [TODO] Sensor: Base Back Camera (Color) -->
     <!-- <gazebo reference="camera_back_link">
@@ -113,184 +117,196 @@
     </gazebo> -->
     <!-- Sensor: Base Back Camera (Color) -->
-    <gazebo reference="camera_back_link">
-      <sensor name="base_back_camera_color" type="camera">
-        <pose>0 0 ${0.0175/2} ${M_PI/2} -${M_PI/2} 0 </pose>
-        <ignition_frame_id>${robot_name}/camera_back_link</ignition_frame_id>
-        <!-- <gz_frame_id>${robot_name}/camera_back_link</gz_frame_id> -->
-        <topic>${robot_name}/base_back_camera/color</topic>
-        <always_on>1</always_on>
-        <visualize>true</visualize>
-        <update_rate>1</update_rate>
-        <camera name="base_back_camera">
-          <horizontal_fov>1.21126</horizontal_fov>
-          <image>
-            <width>640</width>
-            <height>480</height>
-            <format>RGB_INT8</format>
-          </image>
-          <clip>
-            <near>0.1</near>
-            <far>10</far>
-          </clip>
-          <!-- TODO: adjust noise -->
-          <!-- <noise>
-            <type>gaussian</type>
-            <mean>0</mean>
-            <stddev>0.007</stddev>
-          </noise> -->
-        </camera>
-      </sensor>
-    </gazebo>
+    <xacro:if value="${enable_gz_back_cam_color}">
+      <gazebo reference="camera_back_link">
+        <sensor name="base_back_camera_color" type="camera">
+          <pose>0 0 ${0.0175/2} ${M_PI/2} -${M_PI/2} 0 </pose>
+          <ignition_frame_id>${robot_name}/camera_back_link</ignition_frame_id>
+          <!-- <gz_frame_id>${robot_name}/camera_back_link</gz_frame_id> -->
+          <topic>${robot_name}/base_back_camera/color</topic>
+          <always_on>1</always_on>
+          <visualize>true</visualize>
+          <update_rate>1</update_rate>
+          <camera name="base_back_camera">
+            <horizontal_fov>1.21126</horizontal_fov>
+            <image>
+              <width>640</width>
+              <height>480</height>
+              <format>RGB_INT8</format>
+            </image>
+            <clip>
+              <near>0.1</near>
+              <far>10</far>
+            </clip>
+            <!-- TODO: adjust noise -->
+            <!-- <noise>
+              <type>gaussian</type>
+              <mean>0</mean>
+              <stddev>0.007</stddev>
+            </noise> -->
+          </camera>
+        </sensor>
+      </gazebo>
+    </xacro:if>
     <!-- Sensor: Head Camera (Color) -->
-    <gazebo reference="head_camera_color_optical_frame">
-      <sensor name="head_camera_color" type="camera">
-        <pose>0 0 ${0.0175/2} ${M_PI/2} -${M_PI/2} 0 </pose>
-        <ignition_frame_id>${robot_name}/head_camera_color_optical_frame</ignition_frame_id>
-        <!-- <gz_frame_id>${robot_name}/head_camera_color_optical_frame</gz_frame_id> -->
-        <topic>${robot_name}/head_camera/color</topic>
-        <always_on>1</always_on>
-        <visualize>true</visualize>
-        <update_rate>1</update_rate>
-        <camera name="head_camera_color">
-          <horizontal_fov>1.21126</horizontal_fov>
-          <image>
-            <width>640</width>
-            <height>480</height>
-            <format>RGB_INT8</format>
-          </image>
-          <clip>
-            <near>0.1</near>
-            <far>10</far>
-          </clip>
-          <!-- TODO: adjust noise -->
-          <!-- <noise>
-            <type>gaussian</type>
-            <mean>0</mean>
-            <stddev>0.007</stddev>
-          </noise> -->
-        </camera>
-      </sensor>
-    </gazebo>
+    <xacro:if value="${enable_gz_head_cam_color}">
+      <gazebo reference="head_camera_color_optical_frame">
+        <sensor name="head_camera_color" type="camera">
+          <pose>0 0 ${0.0175/2} ${M_PI/2} -${M_PI/2} 0 </pose>
+          <ignition_frame_id>${robot_name}/head_camera_color_optical_frame</ignition_frame_id>
+          <!-- <gz_frame_id>${robot_name}/head_camera_color_optical_frame</gz_frame_id> -->
+          <topic>${robot_name}/head_camera/color</topic>
+          <always_on>1</always_on>
+          <visualize>true</visualize>
+          <update_rate>1</update_rate>
+          <camera name="head_camera_color">
+            <horizontal_fov>1.21126</horizontal_fov>
+            <image>
+              <width>640</width>
+              <height>480</height>
+              <format>RGB_INT8</format>
+            </image>
+            <clip>
+              <near>0.1</near>
+              <far>10</far>
+            </clip>
+            <!-- TODO: adjust noise -->
+            <!-- <noise>
+              <type>gaussian</type>
+              <mean>0</mean>
+              <stddev>0.007</stddev>
+            </noise> -->
+          </camera>
+        </sensor>
+      </gazebo>
+    </xacro:if>
     <!-- Sensor: Head Camera (Depth) -->
-    <gazebo reference="head_camera_depth_optical_frame">
-      <sensor name="head_camera_depth" type="depth">
-        <pose>0 0 ${0.0175/2} ${M_PI/2} -${M_PI/2} 0 </pose>
-        <ignition_frame_id>${robot_name}/head_camera_depth_optical_frame</ignition_frame_id>
-        <!-- <gz_frame_id>${robot_name}/head_camera_depth_optical_frame</gz_frame_id> -->
-        <topic>${robot_name}/head_camera/depth</topic>
-        <always_on>1</always_on>
-        <visualize>true</visualize>
-        <update_rate>1</update_rate>
-        <camera name="head_camera_depth">
-          <horizontal_fov>1.48702</horizontal_fov>
-          <image>
-            <width>1280</width>
-            <height>720</height>
-          </image>
-          <clip>
-            <near>0.1</near>
-            <far>10</far>
-          </clip>
-          <!-- TODO: adjust noise -->
-          <!-- <noise>
-            <type>gaussian</type>
-            <mean>0</mean>
-            <stddev>0.1</stddev>
-          </noise> -->
-        </camera>
-      </sensor>
-    </gazebo>
+    <xacro:if value="${enable_gz_head_cam_depth}">
+      <gazebo reference="head_camera_depth_optical_frame">
+        <sensor name="head_camera_depth" type="depth">
+          <pose>0 0 ${0.0175/2} ${M_PI/2} -${M_PI/2} 0 </pose>
+          <ignition_frame_id>${robot_name}/head_camera_depth_optical_frame</ignition_frame_id>
+          <!-- <gz_frame_id>${robot_name}/head_camera_depth_optical_frame</gz_frame_id> -->
+          <topic>${robot_name}/head_camera/depth</topic>
+          <always_on>1</always_on>
+          <visualize>true</visualize>
+          <update_rate>1</update_rate>
+          <camera name="head_camera_depth">
+            <horizontal_fov>1.48702</horizontal_fov>
+            <image>
+              <width>1280</width>
+              <height>720</height>
+            </image>
+            <clip>
+              <near>0.1</near>
+              <far>10</far>
+            </clip>
+            <!-- TODO: adjust noise -->
+            <!-- <noise>
+              <type>gaussian</type>
+              <mean>0</mean>
+              <stddev>0.1</stddev>
+            </noise> -->
+          </camera>
+        </sensor>
+      </gazebo>
+    </xacro:if>
     <!-- Sensor: Hand Camera (Color) -->
-    <gazebo reference="hand_camera_color_optical_frame">
-      <sensor name="hand_camera_color" type="camera">
-        <pose>0 0 ${0.0175/2} ${M_PI/2} -${M_PI/2} 0 </pose>
-        <ignition_frame_id>${robot_name}/hand_camera_color_optical_frame</ignition_frame_id>
-        <!-- <gz_frame_id>${robot_name}/hand_camera_color_optical_frame</gz_frame_id> -->
-        <topic>${robot_name}/hand_camera/color</topic>
-        <always_on>1</always_on>
-        <visualize>true</visualize>
-        <update_rate>1</update_rate>
-        <camera name="hand_camera_color">
-          <horizontal_fov>1.21126</horizontal_fov>
-          <image>
-            <width>640</width>
-            <height>480</height>
-            <format>RGB_INT8</format>
-          </image>
-          <clip>
-            <near>0.1</near>
-            <far>10</far>
-          </clip>
-          <!-- TODO: adjust noise -->
-          <!-- <noise>
-            <type>gaussian</type>
-            <mean>0</mean>
-            <stddev>0.007</stddev>
-          </noise> -->
-        </camera>
-      </sensor>
-    </gazebo>
+    <xacro:if value="${enable_gz_hand_cam_color}">
+      <gazebo reference="hand_camera_color_optical_frame">
+        <sensor name="hand_camera_color" type="camera">
+          <pose>0 0 ${0.0175/2} ${M_PI/2} -${M_PI/2} 0 </pose>
+          <ignition_frame_id>${robot_name}/hand_camera_color_optical_frame</ignition_frame_id>
+          <!-- <gz_frame_id>${robot_name}/hand_camera_color_optical_frame</gz_frame_id> -->
+          <topic>${robot_name}/hand_camera/color</topic>
+          <always_on>1</always_on>
+          <visualize>true</visualize>
+          <update_rate>1</update_rate>
+          <camera name="hand_camera_color">
+            <horizontal_fov>1.21126</horizontal_fov>
+            <image>
+              <width>640</width>
+              <height>480</height>
+              <format>RGB_INT8</format>
+            </image>
+            <clip>
+              <near>0.1</near>
+              <far>10</far>
+            </clip>
+            <!-- TODO: adjust noise -->
+            <!-- <noise>
+              <type>gaussian</type>
+              <mean>0</mean>
+              <stddev>0.007</stddev>
+            </noise> -->
+          </camera>
+        </sensor>
+      </gazebo>
+    </xacro:if>
     <!-- Sensor: Hand Camera (Depth) -->
-    <gazebo reference="hand_camera_depth_optical_frame">
-      <sensor name="hand_camera_depth" type="depth">
-        <pose>0 0 ${0.0175/2} ${M_PI/2} -${M_PI/2} 0 </pose>
-        <ignition_frame_id>${robot_name}/hand_camera_depth_optical_frame</ignition_frame_id>
-        <!-- <gz_frame_id>${robot_name}/hand_camera_depth_optical_frame</gz_frame_id> -->
-        <topic>${robot_name}/hand_camera/depth</topic>
-        <always_on>1</always_on>
-        <visualize>true</visualize>
-        <update_rate>1</update_rate>
-        <camera name="head_camera_depth">
-          <horizontal_fov>1.48702</horizontal_fov>
-          <image>
-            <width>1280</width>
-            <height>720</height>
-          </image>
-          <clip>
-            <near>0.1</near>
-            <far>10</far>
-          </clip>
-          <!-- TODO: adjust noise -->
-          <!-- <noise>
-            <type>gaussian</type>
-            <mean>0</mean>
-            <stddev>0.1</stddev>
-          </noise> -->
-        </camera>
-      </sensor>
-    </gazebo>
+    <xacro:if value="${enable_gz_hand_cam_depth}">
+      <gazebo reference="hand_camera_depth_optical_frame">
+        <sensor name="hand_camera_depth" type="depth">
+          <pose>0 0 ${0.0175/2} ${M_PI/2} -${M_PI/2} 0 </pose>
+          <ignition_frame_id>${robot_name}/hand_camera_depth_optical_frame</ignition_frame_id>
+          <!-- <gz_frame_id>${robot_name}/hand_camera_depth_optical_frame</gz_frame_id> -->
+          <topic>${robot_name}/hand_camera/depth</topic>
+          <always_on>1</always_on>
+          <visualize>true</visualize>
+          <update_rate>1</update_rate>
+          <camera name="head_camera_depth">
+            <horizontal_fov>1.48702</horizontal_fov>
+            <image>
+              <width>1280</width>
+              <height>720</height>
+            </image>
+            <clip>
+              <near>0.1</near>
+              <far>10</far>
+            </clip>
+            <!-- TODO: adjust noise -->
+            <!-- <noise>
+              <type>gaussian</type>
+              <mean>0</mean>
+              <stddev>0.1</stddev>
+            </noise> -->
+          </camera>
+        </sensor>
+      </gazebo>
+    </xacro:if>
     <!-- Sensor: LiDAR -->
-    <gazebo reference="sim_laser_frame">
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
Commit message: [UPD] include kachaka model from kachaka-api

File: sobit_light_description/robots/sobit_light_robot.urdf.xacro (robot description, xacro)
@@ -25,4 +25,7 @@
   <!-- Add URDF: gazebo -->
   <xacro:include filename="$(find sobit_light_description)/urdf/gazebo.urdf.xacro" />
+  <!-- Add Kachaka -->
+  <xacro:include filename="$(find kachaka_description)/urdf/_values.urdf.xacro" />
+  <xacro:include filename="$(find kachaka_description)/urdf/_kachaka.urdf.xacro" />
   <!-- Add variables -->
   <xacro:arg name="enable_gz"                 default="False" />
@@ -37,14 +40,8 @@
   <xacro:arg name="robot_name"                default="sobit_light" />
   <!-- Connect the Links and Joints -->
-  <xacro:if value="${$(arg enable_gz)}">
-    <link               name="base_footprint"/>
-    <xacro:base         prefix="base"         parent="base_footprint" />
-    <xacro:wheel        prefix="base"         parent="base_link" />
-    <xacro:lidar        prefix="lidar"        parent="base_link" />
-    <xacro:tof          prefix="tof"          parent="base_link" />
-    <xacro:imu          prefix="imu"          parent="base_link" />
-    <xacro:camera_front prefix="camera_front" parent="base_link" />
-    <xacro:camera_back  prefix="camera_back"  parent="base_link" />
-  </xacro:if>
+  <link name="base_footprint" />
+  <xacro:kachaka_robot parent="base_footprint">
+    <origin xyz="0 0 0" rpy="0 0 0"/>
+  </xacro:kachaka_robot>
   <xacro:plate          prefix="plate"        parent="base_link" />
   <xacro:arm            prefix="arm"          parent="plate_middle_link" />

Commit message: [FEAT] toggle robot parts

File: sobit_light_description/robots/sobit_light_robot.urdf.xacro (robot description, xacro)
@@ -39,18 +39,57 @@
   <xacro:arg name="enable_gz_imu"             default="True" />
   <xacro:arg name="robot_name"                default="sobit_light" />
+  <!-- Activate Components -->
+  <xacro:arg name="enable_mobile_base"  default="True" />
+  <xacro:arg name="enable_head"         default="True" />
+  <xacro:arg name="enable_arm"          default="True" />
+  <xacro:arg name="enable_hand"         default="True" />
+  <!-- DXL Ports -->
+  <xacro:arg name="dxl_sl_port"  default="/dev/ttyUSB0" />
   <!-- Connect the Links and Joints -->
   <link name="base_footprint" />
-  <xacro:kachaka_robot parent="base_footprint">
-    <origin xyz="0 0 0" rpy="0 0 0"/>
-  </xacro:kachaka_robot>
-  <xacro:plate          prefix="plate"        parent="base_link" />
-  <xacro:arm            prefix="arm"          parent="plate_middle_link" />
-  <xacro:hand           prefix_hand="hand"    prefix_finger="finger" parent="arm_wrist_roll_link" />
-  <xacro:back           prefix="back"         parent="plate_bottom_link" />
-  <xacro:head           prefix="head"         parent="back_base_link" />
-  <xacro:mic            prefix="mic"          parent="head_pitch_link" />
-  <xacro:speaker        prefix="speaker"      parent="back_base_link" />
-  <xacro:camera_hand    prefix="hand_camera"  parent="arm_wrist_roll_link" />
-  <xacro:camera_head    prefix="head_camera"  parent="head_pitch_link" />
+  <xacro:if value="${$(arg enable_mobile_base)}">
+    <xacro:kachaka_robot parent="base_footprint">
+      <origin xyz="0 0 0" rpy="0 0 0"/>
+    </xacro:kachaka_robot>
+  </xacro:if>
+  <xacro:unless value="${$(arg enable_mobile_base)}">
+    <joint name="base_footprint_joint" type="fixed" >
+      <origin xyz="0.0 0.0 0.0" rpy="0.0 0.0 0.0" />
+      <parent link="base_footprint" />
+      <child link="base_link" />
+    </joint>
+    <link name="base_link">
+      <collision>
+        <origin xyz="0.0435 0.0 0.0475"
+                rpy="0 0 0" />
+        <geometry>
+          <box size="0.387 0.240 0.095" />
+        </geometry>
+      </collision>
+    </link>
+  </xacro:unless>
+  <xacro:plate         prefix="plate"        parent="base_link" />
+  <xacro:if value="${$(arg enable_arm)}">
+    <xacro:arm         prefix="arm"          parent="plate_middle_link" />
+  </xacro:if>
+  <xacro:unless value="${$(arg enable_arm)}">
+    <joint name="arm_wrist_roll_joint" type="fixed" >
+      <origin xyz="${0.122+0.26624862} 0.0 0.18032586" rpy="0.0 0.0 0.0" />
+      <parent link="plate_middle_link" />
+      <child link="arm_wrist_roll_link" />
+    </joint>
+    <link name="arm_wrist_roll_link" />
+  </xacro:unless>
+  <xacro:if value="${$(arg enable_hand)}">
+    <xacro:hand        prefix_hand="hand"    prefix_finger="finger" parent="arm_wrist_roll_link" />
+    <xacro:camera_hand prefix="hand_camera"  parent="arm_wrist_roll_link" />
+  </xacro:if>
+  <xacro:if value="${$(arg enable_head)}">
+    <xacro:back        prefix="back"         parent="plate_bottom_link" />
+    <xacro:head        prefix="head"         parent="back_base_link" />
+    <xacro:mic         prefix="mic"          parent="head_pitch_link" />
+    <xacro:speaker     prefix="speaker"      parent="back_base_link" />
+    <xacro:camera_head prefix="head_camera"  parent="head_pitch_link" />
+  </xacro:if>
   <!-- Add Dynamixel: plugins -->
   <xacro:controllers name="joints_control" enable_gz="$(arg enable_gz)" robot_name="$(arg robot_name)" />
