Commit message: feat(bringup): sim camera parity with the real drivers
Colour topics take the driver's <cam>/color/image_raw + color/camera_info
names, depth gets its own bridge on <cam>/depth/image_rect_raw +
depth/camera_info with the optical frame id, JPEG/PNG republishers add
/compressed and /compressedDepth, and camera_rate replaces the
hard-coded 1 Hz.

Co-Authored-By: Claude Fable 5.1 <noreply@anthropic.com>

File: sobit_light_description/robots/sobit_light_robot.urdf.xacro (robot description, xacro)
@@ -36,4 +36,5 @@
   <xacro:arg name="enable_gz_lidar"           default="True" />
   <xacro:arg name="enable_gz_imu"             default="True" />
+  <xacro:arg name="camera_rate"               default="10" />
   <xacro:arg name="robot_name"                default="sobit_light" />
   <!-- Must match the frame_prefix given to robot_state_publisher. -->
@@ -106,4 +107,5 @@
       enable_gz_lidar="$(arg enable_gz_lidar)"
       enable_gz_imu="$(arg enable_gz_imu)"
+      camera_rate="$(arg camera_rate)"
     />
   </xacro:if>

File: sobit_light_description/urdf/gazebo.urdf.xacro (robot description, xacro)
@@ -2,5 +2,5 @@
 <!-- SOBIT Light (Gazebo) -->
 <robot name="sobit_light_gazebo" xmlns:xacro="http://ros.org/wiki/xacro">
-  <xacro:macro name="gazebo_sensors" params="robot_name enable_tf_prefix:=True enable_gz_front_cam_color:=True enable_gz_back_cam_color:=True enable_gz_head_cam_color:=True enable_gz_head_cam_depth:=True enable_gz_hand_cam_color:=True enable_gz_hand_cam_depth:=True enable_gz_lidar:=True enable_gz_imu:=True">
+  <xacro:macro name="gazebo_sensors" params="robot_name enable_tf_prefix:=True enable_gz_front_cam_color:=True enable_gz_back_cam_color:=True enable_gz_head_cam_color:=True enable_gz_head_cam_depth:=True enable_gz_hand_cam_color:=True enable_gz_hand_cam_depth:=True enable_gz_lidar:=True enable_gz_imu:=True camera_rate:=10">
     <!-- Sensor frame ids must match the TF tree: prefixed only when
          robot_state_publisher runs with frame_prefix (enable_tf_prefix). -->
@@ -85,9 +85,9 @@
         <sensor name="base_front_camera_color" type="camera">
           <pose>0 0 ${0.0175/2} ${M_PI/2} -${M_PI/2} 0 </pose>
-          <gz_frame_id>${tf_prefix}base_front_camera_color</gz_frame_id>
+          <gz_frame_id>${tf_prefix}camera_front_link</gz_frame_id>
           <topic>${robot_name}/base_front_camera/color</topic>
           <always_on>1</always_on>
           <visualize>true</visualize>
-          <update_rate>1</update_rate>
+          <update_rate>${camera_rate}</update_rate>
           <camera name="base_front_camera">
             <horizontal_fov>1.21126</horizontal_fov>
@@ -154,5 +154,5 @@
           <always_on>1</always_on>
           <visualize>true</visualize>
-          <update_rate>1</update_rate>
+          <update_rate>${camera_rate}</update_rate>
           <camera name="base_back_camera">
             <horizontal_fov>1.21126</horizontal_fov>
@@ -185,5 +185,5 @@
           <always_on>1</always_on>
           <visualize>true</visualize>
-          <update_rate>1</update_rate>
+          <update_rate>${camera_rate}</update_rate>
           <camera name="head_camera_color">
             <horizontal_fov>1.21126</horizontal_fov>
@@ -216,5 +216,5 @@
           <always_on>1</always_on>
           <visualize>true</visualize>
-          <update_rate>1</update_rate>
+          <update_rate>${camera_rate}</update_rate>
           <camera name="head_camera_depth">
             <horizontal_fov>1.21126</horizontal_fov>
@@ -246,5 +246,5 @@
           <always_on>1</always_on>
           <visualize>true</visualize>
-          <update_rate>1</update_rate>
+          <update_rate>${camera_rate}</update_rate>
           <camera name="hand_camera_color">
             <horizontal_fov>1.21126</horizontal_fov>
@@ -277,5 +277,5 @@
           <always_on>1</always_on>
           <visualize>true</visualize>
-          <update_rate>1</update_rate>
+          <update_rate>${camera_rate}</update_rate>
           <camera name="hand_camera_depth">
             <horizontal_fov>1.21126</horizontal_fov>

Commit message: Fix the simulated cameras at 10 Hz instead of an argument
camera_rate is deferred, so the rate it carried becomes the literal the
macro used to default to. The parity work it arrived with stays: the
driver's topic names, the depth bridge with its optical frame id, and the
compression republishers.

Co-Authored-By: Claude Opus 5 (1M context) <noreply@anthropic.com>

File: sobit_light_description/robots/sobit_light_robot.urdf.xacro (robot description, xacro)
@@ -36,5 +36,4 @@
   <xacro:arg name="enable_gz_lidar"           default="True" />
   <xacro:arg name="enable_gz_imu"             default="True" />
-  <xacro:arg name="camera_rate"               default="10" />
   <xacro:arg name="robot_name"                default="sobit_light" />
   <!-- Must match the frame_prefix given to robot_state_publisher. -->
@@ -107,5 +106,4 @@
       enable_gz_lidar="$(arg enable_gz_lidar)"
       enable_gz_imu="$(arg enable_gz_imu)"
-      camera_rate="$(arg camera_rate)"
     />
   </xacro:if>

File: sobit_light_description/urdf/gazebo.urdf.xacro (robot description, xacro)
@@ -2,5 +2,5 @@
 <!-- SOBIT Light (Gazebo) -->
 <robot name="sobit_light_gazebo" xmlns:xacro="http://ros.org/wiki/xacro">
-  <xacro:macro name="gazebo_sensors" params="robot_name enable_tf_prefix:=True enable_gz_front_cam_color:=True enable_gz_back_cam_color:=True enable_gz_head_cam_color:=True enable_gz_head_cam_depth:=True enable_gz_hand_cam_color:=True enable_gz_hand_cam_depth:=True enable_gz_lidar:=True enable_gz_imu:=True camera_rate:=10">
+  <xacro:macro name="gazebo_sensors" params="robot_name enable_tf_prefix:=True enable_gz_front_cam_color:=True enable_gz_back_cam_color:=True enable_gz_head_cam_color:=True enable_gz_head_cam_depth:=True enable_gz_hand_cam_color:=True enable_gz_hand_cam_depth:=True enable_gz_lidar:=True enable_gz_imu:=True">
     <!-- Sensor frame ids must match the TF tree: prefixed only when
          robot_state_publisher runs with frame_prefix (enable_tf_prefix). -->
@@ -89,5 +89,5 @@
           <always_on>1</always_on>
           <visualize>true</visualize>
-          <update_rate>${camera_rate}</update_rate>
+          <update_rate>10</update_rate>
           <camera name="base_front_camera">
             <horizontal_fov>1.21126</horizontal_fov>
@@ -154,5 +154,5 @@
           <always_on>1</always_on>
           <visualize>true</visualize>
-          <update_rate>${camera_rate}</update_rate>
+          <update_rate>10</update_rate>
           <camera name="base_back_camera">
             <horizontal_fov>1.21126</horizontal_fov>
@@ -185,5 +185,5 @@
           <always_on>1</always_on>
           <visualize>true</visualize>
-          <update_rate>${camera_rate}</update_rate>
+          <update_rate>10</update_rate>
           <camera name="head_camera_color">
             <horizontal_fov>1.21126</horizontal_fov>
@@ -216,5 +216,5 @@
           <always_on>1</always_on>
           <visualize>true</visualize>
-          <update_rate>${camera_rate}</update_rate>
+          <update_rate>10</update_rate>
           <camera name="head_camera_depth">
             <horizontal_fov>1.21126</horizontal_fov>
@@ -246,5 +246,5 @@
           <always_on>1</always_on>
           <visualize>true</visualize>
-          <update_rate>${camera_rate}</update_rate>
+          <update_rate>10</update_rate>
           <camera name="hand_camera_color">
             <horizontal_fov>1.21126</horizontal_fov>
@@ -277,5 +277,5 @@
           <always_on>1</always_on>
           <visualize>true</visualize>
-          <update_rate>${camera_rate}</update_rate>
+          <update_rate>10</update_rate>
           <camera name="hand_camera_depth">
             <horizontal_fov>1.21126</horizontal_fov>

Commit message: Accept either case for enable_gz
${...} evaluates a Python literal, so only True and False parsed and the
lowercase spelling a launch file accepts failed outright against xacro.
The argument is normalized once into a gz_on property, which every test
then reads, so true, True and 1 all work.

Co-Authored-By: Claude Opus 5 (1M context) <noreply@anthropic.com>

File: sobit_light_description/robots/sobit_light_robot.urdf.xacro (robot description, xacro)
@@ -39,4 +39,6 @@
   <!-- Must match the frame_prefix given to robot_state_publisher. -->
   <xacro:arg name="enable_tf_prefix"          default="True" />
+  <!-- ${...} evaluates a Python literal, where only True/False parse. -->
+  <xacro:property name="gz_on" value="${'$(arg enable_gz)'.lower() in ('true', '1')}" />
   <!-- Activate Components -->
   <xacro:arg name="enable_mobile_base"  default="True" />
@@ -93,7 +95,7 @@
   </xacro:if>
   <!-- Add Dynamixel: plugins -->
-  <xacro:controllers name="joints_control" enable_gz="$(arg enable_gz)" robot_name="$(arg robot_name)" />
+  <xacro:controllers name="joints_control" enable_gz="${gz_on}" robot_name="$(arg robot_name)" />
   <!-- Add Gazebo: plugins -->
-  <xacro:if value="${$(arg enable_gz)}">
+  <xacro:if value="${gz_on}">
     <xacro:gazebo_sensors robot_name="$(arg robot_name)"
       enable_tf_prefix="$(arg enable_tf_prefix)"

File: sobit_light_description/urdf/controllers.urdf.xacro (robot description, xacro)
@@ -5,8 +5,8 @@
     <ros2_control name="dynamixel_controllers" type="system">
       <hardware>
-        <xacro:if value="${$(arg enable_gz)}">
+        <xacro:if value="${gz_on}">
           <plugin>gz_ros2_control/GazeboSimSystem</plugin>
         </xacro:if>
-        <xacro:unless value="${$(arg enable_gz)}">
+        <xacro:unless value="${gz_on}">
           <xacro:property name="dxl_sl_port" value="$(arg dxl_sl_port)"/>
           <plugin>dynamixel_hardware/DynamixelHardware</plugin>
@@ -16,18 +16,18 @@
       </hardware>
       <xacro:if value="${$(arg enable_head)}">
-        <xacro:dxl_head_controllers prefix="head"  enable_gz="${$(arg enable_gz)}"/>
+        <xacro:dxl_head_controllers prefix="head"  enable_gz="${gz_on}"/>
       </xacro:if>
       <xacro:if value="${$(arg enable_arm)}">
-        <xacro:dxl_arm_controllers  prefix="arm"   enable_gz="${$(arg enable_gz)}"/>
+        <xacro:dxl_arm_controllers  prefix="arm"   enable_gz="${gz_on}"/>
       </xacro:if>
       <xacro:if value="${$(arg enable_hand)}">
-        <xacro:dxl_hand_controllers prefix="hand"  enable_gz="${$(arg enable_gz)}"/>
+        <xacro:dxl_hand_controllers prefix="hand"  enable_gz="${gz_on}"/>
       </xacro:if>
       <xacro:if value="${$(arg enable_mobile_base)}">
-        <xacro:wheel_controllers    prefix="wheel" enable_gz="${$(arg enable_gz)}"/>
+        <xacro:wheel_controllers    prefix="wheel" enable_gz="${gz_on}"/>
       </xacro:if>
     </ros2_control>
     <!-- Gazebo ROS2 Control -->
-    <xacro:if value="${$(arg enable_gz)}">
+    <xacro:if value="${gz_on}">
       <gazebo>
         <plugin filename="gz_ros2_control-system" name="gz_ros2_control::GazeboSimROS2ControlPlugin">
@@ -43,5 +43,5 @@
     <!-- Position Drive - Head -->
     <joint name="${prefix}_yaw_joint">
-      <xacro:unless value="${$(arg enable_gz)}">
+      <xacro:unless value="${gz_on}">
         <param name="id">11</param>
         <param name="control_mode">0</param>
@@ -60,5 +60,5 @@
     </joint>
     <joint name="${prefix}_pitch_joint">
-      <xacro:unless value="${$(arg enable_gz)}">
+      <xacro:unless value="${gz_on}">
         <param name="id">12</param>
         <param name="control_mode">0</param>
@@ -80,5 +80,5 @@
     <!-- Position Drive - Arm -->
     <joint name="${prefix}_shoulder_roll_joint">
-      <xacro:unless value="${$(arg enable_gz)}">
+      <xacro:unless value="${gz_on}">
         <param name="id">1</param>
         <param name="control_mode">0</param>
@@ -97,5 +97,5 @@
     </joint>
     <joint name="${prefix}_shoulder_pitch_joint">
-      <xacro:unless value="${$(arg enable_gz)}">
+      <xacro:unless value="${gz_on}">
         <param name="id">3</param>
         <param name="control_mode">0</param>
@@ -114,5 +114,5 @@
     </joint>
     <joint name="${prefix}_elbow_pitch_joint">
-      <xacro:unless value="${$(arg enable_gz)}">
+      <xacro:unless value="${gz_on}">
         <param name="id">4</param>
         <param name="control_mode">0</param>
@@ -131,5 +131,5 @@
     </joint>
     <joint name="${prefix}_forearm_roll_joint">
-      <xacro:unless value="${$(arg enable_gz)}">
+      <xacro:unless value="${gz_on}">
         <param name="id">5</param>
         <param name="control_mode">0</param>
@@ -148,5 +148,5 @@
     </joint>
     <joint name="${prefix}_wrist_pitch_joint">
-      <xacro:unless value="${$(arg enable_gz)}">
+      <xacro:unless value="${gz_on}">
         <param name="id">6</param>
         <param name="control_mode">0</param>
@@ -165,5 +165,5 @@
     </joint>
     <joint name="${prefix}_wrist_roll_joint">
-      <xacro:unless value="${$(arg enable_gz)}">
+      <xacro:unless value="${gz_on}">
         <param name="id">7</param>
         <param name="control_mode">0</param>
@@ -185,5 +185,5 @@
     <!-- Position Drive - Hand -->
     <joint name="${prefix}_joint">
-      <xacro:unless value="${$(arg enable_gz)}">
+      <xacro:unless value="${gz_on}">
         <param name="id">8</param>
         <param name="control_mode">6</param>
@@ -200,5 +200,5 @@
       <!-- <state_interface name="effort"/> -->
     </joint>
-    <xacro:if value="${$(arg enable_gz)}">
+    <xacro:if value="${gz_on}">
       <joint name="${prefix}_sub_joint">
         <param name="mimic">${prefix}_joint</param>
@@ -212,5 +212,5 @@
   </xacro:macro>
   <xacro:macro name="wheel_controllers"  params="prefix enable_gz:=False">
-    <xacro:if value="${$(arg enable_gz)}">
+    <xacro:if value="${gz_on}">
         <joint name="base_l_drive_wheel_joint">
           <command_interface name="velocity">
