Commit message: feat(description): add enable_tf_prefix toggle
Frame prefix on robot_state_publisher and gz sensor frame ids is now
optional, matching sobit_home. Default true keeps current behavior.

File: sobit_light_description/robots/sobit_light_robot.urdf.xacro (robot description, xacro)
@@ -37,4 +37,6 @@
   <xacro:arg name="enable_gz_imu"             default="True" />
   <xacro:arg name="robot_name"                default="sobit_light" />
+  <!-- Must match the frame_prefix given to robot_state_publisher. -->
+  <xacro:arg name="enable_tf_prefix"          default="True" />
   <!-- Activate Components -->
   <xacro:arg name="enable_mobile_base"  default="True" />
@@ -95,4 +97,5 @@
   <xacro:if value="${$(arg enable_gz)}">
     <xacro:gazebo_sensors robot_name="$(arg robot_name)"
+      enable_tf_prefix="$(arg enable_tf_prefix)"
       enable_gz_front_cam_color="$(arg enable_gz_front_cam_color)"
       enable_gz_back_cam_color="$(arg enable_gz_back_cam_color)"

File: sobit_light_description/urdf/gazebo.urdf.xacro (robot description, xacro)
@@ -2,5 +2,8 @@
 <!-- SOBIT Light (Gazebo) -->
 <robot name="sobit_light_gazebo" xmlns:xacro="http://ros.org/wiki/xacro">
-  <xacro:macro name="gazebo_sensors" params="robot_name enable_gz_front_cam_color:=True enable_gz_back_cam_color:=True enable_gz_head_cam_color:=True enable_gz_head_cam_depth:=True enable_gz_hand_cam_color:=True enable_gz_hand_cam_depth:=True enable_gz_lidar:=True enable_gz_imu:=True">
+  <xacro:macro name="gazebo_sensors" params="robot_name enable_tf_prefix:=True enable_gz_front_cam_color:=True enable_gz_back_cam_color:=True enable_gz_head_cam_color:=True enable_gz_head_cam_depth:=True enable_gz_hand_cam_color:=True enable_gz_hand_cam_depth:=True enable_gz_lidar:=True enable_gz_imu:=True">
+    <!-- Sensor frame ids must match the TF tree: prefixed only when
+         robot_state_publisher runs with frame_prefix (enable_tf_prefix). -->
+    <xacro:property name="tf_prefix" value="${robot_name + '/' if str(enable_tf_prefix).lower() == 'true' else ''}"/>
     <!-- Friction and Contact Parameters for Mobile Base -->
     <xacro:if value="${$(arg enable_gz_front_cam_color) and $(arg enable_mobile_base)}">
@@ -63,5 +66,5 @@
         <sensor name="imu_sensor" type="imu">
           <pose>0 0 0 0 0 0</pose>
-          <gz_frame_id>${robot_name}/imu_link</gz_frame_id>
+          <gz_frame_id>${tf_prefix}imu_link</gz_frame_id>
           <topic>${robot_name}/imu</topic>
           <always_on>1</always_on>
@@ -75,5 +78,5 @@
       <sensor name="base_front_camera_color" type="wideanglecamera">
         <pose>0 0 ${0.0175/2} ${M_PI/2} -${M_PI/2} 0 </pose>
-        <gz_frame_id>${robot_name}/camera_front_link</gz_frame_id>
+        <gz_frame_id>${tf_prefix}camera_front_link</gz_frame_id>
         <topic>${robot_name}/base_front_camera/color</topic>
         <always_on>1</always_on>
@@ -110,5 +113,5 @@
         <sensor name="base_front_camera_color" type="camera">
           <pose>0 0 ${0.0175/2} ${M_PI/2} -${M_PI/2} 0 </pose>
-          <gz_frame_id>${robot_name}/base_front_camera_color</gz_frame_id>
+          <gz_frame_id>${tf_prefix}base_front_camera_color</gz_frame_id>
           <topic>${robot_name}/base_front_camera/color</topic>
           <always_on>1</always_on>
@@ -140,5 +143,5 @@
       <sensor name="base_back_camera_color" type="wideanglecamera">
         <pose>0 0 ${0.0175/2} ${M_PI/2} -${M_PI/2} 0 </pose>
-        <gz_frame_id>${robot_name}/camera_back_link</gz_frame_id>
+        <gz_frame_id>${tf_prefix}camera_back_link</gz_frame_id>
         <topic>${robot_name}/base_back_camera/color</topic>
         <always_on>1</always_on>
@@ -175,5 +178,5 @@
         <sensor name="base_back_camera_color" type="camera">
           <pose>0 0 ${0.0175/2} ${M_PI/2} -${M_PI/2} 0 </pose>
-          <gz_frame_id>${robot_name}/camera_back_link</gz_frame_id>
+          <gz_frame_id>${tf_prefix}camera_back_link</gz_frame_id>
           <topic>${robot_name}/base_back_camera/color</topic>
           <always_on>1</always_on>
@@ -206,5 +209,5 @@
         <sensor name="head_camera_color" type="camera">
           <pose>0 0 ${0.0175/2} ${M_PI/2} -${M_PI/2} 0 </pose>
-          <gz_frame_id>${robot_name}/head_camera_color_optical_frame</gz_frame_id>
+          <gz_frame_id>${tf_prefix}head_camera_color_optical_frame</gz_frame_id>
           <topic>${robot_name}/head_camera/color</topic>
           <always_on>1</always_on>
@@ -237,5 +240,5 @@
         <sensor name="head_camera_depth" type="depth">
           <pose>0 0 ${0.0175/2} 0 0 0 </pose>
-          <gz_frame_id>${robot_name}/head_camera_depth_frame</gz_frame_id>
+          <gz_frame_id>${tf_prefix}head_camera_depth_frame</gz_frame_id>
           <topic>${robot_name}/head_camera/depth</topic>
           <always_on>1</always_on>
@@ -267,5 +270,5 @@
         <sensor name="hand_camera_color" type="camera">
           <pose>0 0 ${0.0175/2} ${M_PI/2} -${M_PI/2} 0 </pose>
-          <gz_frame_id>${robot_name}/hand_camera_color_optical_frame</gz_frame_id>
+          <gz_frame_id>${tf_prefix}hand_camera_color_optical_frame</gz_frame_id>
           <topic>${robot_name}/hand_camera/color</topic>
           <always_on>1</always_on>
@@ -298,5 +301,5 @@
         <sensor name="hand_camera_depth" type="depth">
           <pose>0 0 ${0.0175/2} 0 0 0 </pose>
-          <gz_frame_id>${robot_name}/hand_camera_depth_frame</gz_frame_id>
+          <gz_frame_id>${tf_prefix}hand_camera_depth_frame</gz_frame_id>
           <topic>${robot_name}/hand_camera/depth</topic>
           <always_on>1</always_on>
@@ -328,5 +331,5 @@
         <sensor name="lidar" type="gpu_lidar">
           <pose>0 0 0 0 0 0</pose>
-          <gz_frame_id>${robot_name}/laser_frame</gz_frame_id>
+          <gz_frame_id>${tf_prefix}laser_frame</gz_frame_id>
           <topic>${robot_name}/lidar/scan</topic>
           <always_on>1</always_on>

Commit message: [ADD] description: MuJoCo mode (MujocoSystemInterface in the one ros2_control block)
enable_mujoco / mujoco_model / mujoco_headless; wheel joints and hand_sub_joint
follow sim_on (gz or mujoco); docking_joint is a state-only joint under MuJoCo
so MoveIt sees every URDF joint. Real and Gazebo renders are byte-identical.

File: sobit_light_description/robots/sobit_light_robot.urdf.xacro (robot description, xacro)
@@ -28,4 +28,8 @@
   <!-- Add variables -->
   <xacro:arg name="enable_gz"                 default="False" />
+  <!-- MuJoCo (mujoco_ros2_control) supersedes enable_gz; mujoco_model = absolute scene.xml -->
+  <xacro:arg name="enable_mujoco"             default="False" />
+  <xacro:arg name="mujoco_model"              default="" />
+  <xacro:arg name="mujoco_headless"           default="false" />
   <xacro:arg name="enable_gz_front_cam_color" default="True" />
   <xacro:arg name="enable_gz_back_cam_color"  default="True" />
@@ -40,5 +44,8 @@
   <xacro:arg name="enable_tf_prefix"          default="True" />
   <!-- ${...} evaluates a Python literal, where only True/False parse. -->
-  <xacro:property name="gz_on" value="${'$(arg enable_gz)'.lower() in ('true', '1')}" />
+  <xacro:property name="mujoco_on" value="${'$(arg enable_mujoco)'.lower() in ('true', '1')}" />
+  <xacro:property name="gz_on" value="${'$(arg enable_gz)'.lower() in ('true', '1') and not mujoco_on}" />
+  <!-- Any simulator: no real hardware params, sim-only joints (wheels, hand mimic) -->
+  <xacro:property name="sim_on" value="${gz_on or mujoco_on}" />
   <!-- Activate Components -->
   <xacro:arg name="enable_mobile_base"  default="True" />

File: sobit_light_description/urdf/controllers.urdf.xacro (robot description, xacro)
@@ -8,5 +8,12 @@
           <plugin>gz_ros2_control/GazeboSimSystem</plugin>
         </xacro:if>
-        <xacro:unless value="${gz_on}">
+        <!-- Joints map to the MJCF actuators of the same name; sensors live in mujoco_plugins.yaml -->
+        <xacro:if value="${mujoco_on}">
+          <plugin>mujoco_ros2_control/MujocoSystemInterface</plugin>
+          <param name="mujoco_model">$(arg mujoco_model)</param>
+          <param name="headless">$(arg mujoco_headless)</param>
+          <param name="initial_keyframe">home</param>
+        </xacro:if>
+        <xacro:unless value="${sim_on}">
           <xacro:property name="dxl_sl_port" value="$(arg dxl_sl_port)"/>
           <plugin>dynamixel_hardware/DynamixelHardware</plugin>
@@ -43,5 +50,5 @@
     <!-- Position Drive - Head -->
     <joint name="${prefix}_yaw_joint">
-      <xacro:unless value="${gz_on}">
+      <xacro:unless value="${sim_on}">
         <param name="id">11</param>
         <param name="control_mode">0</param>
@@ -60,5 +67,5 @@
     </joint>
     <joint name="${prefix}_pitch_joint">
-      <xacro:unless value="${gz_on}">
+      <xacro:unless value="${sim_on}">
         <param name="id">12</param>
         <param name="control_mode">0</param>
@@ -80,5 +87,5 @@
     <!-- Position Drive - Arm -->
     <joint name="${prefix}_shoulder_roll_joint">
-      <xacro:unless value="${gz_on}">
+      <xacro:unless value="${sim_on}">
         <param name="id">1</param>
         <param name="control_mode">0</param>
@@ -97,5 +104,5 @@
     </joint>
     <joint name="${prefix}_shoulder_pitch_joint">
-      <xacro:unless value="${gz_on}">
+      <xacro:unless value="${sim_on}">
         <param name="id">3</param>
         <param name="control_mode">0</param>
@@ -114,5 +121,5 @@
     </joint>
     <joint name="${prefix}_elbow_pitch_joint">
-      <xacro:unless value="${gz_on}">
+      <xacro:unless value="${sim_on}">
         <param name="id">4</param>
         <param name="control_mode">0</param>
@@ -131,5 +138,5 @@
     </joint>
     <joint name="${prefix}_forearm_roll_joint">
-      <xacro:unless value="${gz_on}">
+      <xacro:unless value="${sim_on}">
         <param name="id">5</param>
         <param name="control_mode">0</param>
@@ -148,5 +155,5 @@
     </joint>
     <joint name="${prefix}_wrist_pitch_joint">
-      <xacro:unless value="${gz_on}">
+      <xacro:unless value="${sim_on}">
         <param name="id">6</param>
         <param name="control_mode">0</param>
@@ -165,5 +172,5 @@
     </joint>
     <joint name="${prefix}_wrist_roll_joint">
-      <xacro:unless value="${gz_on}">
+      <xacro:unless value="${sim_on}">
         <param name="id">7</param>
         <param name="control_mode">0</param>
@@ -185,5 +192,5 @@
     <!-- Position Drive - Hand -->
     <joint name="${prefix}_joint">
-      <xacro:unless value="${gz_on}">
+      <xacro:unless value="${sim_on}">
         <param name="id">8</param>
         <param name="control_mode">6</param>
@@ -200,5 +207,5 @@
       <!-- <state_interface name="effort"/> -->
     </joint>
-    <xacro:if value="${gz_on}">
+    <xacro:if value="${sim_on}">
       <joint name="${prefix}_sub_joint">
         <param name="mimic">${prefix}_joint</param>
@@ -212,5 +219,5 @@
   </xacro:macro>
   <xacro:macro name="wheel_controllers"  params="prefix enable_gz:=False">
-    <xacro:if value="${gz_on}">
+    <xacro:if value="${sim_on}">
         <joint name="base_l_drive_wheel_joint">
           <command_interface name="velocity">
@@ -230,4 +237,11 @@
         </joint>
     </xacro:if>
+    <!-- gz bridges every joint state; MuJoCo reports only these, and MoveIt needs the docking latch too -->
+    <xacro:if value="${mujoco_on}">
+        <joint name="docking_joint">
+          <state_interface name="position"/>
+          <state_interface name="velocity"/>
+        </joint>
+    </xacro:if>
   </xacro:macro>
 </robot>
