Commit message: [FIX] inertia for docking

File: sobit_light_description/urdf/base/base.urdf.xacro (robot description, xacro)
@@ -59,7 +59,7 @@
         <mass value="0.2" />
         <origin xyz="0 0 0" rpy="0 0 0" />
-        <inertia ixx="0.001" ixy="0" ixz="0"
-                 iyy="0.001" iyz="0"
-                 izz="0.001" />
+        <inertia ixx="${1/12*0.2*(3*0.025**2+0.015**2)}" ixy="0" ixz="0"
+                 iyy="${1/12*0.2*(3*0.025**2+0.015**2)}" iyz="0"
+                 izz="${1/2*0.2*0.025**2}" />
       </inertial>
     </link>
