Commit message: [FIX] disable collision

File: sobit_light_description/urdf/base/plate.urdf.xacro (robot description, xacro)
@@ -15,10 +15,10 @@
         <material name="black" />
       </visual>
-      <collision>
+      <!-- <collision>
         <origin xyz="0.0 0.0 -${0.1408/2}" rpy="0 0 0"/>
         <geometry>
           <box size="0.320 0.375 0.1408"/>
         </geometry>
-      </collision>
+      </collision> -->
       <inertial>
         <origin xyz="0.0 0.0 -${0.1408/2}" rpy="0 0 0"/>
