Commit message: [UPD] gz support

File: sobit_light_description/urdf/dxl_control.urdf.xacro (robot description, xacro)
@@ -2,15 +2,24 @@
 <!-- SOBIT Light (Dynamixel Control) -->
 <robot name="sobit_light_dxl_control" xmlns:xacro="http://www.ros.org/wiki/xacro">
-  <xacro:macro name="dxl_control" params="name">
-    <!-- <ros2_control name="${name}" type="system"> -->
-    <ros2_control name="joints_control" type="system">
+  <xacro:macro name="dxl_control" params="name enable_gz:=False">
+    <ros2_control name="${name}" type="system">
+    <!-- <ros2_control name="joints_control" type="system"> -->
       <hardware>
-        <plugin>dynamixel_hardware/DynamixelHardware</plugin>
-        <param name="usb_port">/dev/ttyUSB0</param>
-        <param name="baud_rate">1000000</param>
-        <!-- <param name="use_dummy">true</param> -->
+        <xacro:if value="${$(arg enable_gz)}">
+          <plugin>ign_ros2_control/IgnitionSystem</plugin>
+          <!-- <plugin>gazebo_ros2_control/GazeboHardware</plugin> -->
+        </xacro:if>
+        <xacro:unless value="${$(arg enable_gz)}">
+          <plugin>dynamixel_hardware/DynamixelHardware</plugin>
+          <param name="usb_port">/dev/ttyUSB0</param>
+          <param name="baud_rate">1000000</param>
+          <!-- <param name="use_dummy">true</param> -->
+        </xacro:unless>
       </hardware>
+      <!-- Position Drive: Arm -->
       <joint name="arm_shoulder_roll_joint">
-        <param name="id">1</param>
+        <xacro:unless value="${$(arg enable_gz)}">
+          <param name="id">1</param>
+        </xacro:unless>
         <command_interface name="position">
           <param name="min">-3.141592654</param>
@@ -25,7 +34,9 @@
       </joint>
       <joint name="arm_shoulder_pitch_sub_joint">
-        <param name="id">2</param>
-        <param name="mimic">arm_shoulder_pitch_joint</param>
-        <param name="multiplier">-1</param>
+        <xacro:unless value="${$(arg enable_gz)}">
+          <param name="id">2</param>
+        </xacro:unless>
+        <!-- <param name="mimic">arm_shoulder_pitch_joint</param> -->
+        <!-- <param name="multiplier">-1</param> -->
         <command_interface name="position"/>
         <command_interface name="velocity"/>
@@ -35,5 +46,7 @@
       </joint>
       <joint name="arm_shoulder_pitch_joint">
-        <param name="id">3</param>
+        <xacro:unless value="${$(arg enable_gz)}">
+          <param name="id">3</param>
+        </xacro:unless>
         <command_interface name="position">
           <param name="min">-1.570796327</param>
@@ -48,5 +61,7 @@
       </joint>
       <joint name="arm_elbow_pitch_joint">
-        <param name="id">4</param>
+        <xacro:unless value="${$(arg enable_gz)}">
+          <param name="id">4</param>
+        </xacro:unless>
         <command_interface name="position">
           <param name="min">-1.570796327</param>
@@ -61,5 +76,7 @@
       </joint>
       <joint name="arm_forearm_roll_joint">
-        <param name="id">5</param>
+        <xacro:unless value="${$(arg enable_gz)}">
+          <param name="id">5</param>
+        </xacro:unless>
         <command_interface name="position">
           <param name="min">-3.141592654</param>
@@ -74,5 +91,7 @@
       </joint>
       <joint name="arm_wrist_pitch_joint">
-        <param name="id">6</param>
+        <xacro:unless value="${$(arg enable_gz)}">
+          <param name="id">6</param>
+        </xacro:unless>
         <command_interface name="position">
           <param name="min">-1.570796327</param>
@@ -87,19 +106,23 @@
       </joint>
       <joint name="arm_wrist_roll_joint">
-        <param name="id">7</param>
-        <command_interface name="position">
-          <param name="min">-3.141592654</param>
-          <param name="max">3.141592654</param>
-        </command_interface>
-        <command_interface name="velocity"/>
-        <state_interface name="position">
-          <param name="initial_value">0.0</param>
-        </state_interface>
-        <state_interface name="velocity"/>
-        <state_interface name="effort"/>
-      </joint>
+        <xacro:unless value="${$(arg enable_gz)}">
+          <param name="id">7</param>
+        </xacro:unless>
+        <command_interface name="position">
+          <param name="min">-3.141592654</param>
+          <param name="max">3.141592654</param>
+        </command_interface>
+        <command_interface name="velocity"/>
+        <state_interface name="position">
+          <param name="initial_value">0.0</param>
+        </state_interface>
+        <state_interface name="velocity"/>
+        <state_interface name="effort"/>
+      </joint>
+      <!-- Position Drive: Hand -->
       <joint name="hand_joint">
-      <!-- <joint name="hand_finger_l_joint"> -->
-        <param name="id">8</param>
+        <xacro:unless value="${$(arg enable_gz)}">
+          <param name="id">8</param>
+        </xacro:unless>
         <command_interface name="position"/>
         <command_interface name="velocity"/>
@@ -110,6 +133,20 @@
         <state_interface name="effort"/>
       </joint>
+      <xacro:if value="${$(arg enable_gz)}">
+        <joint name="hand_sub_joint">
+          <param name="mimic">hand_joint</param>
+          <param name="multiplier">-1</param>
+          <command_interface name="position"/>
+          <command_interface name="velocity"/>
+          <state_interface name="position"/>
+          <state_interface name="velocity"/>
+          <state_interface name="effort"/>
+        </joint>
+      </xacro:if>
+      <!-- Position Drive: Head -->
       <joint name="head_yaw_joint">
-        <param name="id">11</param>
+        <xacro:unless value="${$(arg enable_gz)}">
+          <param name="id">11</param>
+        </xacro:unless>
         <command_interface name="position">
           <param name="min">-3.141592654</param>
@@ -124,5 +161,7 @@
       </joint>
       <joint name="head_pitch_joint">
-        <param name="id">12</param>
+        <xacro:unless value="${$(arg enable_gz)}">
+          <param name="id">12</param>
+        </xacro:unless>
         <command_interface name="position">
           <param name="min">-1.570796327</param>
@@ -137,4 +176,45 @@
       </joint>
     </ros2_control>
+    <!-- Differential Drive -->
+    <xacro:if value="${$(arg enable_gz)}">
+      <ros2_control name="base_control" type="system">
+        <hardware>
+          <plugin>ign_ros2_control/IgnitionSystem</plugin>
+          <!-- <plugin>gazebo_ros2_control/GazeboHardware</plugin> -->
+        </hardware>
+        <joint name="base_l_drive_wheel_joint">
+          <command_interface name="velocity">
+            <param name="min">-1.0</param>
+            <param name="max">1.0</param>
+          </command_interface>
+          <state_interface name="position"/>
+          <state_interface name="velocity"/>
+        </joint>
+        <joint name="base_r_drive_wheel_joint">
+          <command_interface name="velocity">
+            <param name="min">-1.0</param>
+            <param name="max">1.0</param>
+          </command_interface>
+          <state_interface name="position"/>
+          <state_interface name="velocity"/>
+        </joint>
+      </ros2_control>
+      <gazebo reference="plate_bottom_link">
+        <mu1>0.0</mu1>
+        <mu2>0.0</mu2>
+      </gazebo>
+    </xacro:if>
+    <!-- Ignition ROS2 Control -->
+    <xacro:if value="${$(arg enable_gz)}">
+      <gazebo>
+        <plugin
+            filename="ign_ros2_control-system"
+            name="ign_ros2_control::IgnitionROS2ControlPlugin">
+            <!-- filename="gz_ros2_control-system"
+            name="gz_ros2_control::GazeboSimROS2ControlPlugin"> -->
+          <parameters>$(find sobit_light_control)/config/controllers_gz.yaml</parameters>
+        </plugin>
+      </gazebo>
+    </xacro:if>
   </xacro:macro>
 </robot>
