Commit message: [ADD] robot name var

File: sobit_light_description/urdf/controllers.urdf.xacro (robot description, xacro)
@@ -2,5 +2,5 @@
 <!-- SOBIT Light (Dynamixel Control) -->
 <robot name="sobit_light_controllers" xmlns:xacro="http://www.ros.org/wiki/xacro">
-  <xacro:macro name="controllers" params="name enable_gz:=False">
+  <xacro:macro name="controllers" params="name enable_gz:=False robot_name:=sobit_light">
     <ros2_control name="${name}_arm" type="system">
     <!-- <ros2_control name="joints_control" type="system"> -->
@@ -210,4 +210,7 @@
         <!-- <plugin filename="gz_ros2_control-system" name="gz_ros2_control::GazeboSimROS2ControlPlugin"> -->
         <plugin filename="ign_ros2_control-system" name="ign_ros2_control::IgnitionROS2ControlPlugin">
+          <ros>
+            <namespace>${robot_name}</namespace>
+          </ros>
           <parameters>$(find sobit_light_control)/config/controllers_gz.yaml</parameters>
         </plugin>

File: sobit_light_description/urdf/gazebo.urdf.xacro (robot description, xacro)
@@ -2,11 +2,11 @@
 <!-- SOBIT Light (Gazebo) -->
 <robot name="sobit_light_gazebo" xmlns:xacro="http://ros.org/wiki/xacro">
-  <xacro:macro name="gazebo_ros2_control" params="prefix">
+  <xacro:macro name="gazebo_sensors" params="prefix robot_name">
     <!-- Sensor: Base Front Camera (Color) -->
     <gazebo reference="imu_link">
       <sensor name="imu_sensor" type="imu">
         <pose>0 0 0 0 0 0</pose>
-        <gz_frame_id>camera_front_link</gz_frame_id>
-        <topic>imu</topic>
+        <gz_frame_id>${robot_name}/camera_front_link</gz_frame_id>
+        <topic>${robot_name}/imu</topic>
         <always_on>1</always_on>
         <visualize>true</visualize>
@@ -18,6 +18,6 @@
       <sensor name="base_front_camera_color" type="wideanglecamera">
         <pose>0 0 ${0.0175/2} ${M_PI/2} -${M_PI/2} 0 </pose>
-        <gz_frame_id>camera_front_link</gz_frame_id>
-        <topic>/base_front_camera/color</topic>
+        <gz_frame_id>${robot_name}/camera_front_link</gz_frame_id>
+        <topic>${robot_name}/base_front_camera/color</topic>
         <always_on>1</always_on>
         <visualize>true</visualize>
@@ -52,7 +52,7 @@
       <sensor name="base_front_camera_color" type="camera">
         <pose>0 0 ${0.0175/2} ${M_PI/2} -${M_PI/2} 0 </pose>
-        <ignition_frame_id>base_front_camera_color</ignition_frame_id>
-        <!-- <gz_frame_id>base_front_camera_color</gz_frame_id> -->
-        <topic>/base_front_camera/color</topic>
+        <ignition_frame_id>${robot_name}/base_front_camera_color</ignition_frame_id>
+        <!-- <gz_frame_id>${robot_name}/base_front_camera_color</gz_frame_id> -->
+        <topic>${robot_name}/base_front_camera/color</topic>
         <always_on>1</always_on>
         <visualize>true</visualize>
@@ -82,6 +82,6 @@
       <sensor name="base_back_camera_color" type="wideanglecamera">
         <pose>0 0 ${0.0175/2} ${M_PI/2} -${M_PI/2} 0 </pose>
-        <gz_frame_id>camera_back_link</gz_frame_id>
-        <topic>/base_back_camera/color</topic>
+        <gz_frame_id>${robot_name}/camera_back_link</gz_frame_id>
+        <topic>${robot_name}/base_back_camera/color</topic>
         <always_on>1</always_on>
         <visualize>true</visualize>
@@ -116,7 +116,7 @@
       <sensor name="base_back_camera_color" type="camera">
         <pose>0 0 ${0.0175/2} ${M_PI/2} -${M_PI/2} 0 </pose>
-        <ignition_frame_id>camera_back_link</ignition_frame_id>
-        <!-- <gz_frame_id>camera_back_link</gz_frame_id> -->
-        <topic>/base_back_camera/color</topic>
+        <ignition_frame_id>${robot_name}/camera_back_link</ignition_frame_id>
+        <!-- <gz_frame_id>${robot_name}/camera_back_link</gz_frame_id> -->
+        <topic>${robot_name}/base_back_camera/color</topic>
         <always_on>1</always_on>
         <visualize>true</visualize>
@@ -146,7 +146,7 @@
       <sensor name="head_camera_color" type="camera">
         <pose>0 0 ${0.0175/2} ${M_PI/2} -${M_PI/2} 0 </pose>
-        <ignition_frame_id>head_camera_color_optical_frame</ignition_frame_id>
-        <!-- <gz_frame_id>head_camera_color_optical_frame</gz_frame_id> -->
-        <topic>/head_camera/color</topic>
+        <ignition_frame_id>${robot_name}/head_camera_color_optical_frame</ignition_frame_id>
+        <!-- <gz_frame_id>${robot_name}/head_camera_color_optical_frame</gz_frame_id> -->
+        <topic>${robot_name}/head_camera/color</topic>
         <always_on>1</always_on>
         <visualize>true</visualize>
@@ -176,7 +176,7 @@
       <sensor name="head_camera_depth" type="depth">
         <pose>0 0 ${0.0175/2} ${M_PI/2} -${M_PI/2} 0 </pose>
-        <ignition_frame_id>head_camera_depth_optical_frame</ignition_frame_id>
-        <!-- <gz_frame_id>head_camera_depth_optical_frame</gz_frame_id> -->
-        <topic>/head_camera/depth</topic>
+        <ignition_frame_id>${robot_name}/head_camera_depth_optical_frame</ignition_frame_id>
+        <!-- <gz_frame_id>${robot_name}/head_camera_depth_optical_frame</gz_frame_id> -->
+        <topic>${robot_name}/head_camera/depth</topic>
         <always_on>1</always_on>
         <visualize>true</visualize>
@@ -205,7 +205,7 @@
       <sensor name="hand_camera_color" type="camera">
         <pose>0 0 ${0.0175/2} ${M_PI/2} -${M_PI/2} 0 </pose>
-        <ignition_frame_id>hand_camera_color_optical_frame</ignition_frame_id>
-        <!-- <gz_frame_id>hand_camera_color_optical_frame</gz_frame_id> -->
-        <topic>/hand_camera/color</topic>
+        <ignition_frame_id>${robot_name}/hand_camera_color_optical_frame</ignition_frame_id>
+        <!-- <gz_frame_id>${robot_name}/hand_camera_color_optical_frame</gz_frame_id> -->
+        <topic>${robot_name}/hand_camera/color</topic>
         <always_on>1</always_on>
         <visualize>true</visualize>
@@ -235,7 +235,7 @@
       <sensor name="hand_camera_depth" type="depth">
         <pose>0 0 ${0.0175/2} ${M_PI/2} -${M_PI/2} 0 </pose>
-        <ignition_frame_id>hand_camera_depth_optical_frame</ignition_frame_id>
-        <!-- <gz_frame_id>hand_camera_depth_optical_frame</gz_frame_id> -->
-        <topic>/hand_camera/depth</topic>
+        <ignition_frame_id>${robot_name}/hand_camera_depth_optical_frame</ignition_frame_id>
+        <!-- <gz_frame_id>${robot_name}/hand_camera_depth_optical_frame</gz_frame_id> -->
+        <topic>${robot_name}/hand_camera/depth</topic>
         <always_on>1</always_on>
         <visualize>true</visualize>
@@ -264,7 +264,7 @@
       <sensor name="lidar" type="gpu_lidar">
         <pose>0 0 0 0 0 0</pose>
-        <ignition_frame_id>sim_laser_frame</ignition_frame_id>
-        <!-- <gz_frame_id>sim_laser_frame</gz_frame_id> -->
-        <topic>kachaka/lidar/scan</topic>
+        <ignition_frame_id>${robot_name}/sim_laser_frame</ignition_frame_id>
+        <!-- <gz_frame_id>${robot_name}/sim_laser_frame</gz_frame_id> -->
+        <topic>${robot_name}/lidar/scan</topic>
         <always_on>1</always_on>
         <visualize>true</visualize>
@@ -316,5 +316,5 @@
       <!-- <plugin filename="ignition-gazebo-joint-state-publisher-system" name="ignition::gazebo::systems::JointStatePublisher"> -->
       <plugin filename="gz-sim-joint-state-publisher-system" name="gz::sim::systems::JointStatePublisher">
-        <topic>joint_states</topic>
+        <topic>${robot_name}/joint_states</topic>
       </plugin>
     </gazebo>
