Commit message: [FEAT] retrieve dxl port, toogle controllers

File: sobit_light_description/urdf/controllers.urdf.xacro (robot description, xacro)
@@ -1,216 +1,227 @@
 <?xml version="1.0" encoding="UTF-8" ?>
-<!-- SOBIT Light (Dynamixel Control) -->
+<!-- SOBIT LIGHT (Dynamixel Control) -->
 <robot name="sobit_light_controllers" xmlns:xacro="http://www.ros.org/wiki/xacro">
   <xacro:macro name="controllers" params="name enable_gz:=False robot_name:=sobit_light">
-    <ros2_control name="${name}" type="system">
-    <!-- <ros2_control name="joints_control" type="system"> -->
+    <ros2_control name="dynamixel_controllers" type="system">
       <hardware>
         <xacro:if value="${$(arg enable_gz)}">
-          <plugin>ign_ros2_control/IgnitionSystem</plugin>
-          <!-- <plugin>gz_ros2_control/GazeboSimSystem</plugin> -->
+          <plugin>gz_ros2_control/GazeboSimSystem</plugin>
         </xacro:if>
         <xacro:unless value="${$(arg enable_gz)}">
+          <xacro:property name="dxl_sl_port" value="$(arg dxl_sl_port)"/>
           <plugin>dynamixel_hardware/DynamixelHardware</plugin>
-          <!-- <param name="usb_port">/dev/ttyUSB-DXL_light</param> -->
-          <param name="port_name">/dev/ttyUSB0</param>
-          <param name="baud_rate">1000000</param>
-          <!-- <param name="use_dummy">true</param> -->
+            <param name="port_name">${dxl_sl_port}</param>
+            <param name="baud_rate">1000000</param>
         </xacro:unless>
       </hardware>
-      <!-- Position Drive - Arm -->
-      <joint name="arm_shoulder_roll_joint">
-        <xacro:unless value="${$(arg enable_gz)}">
-          <param name="id">1</param>
-          <param name="control_mode">0</param>
-          <param name="interface">rs</param>
-        </xacro:unless>
-        <command_interface name="position">
-          <param name="min">-3.141592654</param>
-          <param name="max">3.141592654</param>
-        </command_interface>
-        <!-- <command_interface name="velocity"/> -->
-        <state_interface name="position">
-          <param name="initial_value">0.0</param>
-        </state_interface>
+      <xacro:if value="${$(arg enable_head)}">
+        <xacro:dxl_head_controllers prefix="head"       enable_gz="${$(arg enable_gz)}"/>
+      </xacro:if>
+      <xacro:if value="${$(arg enable_arm)}">
+        <xacro:dxl_arm_controllers  prefix="arm"  enable_gz="${$(arg enable_gz)}"/>
+      </xacro:if>
+      <xacro:if value="${$(arg enable_hand)}">
+        <xacro:dxl_hand_controllers prefix="hand"  enable_gz="${$(arg enable_gz)}"/>
+      </xacro:if>
+      <xacro:if value="${$(arg enable_mobile_base)}">
+        <xacro:wheel_controllers    prefix="wheel"      enable_gz="${$(arg enable_gz)}"/>
+      </xacro:if>
+    </ros2_control>
+    <!-- Gazebo ROS2 Control -->
+    <xacro:if value="${$(arg enable_gz)}">
+      <gazebo>
+        <plugin filename="gz_ros2_control-system" name="gz_ros2_control::GazeboSimROS2ControlPlugin">
+          <ros>
+            <namespace>$(arg robot_name)</namespace>
+          </ros>
+          <parameters>$(find sobit_light_control)/config/gz_controllers.yaml</parameters>
+        </plugin>
+      </gazebo>
+    </xacro:if>
+  </xacro:macro>
+  <xacro:macro name="dxl_head_controllers"  params="prefix enable_gz:=False">
+    <!-- Position Drive - Head -->
+    <joint name="${prefix}_yaw_joint">
+      <xacro:unless value="${$(arg enable_gz)}">
+        <param name="id">11</param>
+        <param name="control_mode">0</param>
+        <param name="interface">rs</param>
+      </xacro:unless>
+      <command_interface name="position">
+        <param name="min">-${M_PI}</param>
+        <param name="max">${M_PI}</param>
+      </command_interface>
+      <state_interface name="position">
+        <param name="initial_value">0.0</param>
+      </state_interface>
+      <state_interface name="velocity"/>
+      <!-- <state_interface name="effort"/> -->
+    </joint>
+    <joint name="${prefix}_pitch_joint">
+      <xacro:unless value="${$(arg enable_gz)}">
+        <param name="id">12</param>
+        <param name="control_mode">0</param>
+        <param name="interface">rs</param>
+      </xacro:unless>
+      <command_interface name="position">
+        <param name="min">-${M_PI/2}</param>
+        <param name="max">${M_PI/2}</param>
+      </command_interface>
+      <state_interface name="position">
+        <param name="initial_value">0.0</param>
+      </state_interface>
+      <state_interface name="velocity"/>
+      <!-- <state_interface name="effort"/> -->
+    </joint>
+  </xacro:macro>
+  <xacro:macro name="dxl_arm_controllers"  params="prefix enable_gz:=False">
+    <!-- Position Drive - Arm -->
+    <joint name="${prefix}_shoulder_roll_joint">
+      <xacro:unless value="${$(arg enable_gz)}">
+        <param name="id">1</param>
+        <param name="control_mode">0</param>
+        <param name="interface">rs</param>
+      </xacro:unless>
+      <command_interface name="position">
+        <param name="min">-${M_PI}</param>
+        <param name="max">${M_PI}</param>
+      </command_interface>
+      <state_interface name="position">
+        <param name="initial_value">0.0</param>
+      </state_interface>
+      <state_interface name="velocity"/>
+      <!-- <state_interface name="effort"/> -->
+    </joint>
+    <joint name="${prefix}_shoulder_pitch_sub_joint">
+      <xacro:unless value="${$(arg enable_gz)}">
+        <param name="id">2</param>
+        <param name="control_mode">0</param>
+        <param name="interface">rs</param>
+      </xacro:unless>
+      <!-- <param name="mimic">arm_shoulder_pitch_joint</param>
+      <param name="multiplier">-1</param> -->
+      <!-- <command_interface name="position"/> -->
+      <command_interface name="position">
+        <param name="min">-${M_PI/2}</param>
+        <param name="max">${M_PI/2}</param>
+      </command_interface>
+      <state_interface name="position">
+        <param name="initial_value">${M_PI/2}</param>
+      </state_interface>
+      <!-- <state_interface name="position"/> -->
+      <state_interface name="velocity"/>
+      <!-- <state_interface name="effort"/> -->
+    </joint>
+    <joint name="${prefix}_shoulder_pitch_joint">
+      <xacro:unless value="${$(arg enable_gz)}">
+        <param name="id">3</param>
+        <param name="control_mode">0</param>
+        <param name="interface">rs</param>
+      </xacro:unless>
+      <command_interface name="position">
+        <param name="min">-${M_PI/2}</param>
+        <param name="max">${M_PI/2}</param>
+      </command_interface>
+      <state_interface name="position">
+        <param name="initial_value">-${M_PI/2}</param>
+      </state_interface>
+      <state_interface name="velocity"/>
+      <!-- <state_interface name="effort"/> -->
+    </joint>
+    <joint name="${prefix}_elbow_pitch_joint">
+      <xacro:unless value="${$(arg enable_gz)}">
+        <param name="id">4</param>
+        <param name="control_mode">0</param>
+        <param name="interface">rs</param>
+      </xacro:unless>
+      <command_interface name="position">
+        <param name="min">-${M_PI/2}</param>
+        <param name="max">${M_PI/2}</param>
+      </command_interface>
+      <state_interface name="position">
+        <param name="initial_value">0.0</param>
+      </state_interface>
+      <state_interface name="velocity"/>
+      <!-- <state_interface name="effort"/> -->
+    </joint>
+    <joint name="${prefix}_forearm_roll_joint">
+      <xacro:unless value="${$(arg enable_gz)}">
+        <param name="id">5</param>
+        <param name="control_mode">0</param>
+        <param name="interface">rs</param>
+      </xacro:unless>
+      <command_interface name="position">
+        <param name="min">-${M_PI}</param>
+        <param name="max">${M_PI}</param>
+      </command_interface>
+      <state_interface name="position">
+        <param name="initial_value">0.0</param>
+      </state_interface>
+      <state_interface name="velocity"/>
+      <!-- <state_interface name="effort"/> -->
+    </joint>
+    <joint name="${prefix}_wrist_pitch_joint">
+      <xacro:unless value="${$(arg enable_gz)}">
+        <param name="id">6</param>
+        <param name="control_mode">0</param>
+        <param name="interface">rs</param>
+      </xacro:unless>
+      <command_interface name="position">
+        <param name="min">-${M_PI/2}</param>
+        <param name="max">${M_PI/2}</param>
+      </command_interface>
+      <state_interface name="position">
+        <param name="initial_value">0.0</param>
+      </state_interface>
+      <state_interface name="velocity"/>
+      <!-- <state_interface name="effort"/> -->
+    </joint>
+    <joint name="${prefix}_wrist_roll_joint">
+      <xacro:unless value="${$(arg enable_gz)}">
+        <param name="id">7</param>
+        <param name="control_mode">0</param>
+        <param name="interface">rs</param>
+      </xacro:unless>
+      <command_interface name="position">
+        <param name="min">-${M_PI}</param>
+        <param name="max">${M_PI}</param>
+      </command_interface>
+      <state_interface name="position">
+        <param name="initial_value">0.0</param>
+      </state_interface>
+      <state_interface name="velocity"/>
+      <!-- <state_interface name="effort"/> -->
+    </joint>
+  </xacro:macro>
+  <xacro:macro name="dxl_hand_controllers"  params="prefix enable_gz:=False">
+    <!-- Position Drive - Hand -->
+    <joint name="${prefix}_joint">
+      <xacro:unless value="${$(arg enable_gz)}">
+        <param name="id">8</param>
+        <param name="control_mode">6</param>
+        <param name="Goal_Current">50</param>
+        <param name="interface">rs</param>
+        <param name="gear_ratio">-59.504383354</param>
+      </xacro:unless>
+      <command_interface name="position"/>
+      <state_interface name="position">
+        <param name="initial_value">0.0</param>
+      </state_interface>
+      <state_interface name="velocity"/>
+      <!-- <state_interface name="effort"/> -->
+    </joint>
+    <xacro:if value="${$(arg enable_gz)}">
+      <joint name="${prefix}_sub_joint">
+        <param name="mimic">${prefix}_joint</param>
+        <param name="multiplier">1</param>
+        <command_interface name="position"/>
+        <state_interface name="position"/>
         <state_interface name="velocity"/>
-        <state_interface name="effort"/>
+        <!-- <state_interface name="effort"/> -->
       </joint>
-      <joint name="arm_shoulder_pitch_sub_joint">
-        <xacro:unless value="${$(arg enable_gz)}">
-          <param name="id">2</param>
-          <param name="control_mode">0</param>
-          <param name="interface">rs</param>
-        </xacro:unless>
-        <!-- <param name="mimic">arm_shoulder_pitch_joint</param>
-        <param name="multiplier">-1</param> -->
-        <!-- <command_interface name="position"/> -->
-        <command_interface name="position">
-          <param name="min">-1.570796327</param>
-          <param name="max">1.570796327</param>
-        </command_interface>
-        <!-- <command_interface name="velocity"/> -->
-        <state_interface name="position">
-          <param name="initial_value">1.57</param>
-        </state_interface>
-        <!-- <state_interface name="position"/> -->
-        <state_interface name="velocity"/>
-        <state_interface name="effort"/>
-      </joint>
-      <joint name="arm_shoulder_pitch_joint">
-        <xacro:unless value="${$(arg enable_gz)}">
-          <param name="id">3</param>
-          <param name="control_mode">0</param>
-          <param name="interface">rs</param>
-        </xacro:unless>
-        <command_interface name="position">
-          <param name="min">-1.570796327</param>
-          <param name="max">1.570796327</param>
-        </command_interface>
-        <!-- <command_interface name="velocity"/> -->
-        <state_interface name="position">
-          <param name="initial_value">-1.57</param>
-        </state_interface>
-        <state_interface name="velocity"/>
-        <state_interface name="effort"/>
-      </joint>
-      <joint name="arm_elbow_pitch_joint">
-        <xacro:unless value="${$(arg enable_gz)}">
-          <param name="id">4</param>
-          <param name="control_mode">0</param>
-          <param name="interface">rs</param>
-        </xacro:unless>
-        <command_interface name="position">
-          <param name="min">-1.570796327</param>
-          <param name="max">1.570796327</param>
-        </command_interface>
-        <!-- <command_interface name="velocity"/> -->
-        <state_interface name="position">
-          <param name="initial_value">0.0</param>
-        </state_interface>
-        <state_interface name="velocity"/>
-        <state_interface name="effort"/>
-      </joint>
-      <joint name="arm_forearm_roll_joint">
-        <xacro:unless value="${$(arg enable_gz)}">
-          <param name="id">5</param>
-          <param name="control_mode">0</param>
-          <param name="interface">rs</param>
-        </xacro:unless>
-        <command_interface name="position">
-          <param name="min">-3.141592654</param>
-          <param name="max">3.141592654</param>
-        </command_interface>
-        <!-- <command_interface name="velocity"/> -->
-        <state_interface name="position">
-          <param name="initial_value">0.0</param>
-        </state_interface>
-        <state_interface name="velocity"/>
-        <state_interface name="effort"/>
-      </joint>
-      <joint name="arm_wrist_pitch_joint">
-        <xacro:unless value="${$(arg enable_gz)}">
-          <param name="id">6</param>
-          <param name="control_mode">0</param>
-          <param name="interface">rs</param>
-        </xacro:unless>
-        <command_interface name="position">
-          <param name="min">-1.570796327</param>
-          <param name="max">1.570796327</param>
-        </command_interface>
-        <!-- <command_interface name="velocity"/> -->
-        <state_interface name="position">
-          <param name="initial_value">0.0</param>
-        </state_interface>
-        <state_interface name="velocity"/>
-        <state_interface name="effort"/>
-      </joint>
-      <joint name="arm_wrist_roll_joint">
-        <xacro:unless value="${$(arg enable_gz)}">
-          <param name="id">7</param>
-          <param name="control_mode">0</param>
-          <param name="interface">rs</param>
-        </xacro:unless>
-        <command_interface name="position">
-          <param name="min">-3.141592654</param>
-          <param name="max">3.141592654</param>
-        </command_interface>
-        <!-- <command_interface name="velocity"/> -->
-        <state_interface name="position">
-          <param name="initial_value">0.0</param>
-        </state_interface>
-        <state_interface name="velocity"/>
-        <state_interface name="effort"/>
-      </joint>
-      <!-- Position Drive - Hand -->
-      <joint name="hand_joint">
-        <xacro:unless value="${$(arg enable_gz)}">
-          <param name="id">8</param>
-          <param name="control_mode">6</param>
-          <param name="Goal_Current">50</param>
-          <param name="interface">rs</param>
-          <param name="gear_ratio">-59.504383354</param>
-        </xacro:unless>
-        <command_interface name="position"/>
-        <!-- <command_interface name="velocity"/> -->
-        <state_interface name="position">
-          <param name="initial_value">0.0</param>
-        </state_interface>
-        <state_interface name="velocity"/>
-        <state_interface name="effort"/>
-      </joint>
-      <xacro:if value="${$(arg enable_gz)}">
-        <joint name="hand_sub_joint">
-          <param name="mimic">hand_joint</param>
-          <param name="multiplier">1</param>
-          <command_interface name="position"/>
-          <!-- <command_interface name="velocity"/> -->
-          <state_interface name="position"/>
-          <state_interface name="velocity"/>
-          <state_interface name="effort"/>
-        </joint>
-      </xacro:if>
-      <!-- Position Drive - Head -->
-      <joint name="head_yaw_joint">
-        <xacro:unless value="${$(arg enable_gz)}">
-          <param name="id">11</param>
-          <param name="control_mode">0</param>
-          <param name="interface">rs</param>
-        </xacro:unless>
-        <command_interface name="position">
-          <param name="min">-3.141592654</param>
-          <param name="max">3.141592654</param>
-        </command_interface>
-        <!-- <command_interface name="velocity"/> -->
-        <state_interface name="position">
-          <param name="initial_value">0.0</param>
-        </state_interface>
-        <state_interface name="velocity"/>
-        <state_interface name="effort"/>
-      </joint>
-      <joint name="head_pitch_joint">
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