Commit message: [UPD] comment out shoulder_pitch_sub_joint in arm controllers due to mimic joint

File: sobit_light_description/urdf/controllers.urdf.xacro (robot description, xacro)
@@ -96,5 +96,5 @@
       <!-- <state_interface name="effort"/> -->
     </joint>
-    <joint name="${prefix}_shoulder_pitch_sub_joint">
+    <!-- <joint name="${prefix}_shoulder_pitch_sub_joint">
       <xacro:unless value="${$(arg enable_gz)}">
         <param name="id">2</param>
@@ -107,11 +107,11 @@
       </state_interface>
       <state_interface name="velocity"/>
-      <!-- <state_interface name="effort"/> -->
-      <!-- <xacro:unless value="${$(arg enable_gz)}">
+      <state_interface name="effort"/>
+      <xacro:unless value="${$(arg enable_gz)}">
         <command_interface name="position"/>
-      </xacro:unless> -->
+      </xacro:unless>
       <param name="mimic">${prefix}_shoulder_pitch_joint</param>
       <param name="multiplier">-1</param>
-    </joint>
+    </joint> -->
     <joint name="${prefix}_shoulder_pitch_joint">
       <xacro:unless value="${$(arg enable_gz)}">
