Commit message: [UPD] axis for direction

File: sobit_light_description/urdf/hand/hand.urdf.xacro (robot description, xacro)
@@ -68,5 +68,5 @@
       <child link="${prefix_hand}_link"/>
       <origin xyz="0.0 0.04 0.0" rpy="0 0 0"/>
-      <axis xyz="0 1 0"/>
+      <axis xyz="0 -1 0"/>
       <limit velocity="4.8" effort="1" lower="${-0.055+0.02675}" upper="0.0" />
     </joint>
@@ -102,8 +102,8 @@
       <child link="${prefix_hand}_sub_link"/>
       <origin xyz="0.0 -0.04 0.0" rpy="0 0 0"/>
-      <axis xyz="0 -1 0"/>
+      <axis xyz="0 1 0"/>
       <limit velocity="4.8" effort="1" lower="${-0.055+0.02675}" upper="0.0" />
       <!-- <mimic joint="${prefix_hand}_${prefix_finger}_l_joint" multiplier="1"/> -->
-      <mimic joint="${prefix_hand}_joint" multiplier="1"/>
+      <mimic joint="${prefix_hand}_joint" multiplier="-1"/>
     </joint>
     <!--  Act 8: Hand Finger (right) -->

File: sobit_light_description/urdf/head/head.urdf.xacro (robot description, xacro)
@@ -66,5 +66,5 @@
       <child link="${prefix}_pitch_link" />
       <origin xyz="0.0 0.0 0.0405" rpy="0.0 0.0 0.0" />
-      <axis xyz="0 -1 0" />
+      <axis xyz="0 1 0" />
       <limit effort="30" lower="${-M_PI/2.0}" upper="${M_PI/2.0}" velocity="${M_PI/2.0}" />
     </joint>

Commit message: [FIX] hand mimic limit

File: sobit_light_description/urdf/hand/hand.urdf.xacro (robot description, xacro)
@@ -62,15 +62,12 @@
     </link>
     <!--  Act 8: Hand Finger (left) -->
-    <!-- <joint name="${prefix_hand}_${prefix_finger}_l_joint" type="prismatic"> -->
     <joint name="${prefix_hand}_joint" type="prismatic">
       <parent link="${prefix_hand}_sub_l_link"/>
-      <!-- <child link="${prefix_hand}_${prefix_finger}_l_link"/> -->
       <child link="${prefix_hand}_link"/>
       <origin xyz="0.0 0.04 0.0" rpy="0 0 0"/>
-      <axis xyz="0 -1 0"/>
-      <limit velocity="4.8" effort="1" lower="${-0.055+0.02675}" upper="0.0" />
+      <axis xyz="0 1 0"/>
+      <limit velocity="4.8" effort="1" lower="0.0" upper="${0.02675-0.055}" />
     </joint>
     <!--  Act 8: Hand Finger (left) -->
-    <!-- <link name="${prefix_hand}_${prefix_finger}_l_link"> -->
     <link name="${prefix_hand}_link">
       <visual>
@@ -96,17 +93,13 @@
     </link>
     <!--  Act 8: Hand Finger (right) -->
-    <!-- <joint name="${prefix_hand}_${prefix_finger}_r_joint" type="prismatic"> -->
     <joint name="${prefix_hand}_sub_joint" type="prismatic">
       <parent link="${prefix_hand}_sub_r_link"/>
-      <!-- <child link="${prefix_hand}_${prefix_finger}_r_link"/> -->
       <child link="${prefix_hand}_sub_link"/>
       <origin xyz="0.0 -0.04 0.0" rpy="0 0 0"/>
       <axis xyz="0 1 0"/>
-      <limit velocity="4.8" effort="1" lower="${-0.055+0.02675}" upper="0.0" />
-      <!-- <mimic joint="${prefix_hand}_${prefix_finger}_l_joint" multiplier="1"/> -->
+      <limit velocity="4.8" effort="1" lower="-1.57" upper="1.57"/>
       <mimic joint="${prefix_hand}_joint" multiplier="-1"/>
     </joint>
     <!--  Act 8: Hand Finger (right) -->
-    <!-- <link name="${prefix_hand}_${prefix_finger}_r_link"> -->
     <link name="${prefix_hand}_sub_link">
       <visual>
@@ -133,5 +126,4 @@
     <!--  Joint: Hand Tip Left -->
     <joint name="${prefix_hand}_${prefix_finger}_tip_l_joint" type="fixed">
-      <!-- <parent link="${prefix_hand}_${prefix_finger}_l_link"/> -->
       <parent link="${prefix_hand}_link"/>
       <child link="${prefix_hand}_${prefix_finger}_tip_l_link"/>
@@ -163,5 +155,4 @@
     <!--  Joint: Hand Tip Right -->
     <joint name="${prefix_hand}_${prefix_finger}_tip_r_joint" type="fixed">
-      <!-- <parent link="${prefix_hand}_${prefix_finger}_r_link"/> -->
       <parent link="${prefix_hand}_sub_link"/>
       <child link="${prefix_hand}_${prefix_finger}_tip_r_link"/>

Commit message: [FIX] gripper mesh and pos

File: sobit_light_description/urdf/hand/hand.urdf.xacro (robot description, xacro)
@@ -63,16 +63,20 @@
     <!--  Act 8 - Hand Finger (left) -->
     <joint name="${prefix_hand}_joint" type="prismatic">
-      <parent link="${prefix_hand}_sub_l_link"/>
+      <!-- <parent link="${prefix_hand}_sub_l_link"/> -->
+      <parent link="${parent}"/>
       <child link="${prefix_hand}_link"/>
-      <origin xyz="0.0 0.04 0.0" rpy="0 0 0"/>
+      <!-- <origin xyz="0.0 0.04 0.0" rpy="0 0 0"/> -->
+      <origin xyz="0.0093 0.021 0.0" rpy="0 0 0"/>
       <axis xyz="0 1 0"/>
-      <limit velocity="4.8" effort="1" lower="0.0" upper="${0.02675-0.055}" />
+      <limit velocity="4.8" effort="1" lower="-0.01" upper="0.019" />
     </joint>
     <!--  Act 8 - Hand Finger (left) -->
     <link name="${prefix_hand}_link">
       <visual>
-        <origin xyz="0.0 0.0 0" rpy="0 0 ${M_PI/2}"/>
-        <geometry>
-          <mesh filename="file://$(find sobit_light_description)/meshes/hand/omx1_link11-12_finger.stl" scale="0.001 0.001 0.001"/>
+        <!-- <origin xyz="0.0 0.0 0.0" rpy="0 0 ${M_PI/2}"/> -->
+        <origin xyz="0.0 0.0 0.0" rpy="0 0 0"/>
+        <geometry>
+          <!-- <mesh filename="file://$(find sobit_light_description)/meshes/hand/omx1_link11-12_finger.stl" scale="0.001 0.001 0.001"/> -->
+          <mesh filename="file://$(find sobit_light_description)/meshes/hand/omx1_link11-12_finger_new.stl" scale="0.001 0.001 0.001"/>
         </geometry>
         <material name="black"/>
@@ -94,17 +98,21 @@
     <!--  Act 8 - Hand Finger (right) -->
     <joint name="${prefix_hand}_sub_joint" type="prismatic">
-      <parent link="${prefix_hand}_sub_r_link"/>
+      <!-- <parent link="${prefix_hand}_sub_r_link"/> -->
+      <parent link="${parent}"/>
       <child link="${prefix_hand}_sub_link"/>
-      <origin xyz="0.0 -0.04 0.0" rpy="0 0 0"/>
-      <axis xyz="0 1 0"/>
+      <!-- <origin xyz="0.0 -0.04 0.0" rpy="0 0 0"/> -->
+      <origin xyz="0.0093 -0.021 0.0" rpy="0 0 0"/>
+      <axis xyz="0 -1 0"/>
       <limit velocity="4.8" effort="1" lower="-1.57" upper="1.57"/>
-      <mimic joint="${prefix_hand}_joint" multiplier="-1"/>
+      <mimic joint="${prefix_hand}_joint" multiplier="1"/>
     </joint>
     <!--  Act 8 - Hand Finger (right) -->
     <link name="${prefix_hand}_sub_link">
       <visual>
-        <origin xyz="0.0 -0.0 0" rpy="0 ${M_PI} ${M_PI/2}"/>
-        <geometry>
-          <mesh filename="file://$(find sobit_light_description)/meshes/hand/omx1_link11-12_finger.stl" scale="0.001 0.001 0.001"/>
+        <!-- <origin xyz="0.0 0.0 0.0" rpy="0 ${M_PI} ${M_PI/2}"/> -->
+        <origin xyz="0.0 0.0 0.0" rpy="${M_PI} 0 0"/>
+        <geometry>
+          <!-- <mesh filename="file://$(find sobit_light_description)/meshes/hand/omx1_link11-12_finger.stl" scale="0.001 0.001 0.001"/> -->
+          <mesh filename="file://$(find sobit_light_description)/meshes/hand/omx1_link11-12_finger_new.stl" scale="0.001 0.001 0.001"/>
         </geometry>
         <material name="black"/>

Commit message: [FIX] slash is not used for model naming

File: sobit_light_description/urdf/hand/hand.urdf.xacro (robot description, xacro)
@@ -17,5 +17,5 @@
         <origin xyz="0.0 0.0 0.0" rpy="0 0 ${M_PI/2}"/>
         <geometry>
-          <mesh filename="file://$(find sobit_light_description)/meshes/hand/omx1_link11-12_finger.stl" scale="0.001 0.001 0.001"/>
+          <mesh filename="file://$(find sobit_light_description)/meshes/hand/omx1_link1112_finger.stl" scale="0.001 0.001 0.001"/>
         </geometry>
         <material name="black"/>
@@ -49,5 +49,5 @@
         <origin xyz="0.0 0.0 0.0" rpy="0 ${M_PI} ${M_PI/2}"/>
         <geometry>
-          <mesh filename="file://$(find sobit_light_description)/meshes/hand/omx1_link11-12_finger.stl" scale="0.001 0.001 0.001"/>
+          <mesh filename="file://$(find sobit_light_description)/meshes/hand/omx1_link1112_finger.stl" scale="0.001 0.001 0.001"/>
         </geometry>
         <material name="black"/>
@@ -78,5 +78,5 @@
         <origin xyz="0.0 -0.0 0" rpy="0 0 ${M_PI/2}"/>
         <geometry>
-          <mesh filename="file://$(find sobit_light_description)/meshes/hand/omx1_link13-14_finger.stl" scale="0.001 0.001 0.001"/>
+          <mesh filename="file://$(find sobit_light_description)/meshes/hand/omx1_link1314_finger.stl" scale="0.001 0.001 0.001"/>
         </geometry>
         <material name="black"/>
@@ -107,5 +107,5 @@
         <origin xyz="0.0 -0.0 0" rpy="0 ${M_PI} ${M_PI/2}"/>
         <geometry>
-          <mesh filename="file://$(find sobit_light_description)/meshes/hand/omx1_link13-14_finger.stl" scale="0.001 0.001 0.001"/>
+          <mesh filename="file://$(find sobit_light_description)/meshes/hand/omx1_link1314_finger.stl" scale="0.001 0.001 0.001"/>
         </geometry>
         <material name="black"/>
