Commit message: fix(description): hand_sub_joint bounds match hand_joint
The mimic finger is prismatic but carried the +-1.57 range copied from a
revolute joint. Use the same -0.0179..0.0290 m travel as hand_joint.

File: sobit_light_description/urdf/hand/hand.urdf.xacro (robot description, xacro)
@@ -41,5 +41,5 @@
       <origin xyz="0.059 -0.05498805 0.0" rpy="0 0 0"/>
       <axis xyz="0 -1 0"/>
-      <limit velocity="${XM430_W350_VELOCITY / HAND_GEAR_RATIO}" effort="${XM430_W350_TORQUE * HAND_GEAR_RATIO * effort_ratio}" lower="-1.57" upper="1.57"/>
+      <limit velocity="${XM430_W350_VELOCITY / HAND_GEAR_RATIO}" effort="${XM430_W350_TORQUE * HAND_GEAR_RATIO * effort_ratio}" lower="-0.01791787" upper="0.02901195" />
       <mimic joint="${prefix_hand}_joint" multiplier="1"/>
     </joint>
