Commit message: [FIX] replace cylinder to sphere for better collision gz

File: sobit_light_description/urdf/wheel/wheel.urdf.xacro (robot description, xacro)
@@ -8,5 +8,5 @@
       <origin xyz="0.0 0.100 0.045" rpy="0 0 0" />
       <axis xyz="0 1 0" />
-      <limit velocity="10" effort="100" />
+      <limit velocity="10" effort="1000" />
     </joint>
     <link name="${prefix}_l_drive_wheel_link">
@@ -14,5 +14,6 @@
         <origin xyz="0 0 0" rpy="${M_PI / 2.0} 0 0" />
         <geometry>
-          <cylinder length="0.025" radius="0.045" />
+          <!-- <cylinder length="0.025" radius="0.045" /> -->
+          <sphere radius="0.045" />
         </geometry>
         <material name="tire" />
@@ -21,5 +22,6 @@
         <origin xyz="0 0 0" rpy="${M_PI / 2.0} 0 0" />
         <geometry>
-          <cylinder length="0.025" radius="0.045" />
+          <!-- <cylinder length="0.025" radius="0.045" /> -->
+          <sphere radius="0.045" />
         </geometry>
         <material name="tire" />
@@ -28,7 +30,7 @@
         <origin xyz="0 0 0" rpy="0 0 0" />
         <mass value="0.2" />
-        <inertia ixx="0.001" ixy="0" ixz="0"
-                 iyy="0.001" iyz="0"
-                 izz="0.001" />
+        <inertia ixx="${2/5*0.2*0.045**2}" ixy="0" ixz="0"
+                 iyy="${2/5*0.2*0.045**2}" iyz="0"
+                 izz="${2/5*0.2*0.045**2}" />
       </inertial>
     </link>
@@ -39,5 +41,5 @@
       <origin xyz="0.0 -0.100 0.045" rpy="0 0 0" />
       <axis xyz="0 1 0" />
-      <limit velocity="10" effort="100" />
+      <limit velocity="10" effort="1000" />
     </joint>
     <link name="${prefix}_r_drive_wheel_link">
@@ -45,5 +47,6 @@
         <origin xyz="0 0 0" rpy="${M_PI / 2.0} 0 0" />
         <geometry>
-          <cylinder length="0.025" radius="0.045" />
+          <!-- <cylinder length="0.025" radius="0.045" /> -->
+          <sphere radius="0.045" />
         </geometry>
         <material name="tire" />
@@ -52,5 +55,6 @@
         <origin xyz="0 0 0" rpy="${M_PI / 2.0} 0 0" />
         <geometry>
-          <cylinder length="0.025" radius="0.045" />
+          <!-- <cylinder length="0.025" radius="0.045" /> -->
+          <sphere radius="0.045" />
         </geometry>
         <material name="tire" />
@@ -59,7 +63,7 @@
         <origin xyz="0 0 0" rpy="0 0 0" />
         <mass value="0.2" />
-        <inertia ixx="0.001" ixy="0" ixz="0"
-                 iyy="0.001" iyz="0"
-                 izz="0.001" />
+        <inertia ixx="${2/5*0.2*0.045**2}" ixy="0" ixz="0"
+                 iyy="${2/5*0.2*0.045**2}" iyz="0"
+                 izz="${2/5*0.2*0.045**2}" />
       </inertial>
     </link>

Commit message: [FIX] Restore wheel collision shape from sphere to cylinder

File: sobit_light_description/urdf/wheel/wheel.urdf.xacro (robot description, xacro)
@@ -14,6 +14,6 @@
         <origin xyz="0 0 0" rpy="${M_PI / 2.0} 0 0" />
         <geometry>
-          <!-- <cylinder length="0.025" radius="0.045" /> -->
-          <sphere radius="0.045" />
+          <cylinder length="0.025" radius="0.045" />
+          <!-- <sphere radius="0.045" /> -->
         </geometry>
         <material name="tire" />
@@ -22,6 +22,6 @@
         <origin xyz="0 0 0" rpy="${M_PI / 2.0} 0 0" />
         <geometry>
-          <!-- <cylinder length="0.025" radius="0.045" /> -->
-          <sphere radius="0.045" />
+          <cylinder length="0.025" radius="0.045" />
+          <!-- <sphere radius="0.045" /> -->
         </geometry>
         <material name="tire" />
@@ -47,6 +47,6 @@
         <origin xyz="0 0 0" rpy="${M_PI / 2.0} 0 0" />
         <geometry>
-          <!-- <cylinder length="0.025" radius="0.045" /> -->
-          <sphere radius="0.045" />
+          <cylinder length="0.025" radius="0.045" />
+          <!-- <sphere radius="0.045" /> -->
         </geometry>
         <material name="tire" />
@@ -55,6 +55,6 @@
         <origin xyz="0 0 0" rpy="${M_PI / 2.0} 0 0" />
         <geometry>
-          <!-- <cylinder length="0.025" radius="0.045" /> -->
-          <sphere radius="0.045" />
+          <cylinder length="0.025" radius="0.045" />
+          <!-- <sphere radius="0.045" /> -->
         </geometry>
         <material name="tire" />
