Commit message: feat(moveit): SRDF chain groups and arm end effector
Define arm and head as kinematic chains ending in hand_end_effector_link
and head_pitch_link, add a head_arm group, name the default group states
initial_pose for head, arm and hand, and declare the arm_ee end effector on
hand_end_effector_link with parent_group arm so kinematics plugins (and
MoveIt Servo, which takes its tip frame from the IK solver) target the
gripper tip rather than the wrist.

File: sobit_light_moveit_config/config/sobit_light.srdf.xacro (robot description, xacro)
@@ -32,12 +32,7 @@
     <xacro:if value="${ARM}">
         <group name="arm">
-            <joint name="arm_platform_joint"/>
-            <joint name="arm_base_joint"/>
+            <link name="hand_end_effector_link"/>
             <joint name="arm_shoulder_roll_joint"/>
-            <joint name="arm_shoulder_pitch_joint"/>
-            <joint name="arm_elbow_pitch_joint"/>
-            <joint name="arm_forearm_roll_joint"/>
-            <joint name="arm_wrist_pitch_joint"/>
-            <joint name="arm_wrist_roll_joint"/>
+            <chain base_link="arm_shoulder_roll_link" tip_link="arm_wrist_roll_link"/>
         </group>
     </xacro:if>
@@ -46,4 +41,5 @@
     <xacro:if value="${HAND}">
         <group name="hand">
+            <link name="hand_end_effector_link"/>
             <joint name="hand_joint"/>
         </group>
@@ -51,11 +47,24 @@
     <xacro:if value="${HEAD}">
         <group name="head">
+            <link name="head_pitch_link"/>
             <joint name="head_yaw_joint"/>
-            <joint name="head_pitch_joint"/>
+            <chain base_link="head_yaw_link" tip_link="head_pitch_link"/>
         </group>
     </xacro:if>
+    <xacro:if value="${HEAD and ARM}">
+        <group name="head_arm">
+            <group name="head"/>
+            <group name="arm"/>
+        </group>
+    </xacro:if>
     <!--GROUP STATES: Purpose: Define a named state for a particular group, in terms of joint values. This is useful to define states like 'folded arms'-->
+    <xacro:if value="${HEAD}">
+        <group_state name="initial_pose" group="head">
+            <joint name="head_yaw_joint" value="0"/>
+            <joint name="head_pitch_joint" value="0"/>
+        </group_state>
+    </xacro:if>
     <xacro:if value="${ARM}">
-        <group_state name="home" group="arm">
+        <group_state name="initial_pose" group="arm">
             <joint name="arm_elbow_pitch_joint" value="0.0"/>
             <joint name="arm_forearm_roll_joint" value="0.0"/>
@@ -66,7 +75,12 @@
         </group_state>
     </xacro:if>
+    <xacro:if value="${HAND}">
+        <group_state name="initial_pose" group="hand">
+            <joint name="hand_joint" value="0.0"/>
+        </group_state>
+    </xacro:if>
     <!--END EFFECTOR: Purpose: Represent information about an end effector.-->
     <xacro:if value="${HAND}">
-        <end_effector name="hand" parent_link="arm_wrist_roll_link" group="hand"/>
+        <end_effector name="arm_ee" parent_link="hand_end_effector_link" group="hand" parent_group="arm"/>
     </xacro:if>
     <!--VIRTUAL JOINT: Purpose: this element defines a virtual joint between a robot link and an external frame of reference (considered fixed with respect to the robot)-->
